File: Power/PCB/MAX17634C/12V buck converter/12V buck converter.kicad_sch (KiCad schematic)
At the start: 11 parts, among them IC1 MAX17634

Commit message: Update pcb
Parts:
- IC1: Order (none) -> https://nl.farnell.com/analog-devices/max17634catp/dc-dc-co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
- L1: footprint (none) -> Inductor_SMD:L_6.3x6.3_H3
- R1, R2, R3: footprint (none) -> Resistor_SMD:R_0402_1005Metric
Connections:
- net Vin: now reaches C1.1, C2.1, IC1.14 (IN), IC1.2 (IN), IC1.3 (IN), IC1.4 (EN/UVLO)
- net Earth renamed GND
- net GND: now also IC1.21 (SGND)
- no-connect marks 0 -> 2
Other:
- moved on the sheet: R3
