File: KiCAD/Main board/DAC CH 5_6.kicad_sch (KiCad schematic)
At the start: 0 parts

Commit message: Updated BACK-END
Parts:
- added C1, C20, C22, C23, C24, C28, C30, C4, C5: 22uF, Capacitor_THT:CP_Radial_D5.0mm_P2.00mm, symbol Device:C_Polarized
- added C10, C17: 680p, Capacitor_SMD:C_0805_2012Metric, symbol Device:C
- added C11, C18: 680, Capacitor_SMD:C_0805_2012Metric, symbol Device:C
- added C12, C27: 2.2n, Capacitor_SMD:C_0805_2012Metric, symbol Device:C
- added C15, C16, C21, C25, C26: 100nF, Capacitor_SMD:C_0805_2012Metric, symbol Device:C
- added C19, C2, C3, C35: 100n, Capacitor_SMD:C_0805_2012Metric, symbol Device:C
- added R1 (x4): 22R, Resistor_SMD:R_0805_2012Metric, symbol Device:R
- added R12, R16, R20, R21: 1k, Resistor_SMD:R_0805_2012Metric, symbol Device:R
- added R13, R17, R22, R23: 4.7k, Resistor_SMD:R_0805_2012Metric, symbol Device:R
- added R14, R15, R30, R37: 39, Resistor_SMD:R_0805_2012Metric, symbol Device:R
- added R24, R31, R32, R33, R34, R35, R36, R38: 10, Resistor_SMD:R_0805_2012Metric, symbol Device:R
- added U1: LM4562, Package_SO:SOIC-8_3.9x4.9mm_P1.27mm, symbol Main board-rescue:LM4562-Audio_DSP
- added U3, U4: OPA1632DR, Audio_DSP:VSSOP-8_3.0x3.0mm_P0.65_TP1.8x1.5, symbol Audio-DSP:OPA1632DR
Connections:
- new net: C1.1, C3.1, R34.1, U1.16 (VCC2)
- new net: C16.2, C24.2, R35.2, U3.6 (V-)
- new net: C17.1, R20.2, R22.1, U4.8 (VIN+)
- new net: C18.1, R21.2, R23.1, U4.1 (VIN-)
- new net: C18.2, R37.1, U4.4 (VOUT+)
- new net: C17.2, R30.1, U4.5 (VOUT-)
- new net: C15.1, C23.1, R24.1, U3.3 (V+)
- new net: C25.1, C28.1, R36.1, U4.3 (V+)
- new net: C21.2, C22.2, R31.2, U1.4 (V-)
- new net: R20.1, U1.13 (VOUTR+)
- new net: C35.1, C4.1, R32.1, U1.8 (V+)
- new net: C2.1, C5.1, R33.1, U1.8 (VCC1)
- new net: C11.1, R16.2, R17.1, U3.1 (VIN-)
- new net: C11.2, R15.1, U3.4 (VOUT+)
- new net: C10.2, R14.1, U3.5 (VOUT-)
- new net: C10.1, R12.2, R13.1, U3.8 (VIN+)
- new net: R1.2, U1.2 (BCK)
- new net: R1.2, U1.5 (SCKI)
- new net: R1.2, U1.3 (DIN)
- new net: C26.2, C30.2, R38.2, U4.6 (V-)
- new net: R21.1, U1.14 (VOUTR-)
- new net: R16.1, U1.11 (VOUTL-)
- new net: R1.2, U1.1 (LRCK)
- new net: R12.1, U1.12 (VOUTL+)
- new net +12V: R24.2, R32.2, R36.2
- new net +3.3V: C19.1, C20.1, U1.6 (VDD)
- new net +5V: R33.2, R34.2
- new net -12V: R31.1, R35.1, R38.1
- new net AMUTEI: U1.17 (AMUTEI)
- new net BCK: R1.1
- new net DIN: R1.1
- new net GND: C1.2, C15.2, C16.1, C19.2, C2.2, C20.2, C21.1, C22.1, C23.2, C24.1, C25.2, C26.1, C28.2, C3.2, C30.1, C35.2, C4.2, C5.2, U1.10 (AGND1), U1.15 (AGND2), U1.23 (MS/ADR0/RSV), U1.24 (ADR5/ADR1/RSV), U1.7 (DGND), U3.2 (VOCM), U3.7 (ENABLE), U3.9 (GND), U4.2 (VOCM), U4.7 (ENABLE), U4.9 (GND)
- new net LRCK: R1.1
- new net MC/SCL/FMT: U1.22 (MC/SCL/FMT)
- new net MD/SDA/DEMP: U1.21 (MD/SDA/DEMP)
- new net MODE: U1.20 (MODE)
- new net RST: U1.4 (RST)
- new net SCKI: R1.1
- new net VOUT CH5(+): C12.2, R15.2, R17.2
- new net VOUT CH5(-): C12.1, R13.2, R14.2
- new net VOUT CH6(+): C27.2, R23.2, R37.2
- new net VOUT CH6(-): C27.1, R22.2, R30.2
- no-connect marks 0 -> 3
