File: KiCAD/Main board/untitled.kicad_sch (KiCad schematic)
At the start: 5 parts, among them IC1 OPA1632DR, IC2 PCM1789-Q1, U1 LM4562

Commit message: Started on Front-END
Parts:
- removed C1: C, symbol Device:C
- removed IC1: OPA1632DR, Audio_DSP:VSSOP-8_3.0x3.0mm_P0.65_TP1.8x1.5, symbol Main board-rescue:OPA1632DR-Audio_DSP
- removed IC2: PCM1789-Q1, Package_SO:TSSOP-24_4.4x7.8mm_P0.65mm, symbol Main board-rescue:PCM1789-Q1-Audio_DSP
- removed R1: 1k, Resistor_SMD:R_0805_2012Metric, symbol Device:R
- removed U1: LM4562, Package_SO:SOIC-8_3.9x4.9mm_P1.27mm, symbol Main board-rescue:LM4562-Audio_DSP
- added C10, C11: 1n, Capacitor_SMD:C_0805_2012Metric, symbol Device:C
- added C12: 2.7n, Capacitor_SMD:C_0805_2012Metric, symbol Device:C
- added C21 (x2), C25, C26: 100nF, Capacitor_SMD:C_0805_2012Metric, symbol Device:C
- added C22 (x2), C28, C30, C4 (x2): 22uF, Capacitor_THT:CP_Radial_D5.0mm_P2.00mm, symbol Device:C_Polarized
- added C35 (x2): 100n, Capacitor_SMD:C_0805_2012Metric, symbol Device:C
- added C82: 100n, symbol Device:C
- added C83, C97: 3n3, symbol Device:C
- added R103: 2.2MEG, symbol Device:R
- added R105, R116, R117: R, symbol Device:R
- added R114, R94: 47K, symbol Device:R
- added R115, R95: 220, symbol Device:R
- added R118: 1K, symbol Device:R
- added R12: 1k, Resistor_SMD:R_0805_2012Metric, symbol Device:R
- added R13: 270, Resistor_SMD:R_0805_2012Metric, symbol Device:R
- added R14, R15: 39, Resistor_SMD:R_0805_2012Metric, symbol Device:R
- added R31 (x2), R32 (x2), R36, R38: 10, Resistor_SMD:R_0805_2012Metric, symbol Device:R
- added R93: 1k, symbol Device:R
- added R97: 270, symbol Device:R
- added R98, R99: 10k, symbol Device:R
- added U14, U17: LM4562, symbol Amplifier_Operational:LM4562
- added U5: OPA1632DR, Audio_DSP:VSSOP-8_3.0x3.0mm_P0.65_TP1.8x1.5, symbol Audio-DSP:OPA1632DR
Connections:
- new net: R114.2, R115.1
- new net: C97.2, R115.2, U17.3 (+)
- new net: R103.1, R114.1, R94.2
- new net: R105.2, R118.1, U17.1
- new net: R105.1, R116.2, U17.2 (-)
- new net: C11.1, R118.2, R97.1, U5.1 (VIN-)
- new net: C21.2, C22.2, R31.2, U17.4 (V-)
- new net: C35.1, C4.1, R32.1, U17.8 (V+)
- new net: C35.1, C4.1, R32.1, U14.4 (V-)
- new net: C26.2, C30.2, R38.2, U5.6 (V-)
- new net: C11.2, R15.1, U5.4 (VOUT+)
- new net: C12.2, R15.2, R97.2, R99.1
- new net: C25.1, C28.1, R36.1, U5.3 (V+)
- new net: C21.2, C22.2, R31.2, U14.8 (V+)
- new net: R94.1, R95.1
- new net: C83.1, R95.2, U14.3 (+)
- new net: R117.2, R12.1, U14.1
- new net: C10.1, R12.2, R13.1, U5.8 (VIN+)
- new net: C12.1, R13.2, R14.2, R98.1
- new net: C10.2, R14.1, U5.5 (VOUT-)
- new net: R117.1, U14.2 (-)
- new net: C82.1, R93.1, U14.5 (+)
- new net: U14.6 (-), U14.7, U5.2 (VOCM)
- new net +12V: R32.2, R32.2, R36.2
- new net -12V: R31.1, R31.1, R38.1
- new net GND: C21.1, C21.1, C22.1, C22.1, C25.2, C26.1, C28.2, C30.1, C35.2, C35.2, C4.2, C4.2, C82.2, C83.2, C97.1, R103.2, R98.2, R99.2, U5.7 (ENABLE), U5.9 (GND)
- no-connect marks 0 -> 3
