File: KiCAD/Main board/Main board.kicad_pcb (KiCad board)
At the start: 2 copper layers, 5 parts, among them IC1 OPA1632DR, IC2 PCM1789-Q1, J1 Conn_01x03, U1 LM4562

Commit message: BACK-END PCB
Parts:
- added IC2: PCM1789-Q1, Package_SO:TSSOP-24_4.4x7.8mm_P0.65mm, F.Cu at (77.2, 48.9)
- added J2: Conn_01x03, Connector_JST:JST_PH_B3B-PH-K_1x03_P2.00mm_Vertical, F.Cu at (75.8, 58.3)
- added R1: 22R, Resistor_SMD:R_0805_2012Metric, F.Cu at (75.1, 28.0)
- added R10: R, Resistor_SMD:R_0805_2012Metric, F.Cu at (79.5, 36.8)
- added R11: R, Resistor_SMD:R_0805_2012Metric, F.Cu at (79.5, 39.8)
- added R12: R, Resistor_SMD:R_0805_2012Metric, F.Cu at (79.5, 42.7)
- added R13: R, Resistor_SMD:R_0805_2012Metric, F.Cu at (83.9, 28.0)
- added R14: R, Resistor_SMD:R_0805_2012Metric, F.Cu at (83.9, 30.9)
- added R15: R, Resistor_SMD:R_0805_2012Metric, F.Cu at (83.9, 33.9)
- added R16: R, Resistor_SMD:R_0805_2012Metric, F.Cu at (83.9, 36.8)
- added R17: R, Resistor_SMD:R_0805_2012Metric, F.Cu at (83.9, 39.8)
- added R18: R, Resistor_SMD:R_0805_2012Metric, F.Cu at (83.9, 42.7)
- added R19: R, Resistor_SMD:R_0805_2012Metric, F.Cu at (88.3, 28.0)
- added R2: 22R, Resistor_SMD:R_0805_2012Metric, F.Cu at (75.1, 30.9)
- added R20: R, Resistor_SMD:R_0805_2012Metric, F.Cu at (88.3, 30.9)
- added R21: R, Resistor_SMD:R_0805_2012Metric, F.Cu at (88.3, 33.9)
- added R22: R, Resistor_SMD:R_0805_2012Metric, F.Cu at (88.3, 36.8)
- added R23: R, Resistor_SMD:R_0805_2012Metric, F.Cu at (88.3, 39.8)
- added R24: R, Resistor_SMD:R_0805_2012Metric, F.Cu at (88.3, 42.7)
- added R25: R, Resistor_SMD:R_0805_2012Metric, F.Cu at (92.7, 28.0)
- added R26: R, Resistor_SMD:R_0805_2012Metric, F.Cu at (92.7, 30.9)
- added R27: R, Resistor_SMD:R_0805_2012Metric, F.Cu at (92.7, 33.9)
- added R28: R, Resistor_SMD:R_0805_2012Metric, F.Cu at (92.7, 36.8)
- added R29: R, Resistor_SMD:R_0805_2012Metric, F.Cu at (92.7, 39.8)
- added R3: 22R, Resistor_SMD:R_0805_2012Metric, F.Cu at (75.1, 33.9)
- added R30: R, Resistor_SMD:R_0805_2012Metric, F.Cu at (92.7, 42.7)
- added R4: 22R, Resistor_SMD:R_0805_2012Metric, F.Cu at (75.1, 36.8)
- added R5: R, Resistor_SMD:R_0805_2012Metric, F.Cu at (75.1, 39.8)
- added R6: R, Resistor_SMD:R_0805_2012Metric, F.Cu at (75.1, 42.7)
- added R7: R, Resistor_SMD:R_0805_2012Metric, F.Cu at (79.5, 28.0)
- added R8: R, Resistor_SMD:R_0805_2012Metric, F.Cu at (79.5, 30.9)
- added R9: R, Resistor_SMD:R_0805_2012Metric, F.Cu at (79.5, 33.9)
- added U1: LM4562, Package_SO:SOIC-8_3.9x4.9mm_P1.27mm, F.Cu at (99.1, 29.7)
- added U2: LM4562, Package_SO:SOIC-8_3.9x4.9mm_P1.27mm, F.Cu at (99.1, 36.2)
- moved IC1 67.1 mm to (110.0, 67.6)
- moved J1 67.1 mm to (102.4, 53.6)
- moved R1 67.1 mm to (92.2, 59.9)
- moved U1 67.1 mm to (110.2, 62.0)
- moved IC2 67.1 mm to (101.6, 63.5)
Connections:
- J1 pad 1: Net-(J1-Pad1) -> unconnected-(J1-Pin_1-Pad1)
- J1 pad 2: Net-(J1-Pad2) -> unconnected-(J1-Pin_2-Pad2)
- J1 pad 3: Net-(J1-Pad3) -> unconnected-(J1-Pin_3-Pad3)
Other:
- net class Default removed

Commit message: KICAD
Parts:
- added C1: 22uF, Capacitor_THT:CP_Radial_D5.0mm_P2.00mm, F.Cu at (78.7, 27.1)
- added C10: 680p, Capacitor_SMD:C_0805_2012Metric, F.Cu at (78.5, 63.0)
- added C11: 680, Capacitor_SMD:C_0805_2012Metric, F.Cu at (83.0, 44.9)
- added C12: 2.2n, Capacitor_SMD:C_0805_2012Metric, F.Cu at (83.0, 47.9)
- added C13: 5.6n, Capacitor_SMD:C_0805_2012Metric, F.Cu at (83.0, 51.0)
- added C14: 2.2n, Capacitor_SMD:C_0805_2012Metric, F.Cu at (83.0, 54.0)
- added C15: 100nF, Capacitor_SMD:C_0805_2012Metric, F.Cu at (83.0, 57.0)
- added C16: 22uF, Capacitor_THT:CP_Radial_D5.0mm_P2.00mm, F.Cu at (85.3, 27.1)
- added C17: 1N, Capacitor_SMD:C_0805_2012Metric, F.Cu at (83.0, 60.0)
- added C18: 680p, Capacitor_SMD:C_0805_2012Metric, F.Cu at (83.0, 63.0)
- added C19: 100nF, Capacitor_SMD:C_0805_2012Metric, F.Cu at (87.4, 44.9)
- added C2: 100nF, Capacitor_SMD:C_0805_2012Metric, F.Cu at (78.5, 44.9)
- added C20: 22uF, Capacitor_THT:CP_Radial_D5.0mm_P2.00mm, F.Cu at (85.3, 33.6)
- added C21: 100nF, Capacitor_SMD:C_0805_2012Metric, F.Cu at (87.4, 47.9)
- added C22: 22uF, Capacitor_THT:CP_Radial_D5.0mm_P2.00mm, F.Cu at (85.3, 40.1)
- added C23: 100nF, Capacitor_SMD:C_0805_2012Metric, F.Cu at (87.4, 51.0)
- added C24: 22uF, Capacitor_THT:CP_Radial_D5.0mm_P2.00mm, F.Cu at (92.0, 27.1)
- added C25: 100nF, Capacitor_SMD:C_0805_2012Metric, F.Cu at (87.4, 54.0)
- added C26: 22uF, Capacitor_THT:CP_Radial_D5.0mm_P2.00mm, F.Cu at (92.0, 33.6)
- added C27: 680, Capacitor_SMD:C_0805_2012Metric, F.Cu at (87.4, 57.0)
- added C28: 100nF, Capacitor_SMD:C_0805_2012Metric, F.Cu at (87.4, 60.0)
- added C29: 2.2n, Capacitor_SMD:C_0805_2012Metric, F.Cu at (87.4, 63.0)
- added C3: 100nF, Capacitor_SMD:C_0805_2012Metric, F.Cu at (78.5, 47.9)
- added C30: 22uF, Capacitor_THT:CP_Radial_D5.0mm_P2.00mm, F.Cu at (92.0, 40.1)
- added C4: 22uF, Capacitor_THT:CP_Radial_D5.0mm_P2.00mm, F.Cu at (78.7, 33.6)
- added C5: 22uF, Capacitor_THT:CP_Radial_D5.0mm_P2.00mm, F.Cu at (78.7, 40.1)
- added C6: 100nF, Capacitor_SMD:C_0805_2012Metric, F.Cu at (78.5, 51.0)
- added C7: 5.6n, Capacitor_SMD:C_0805_2012Metric, F.Cu at (78.5, 54.0)
- added C8: 2.2n, Capacitor_SMD:C_0805_2012Metric, F.Cu at (78.5, 57.0)
- added C9: 1N, Capacitor_SMD:C_0805_2012Metric, F.Cu at (78.5, 60.0)
- added J3: Conn_01x02, Connector_JST:JST_PH_B2B-PH-K_1x02_P2.00mm_Vertical, F.Cu at (109.6, 26.5)
- added J4: Conn_01x03, Connector_JST:JST_PH_B3B-PH-K_1x03_P2.00mm_Vertical, F.Cu at (117.6, 26.5)
- added J5: Conn_01x02, Connector_JST:JST_PH_B2B-PH-K_1x02_P2.00mm_Vertical, F.Cu at (109.6, 49.9)
- added R18: 10K, Resistor_SMD:R_0805_2012Metric, F.Cu at (91.9, 44.9)
- added R19: 10K, Resistor_SMD:R_0805_2012Metric, F.Cu at (91.9, 47.9)
- added R20: 1k, Resistor_SMD:R_0805_2012Metric, F.Cu at (91.9, 50.8)
- added R21: 1k, Resistor_SMD:R_0805_2012Metric, F.Cu at (91.9, 53.8)
- added R22: 4.7k, Resistor_SMD:R_0805_2012Metric, F.Cu at (91.9, 56.7)
- added R23: 4.3k, Resistor_SMD:R_0805_2012Metric, F.Cu at (91.9, 59.6)
- added R24: 10, Resistor_SMD:R_0805_2012Metric, F.Cu at (91.9, 62.6)
- added R25: 820, Resistor_SMD:R_0805_2012Metric, F.Cu at (96.3, 44.9)
- added R26: 820, Resistor_SMD:R_0805_2012Metric, F.Cu at (96.3, 47.9)
- added R27: 4.7k, Resistor_SMD:R_0805_2012Metric, F.Cu at (96.3, 50.8)
- added R28: 4.3K, Resistor_SMD:R_0805_2012Metric, F.Cu at (96.3, 53.8)
- added R29: 22, Resistor_SMD:R_0805_2012Metric, F.Cu at (96.3, 56.7)
- added R30: 39, Resistor_SMD:R_0805_2012Metric, F.Cu at (96.3, 59.6)
- added R31: 10, Resistor_SMD:R_0805_2012Metric, F.Cu at (96.3, 62.6)
- added R32: 10, Resistor_SMD:R_0805_2012Metric, F.Cu at (100.7, 44.9)
- added R33: 10, Resistor_SMD:R_0805_2012Metric, F.Cu at (100.7, 47.9)
- added R34: 10, Resistor_SMD:R_0805_2012Metric, F.Cu at (100.7, 50.8)
- added R35: 10, Resistor_SMD:R_0805_2012Metric, F.Cu at (100.7, 53.8)
- added R36: 10, Resistor_SMD:R_0805_2012Metric, F.Cu at (100.7, 56.7)
- added R37: 39, Resistor_SMD:R_0805_2012Metric, F.Cu at (100.7, 59.6)
- added R38: 10, Resistor_SMD:R_0805_2012Metric, F.Cu at (100.7, 62.6)
- added U2: LM4562, Package_SO:SOIC-8_3.9x4.9mm_P1.27mm, F.Cu at (100.4, 27.0)
- R1: value 1k -> 22R
- R10, R29: value R -> 22
- R11, R28: value R -> 4.3K
- R12, R16, R20, R21: value R -> 1k
- R13, R17, R22, R27: value R -> 4.7k
- R14, R15, R30: value R -> 39
- R18, R19, R5, R6: value R -> 10K
- R23, R9: value R -> 4.3k
- R24: value R -> 10
- R25, R26, R7, R8: value R -> 820
- moved IC1 76.0 mm to (34.0, 66.7)
- moved IC2 76.0 mm to (25.6, 62.6)
- moved IC2 76.0 mm to (1.26, 48.0)
- moved J1 76.0 mm to (26.4, 52.7)
- moved J2 76.0 mm to (-0.14, 57.4)
- moved R1 76.0 mm to (16.2, 59.0)
- moved R1 76.0 mm to (-0.91, 27.1)
- moved R10 76.0 mm to (3.50, 35.9)
- moved R11 76.0 mm to (3.50, 38.9)
- moved R12 76.0 mm to (3.50, 41.8)
- moved R13 76.0 mm to (7.91, 27.1)
- moved R14 76.0 mm to (7.91, 30.0)
- moved R15 76.0 mm to (7.91, 33.0)
- moved R16 76.0 mm to (7.91, 35.9)
- moved R17 76.0 mm to (7.91, 38.9)
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Connections:
- IC1 pad 1: Net-(IC1-Pad1) -> Net-(IC1-VIN-)
- IC1 pad 2: Net-(IC1-Pad2) -> GND
- IC1 pad 3: Net-(IC1-Pad3) -> GND
- IC1 pad 4: Net-(IC1-Pad4) -> Net-(IC1-VOUT+)
- IC1 pad 5: Net-(IC1-Pad5) -> Net-(IC1-VOUT-)
- IC1 pad 6: Net-(IC1-Pad6) -> GND
- IC1 pad 7: Net-(IC1-Pad7) -> GND
- IC1 pad 8: Net-(IC1-Pad8) -> Net-(IC1-VIN+)
- IC1 pad 9: Net-(IC1-Pad9) -> GND
- IC2 pad 1: Net-(IC2-Pad1) -> Net-(IC2-LRCK)
- IC2 pad 10: Net-(IC2-Pad10) -> GND
- IC2 pad 11: Net-(IC2-Pad11) -> Net-(IC2-VOUTL-)
- IC2 pad 12: Net-(IC2-Pad12) -> Net-(IC2-VOUTL+)
- IC2 pad 13: Net-(IC2-Pad13) -> Net-(IC2-VOUTR+)
- IC2 pad 14: Net-(IC2-Pad14) -> Net-(IC2-VOUTR-)
- IC2 pad 15: Net-(IC2-Pad15) -> GND
- IC2 pad 16: Net-(IC2-Pad16) -> GND
- IC2 pad 17: Net-(IC2-Pad17) -> /DAC CH1_2/AMUTEI
- IC2 pad 18: Net-(IC2-Pad18) -> unconnected-(IC2-ZERO2/AMUTEO-Pad18)
- IC2 pad 19: Net-(IC2-Pad19) -> unconnected-(IC2-ZERO1-Pad19)
- IC2 pad 2: Net-(IC2-Pad2) -> Net-(IC2-BCK)
- IC2 pad 20: Net-(IC2-Pad20) -> /DAC CH1_2/MODE
- IC2 pad 21: Net-(IC2-Pad21) -> /DAC CH1_2/MD/SDA/DEMP
- IC2 pad 22: Net-(IC2-Pad22) -> /DAC CH1_2/MC/SCL/FMT
- IC2 pad 23: Net-(IC2-Pad23) -> /DAC CH1_2/ADR0
- IC2 pad 24: Net-(IC2-Pad24) -> /DAC CH1_2/ADR1
- IC2 pad 3: Net-(IC2-Pad3) -> Net-(IC2-DIN)
- IC2 pad 4: Net-(IC2-Pad4) -> /DAC CH1_2/RST
- IC2 pad 5: Net-(IC2-Pad5) -> Net-(IC2-SCKI)
- IC2 pad 6: Net-(IC2-Pad6) -> +3.3V
- IC2 pad 7: Net-(IC2-Pad7) -> GND
- IC2 pad 8: Net-(IC2-Pad8) -> GND
- IC2 pad 9: Net-(IC2-Pad9) -> unconnected-(IC2-VCOM-Pad9)
- IC2 pad 10: +3.3V -> GND
- IC2 pad 15: +3.3V -> GND
- IC2 pad 16: +3.3V -> GND
- IC2 pad 7: +3.3V -> GND
- IC2 pad 8: +3.3V -> GND
- J2 pad 1: unconnected-(J2-Pin_1-Pad1) -> /DAC CH1_2/VOUT CH1(+)
- J2 pad 2: unconnected-(J2-Pin_2-Pad2) -> GND
- J2 pad 3: unconnected-(J2-Pin_3-Pad3) -> /DAC CH1_2/VOUT CH1(-)
- R1 pad 1: Net-(R1-Pad1) -> /DAC CH1_2/LRCK
- R1 pad 2: Net-(R1-Pad2) -> Net-(IC2-LRCK)
- R10 pad 1: Net-(C6-Pad2) -> Net-(C9-Pad2)
- R10 pad 2: /DAC CH1_2/RCA JACK L -> /DAC CH1_2/RCA JACK CH1
- R11 pad 2: Net-(C6-Pad2) -> Net-(C9-Pad2)
- R13 pad 2: /DAC CH1_2/VOUTL- -> /DAC CH1_2/VOUT CH1(-)
- R14 pad 2: /DAC CH1_2/VOUTL- -> /DAC CH1_2/VOUT CH1(-)
- R15 pad 2: /DAC CH1_2/VOUTL+ -> /DAC CH1_2/VOUT CH1(+)
- R17 pad 2: /DAC CH1_2/VOUTL+ -> /DAC CH1_2/VOUT CH1(+)
- R18 pad 1: Net-(IC2-VOUTR-) -> Net-(C13-Pad1)
- R18 pad 2: Net-(IC3-VIN-) -> Net-(IC2-VOUTR-)
- R19 pad 1: Net-(C9-Pad1) -> Net-(IC2-VOUTR+)
- R19 pad 2: Net-(IC2-VOUTR-) -> Net-(C13-Pad2)
- R20 pad 1: Net-(IC2-VOUTR+) -> Net-(IC2-VOUTR-)
- R20 pad 2: Net-(C9-Pad2) -> Net-(IC3-VIN-)
- R22 pad 2: /DAC CH1_2/VOUTR+ -> /DAC CH1_2/VOUT CH1(+)
- R23 pad 1: Net-(C9-Pad2) -> Net-(C13-Pad2)
- R23 pad 2: +3.3V -> GND
- R24 pad 1: Net-(C9-Pad2) -> -12V
- R24 pad 2: Net-(U2B--) -> Net-(C15-Pad2)
- R25 pad 1: Net-(C9-Pad1) -> Net-(C13-Pad1)
- R25 pad 2: Net-(U2B-+) -> Net-(U2A-+)
- R26 pad 1: Net-(IC3-VIN+) -> Net-(C13-Pad2)
- R26 pad 2: /DAC CH1_2/VOUTR- -> Net-(U2A--)
- R27 pad 1: Net-(C9-Pad1) -> Net-(IC3-VIN+)
- R27 pad 2: Net-(C11-Pad2) -> /DAC CH1_2/VOUT CH1(-)
- R28 pad 1: Net-(C11-Pad2) -> Net-(C13-Pad1)
- R28 pad 2: /DAC CH1_2/RCA/JACK R -> Net-(C17-Pad2)
- R29 pad 1: Net-(IC3-VOUT-) (its old number) -> Net-(C17-Pad2)
- R29 pad 2: /DAC CH1_2/VOUTR- -> /DAC CH1_2/RCA JACK CH1
- R30 pad 2: /DAC CH1_2/VOUTR+ -> /DAC CH1_2/VOUT CH1(-)
- R9 pad 2: +3.3V -> GND
- U1 pad 1: Net-(U1-Pad1) -> Net-(C9-Pad2)
- U1 pad 2: Net-(U1-Pad2) -> Net-(U1A--)
- U1 pad 3: Net-(U1-Pad3) -> Net-(U1A-+)
- U1 pad 4: Net-(U1-Pad4) -> Net-(U1C-V-)
- U1 pad 5: Net-(U1-Pad5) -> (no net)
- U1 pad 6: Net-(U1-Pad6) -> (no net)
- U1 pad 7: Net-(U1-Pad7) -> (no net)
- U1 pad 8: Net-(U1-Pad8) -> Net-(U1C-V+)
- U1 pad 1: Net-(C6-Pad2) -> Net-(C9-Pad2)
- U1 pad 4: -12V -> Net-(U1C-V-)
- U1 pad 8: +12V -> Net-(U1C-V+)
- U2 pad 1: (no net) -> Net-(C17-Pad2)
- U2 pad 2: (no net) -> Net-(U2A--)
- U2 pad 3: (no net) -> Net-(U2A-+)
- U2 pad 5: Net-(U2B-+) -> (no net)
- U2 pad 6: Net-(U2B--) -> (no net)
- U2 pad 7: Net-(C11-Pad2) -> (no net)

Commit message: Worked on KiCAD
Parts:
- removed IC1: OPA1632DR, Audio_DSP:VSSOP-8_3.0x3.0mm_P0.65_TP1.8x1.5
- removed IC2 (x2): PCM1789-Q1, Package_SO:TSSOP-24_4.4x7.8mm_P0.65mm
- removed the R1 at (16.2, 59.0)
- removed the R1 at (-0.91, 27.1)
- removed the R18 at (7.91, 41.8)
- removed the R18 at (91.9, 44.9)
- removed the R19 at (91.9, 47.9)
- removed the R19 at (12.3, 27.1)
- removed the R20 at (91.9, 50.8)
- removed the R20 at (12.3, 30.0)
- removed the R21 at (91.9, 53.8)
- removed the R21 at (12.3, 33.0)
- removed the R22 at (91.9, 56.7)
- removed the R22 at (12.3, 35.9)
- removed the R23 at (12.3, 38.9)
- removed the R23 at (91.9, 59.6)
- removed the R24 at (12.3, 41.8)
- removed the R24 at (91.9, 62.6)
- removed the R25 at (16.7, 27.1)
- removed the R25 at (96.3, 44.9)
- removed the R26 at (16.7, 30.0)
- removed the R26 at (96.3, 47.9)
- removed the R27 at (16.7, 33.0)
- removed the R27 at (96.3, 50.8)
- removed the R28 at (96.3, 53.8)
- removed the R28 at (16.7, 35.9)
- removed the R29 at (96.3, 56.7)
- removed the R29 at (16.7, 38.9)
- removed the R30 at (96.3, 59.6)
- removed the R30 at (16.7, 41.8)
- removed the U1 at (34.2, 61.1)
- removed the U1 at (23.2, 28.8)
- removed the U2 at (23.2, 35.3)
- removed the U2 at (100.4, 27.0)
- added C100: 22uF, Capacitor_THT:CP_Radial_D5.0mm_P2.00mm, F.Cu at (385.9, 72.6)
- added C101: 22uF, Capacitor_THT:CP_Radial_D5.0mm_P2.00mm, F.Cu at (385.9, 79.1)
- added C102: 100n, Capacitor_SMD:C_0805_2012Metric, F.Cu at (396.8, 91.6)
- added C103: 100nF, Capacitor_SMD:C_0805_2012Metric, F.Cu at (401.3, 85.6)
- added C104: 22uF, Capacitor_THT:CP_Radial_D5.0mm_P2.00mm, F.Cu at (385.9, 85.7)
- added C105: 22uF, Capacitor_THT:CP_Radial_D5.0mm_P2.00mm, F.Cu at (385.9, 92.2)
- added C106: 100n, Capacitor_SMD:C_0805_2012Metric, F.Cu at (401.3, 88.6)
- added C107: 100nF, Capacitor_SMD:C_0805_2012Metric, F.Cu at (401.3, 91.6)
- added C108: 22uF, Capacitor_THT:CP_Radial_D5.0mm_P2.00mm, F.Cu at (385.9, 98.8)
- added C109: 22uF, Capacitor_THT:CP_Radial_D5.0mm_P2.00mm, F.Cu at (385.9, 105.3)
- added C31: 100nF, Capacitor_SMD:C_0805_2012Metric, F.Cu at (314.4, 93.5)
- added C32: 22uF, Capacitor_THT:CP_Radial_D5.0mm_P2.00mm, F.Cu at (314.6, 72.6)
- added C33: 22uF, Capacitor_THT:CP_Radial_D5.0mm_P2.00mm, F.Cu at (314.6, 79.1)
- added C34: 22uF, Capacitor_THT:CP_Radial_D5.0mm_P2.00mm, F.Cu at (314.6, 85.7)
- added C35: 100n, Capacitor_SMD:C_0805_2012Metric, F.Cu at (373.9, 41.0)
- added C36: 100n, Capacitor_SMD:C_0805_2012Metric, F.Cu at (314.4, 96.5)
- added C37: 100nF, Capacitor_SMD:C_0805_2012Metric, F.Cu at (314.4, 99.5)
- added C38: 100nF, Capacitor_SMD:C_0805_2012Metric, F.Cu at (314.4, 102.5)
- added C39: 100n, Capacitor_SMD:C_0805_2012Metric, F.Cu at (314.4, 105.5)
- added C40: 22uF, Capacitor_THT:CP_Radial_D5.0mm_P2.00mm, F.Cu at (321.2, 72.6)
- added C41: 22uF, Capacitor_THT:CP_Radial_D5.0mm_P2.00mm, F.Cu at (321.2, 79.1)
- added C42: 100n, Capacitor_SMD:C_0805_2012Metric, F.Cu at (318.9, 90.5)
- added C43: 22uF, Capacitor_THT:CP_Radial_D5.0mm_P2.00mm, F.Cu at (321.2, 85.7)
- added C44: 22uF, Capacitor_THT:CP_Radial_D5.0mm_P2.00mm, F.Cu at (83.2, 86.5)
- added C45: 100nF, Capacitor_SMD:C_0805_2012Metric, F.Cu at (318.9, 93.5)
- added C46: 100nF, Capacitor_SMD:C_0805_2012Metric, F.Cu at (318.9, 96.5)
- added C47: 100n, Capacitor_SMD:C_0805_2012Metric, F.Cu at (109.3, 104.4)
- added C48: 100nF, Capacitor_SMD:C_0805_2012Metric, F.Cu at (109.3, 107.4)
- added C49: 22uF, Capacitor_THT:CP_Radial_D5.0mm_P2.00mm, F.Cu at (83.2, 93.1)
- added C50: 22uF, Capacitor_THT:CP_Radial_D5.0mm_P2.00mm, F.Cu at (83.2, 99.6)
- added C51: 22uF, Capacitor_THT:CP_Radial_D5.0mm_P2.00mm, F.Cu at (91.8, 86.5)
- added C52: 22uF, Capacitor_THT:CP_Radial_D5.0mm_P2.00mm, F.Cu at (91.8, 93.1)
- added C53: 22uF, Capacitor_THT:CP_Radial_D5.0mm_P2.00mm, F.Cu at (91.8, 99.6)
- added C54: 100n, Capacitor_SMD:C_0805_2012Metric, F.Cu at (109.3, 110.4)
- added C55: 680p, Capacitor_SMD:C_0805_2012Metric, F.Cu at (318.9, 99.5)
- added C56: 680, Capacitor_SMD:C_0805_2012Metric, F.Cu at (318.9, 102.5)
- added C57: 680p, Capacitor_SMD:C_0805_2012Metric, F.Cu at (318.9, 105.5)
- added C58: 680, Capacitor_SMD:C_0805_2012Metric, F.Cu at (323.3, 90.5)
- added C59: 2.2n, Capacitor_SMD:C_0805_2012Metric, F.Cu at (323.3, 93.5)
- added C60: 2.2n, Capacitor_SMD:C_0805_2012Metric, F.Cu at (323.3, 96.5)
- added C61: 100n, Capacitor_SMD:C_0805_2012Metric, F.Cu at (109.3, 113.4)
- added C62: 100nF, Capacitor_SMD:C_0805_2012Metric, F.Cu at (109.3, 116.4)
- added C63: 100nF, Capacitor_SMD:C_0805_2012Metric, F.Cu at (109.3, 119.5)
- added C64: 100n, Capacitor_SMD:C_0805_2012Metric, F.Cu at (113.8, 104.4)
- added C65: 22uF, Capacitor_THT:CP_Radial_D5.0mm_P2.00mm, F.Cu at (98.4, 86.5)
- added C66: 22uF, Capacitor_THT:CP_Radial_D5.0mm_P2.00mm, F.Cu at (98.4, 93.1)
- added C67: 22uF, Capacitor_THT:CP_Radial_D5.0mm_P2.00mm, F.Cu at (98.4, 99.6)
- added C68: 22uF, Capacitor_THT:CP_Radial_D5.0mm_P2.00mm, F.Cu at (105.1, 86.5)
- added C69: 100nF, Capacitor_SMD:C_0805_2012Metric, F.Cu at (113.8, 107.4)
- added C70: 100nF, Capacitor_SMD:C_0805_2012Metric, F.Cu at (113.8, 110.4)
- added C71: 22uF, Capacitor_THT:CP_Radial_D5.0mm_P2.00mm, F.Cu at (105.1, 93.1)
- added C72: 22uF, Capacitor_THT:CP_Radial_D5.0mm_P2.00mm, F.Cu at (105.1, 99.6)
- added C73: 680p, Capacitor_SMD:C_0805_2012Metric, F.Cu at (113.8, 113.4)
- added C74: 680, Capacitor_SMD:C_0805_2012Metric, F.Cu at (113.8, 116.4)
- added C75: 680p, Capacitor_SMD:C_0805_2012Metric, F.Cu at (113.8, 119.5)
- added C76: 680, Capacitor_SMD:C_0805_2012Metric, F.Cu at (118.2, 104.4)
- added C77: 2.2n, Capacitor_SMD:C_0805_2012Metric, F.Cu at (118.2, 107.4)
- added C78: 2.2n, Capacitor_SMD:C_0805_2012Metric, F.Cu at (118.2, 110.4)
- added C79: 1n, Capacitor_SMD:C_0805_2012Metric, F.Cu at (307.8, 110.5)
- added C80: 1n, Capacitor_SMD:C_0805_2012Metric, F.Cu at (307.8, 113.5)
- added C81: 2.7n, Capacitor_SMD:C_0805_2012Metric, F.Cu at (307.8, 116.5)
- added C84: 100n, Capacitor_SMD:C_0805_2012Metric, F.Cu at (307.8, 119.5)
- added C85: 100nF, Capacitor_SMD:C_0805_2012Metric, F.Cu at (307.8, 122.6)
- added C86: 22uF, Capacitor_THT:CP_Radial_D5.0mm_P2.00mm, F.Cu at (296.9, 112.3)
- added C87: 22uF, Capacitor_THT:CP_Radial_D5.0mm_P2.00mm, F.Cu at (296.9, 118.8)
- added C88: 100nF, Capacitor_SMD:C_0805_2012Metric, F.Cu at (307.8, 125.6)
- added C89: 100nF, Capacitor_SMD:C_0805_2012Metric, F.Cu at (307.8, 128.6)
- added C90: 22uF, Capacitor_THT:CP_Radial_D5.0mm_P2.00mm, F.Cu at (296.9, 125.4)
- added C91: 22uF, Capacitor_THT:CP_Radial_D5.0mm_P2.00mm, F.Cu at (296.9, 131.9)
- added C94: 1n, Capacitor_SMD:C_0805_2012Metric, F.Cu at (392.4, 85.6)
- added C95: 1n, Capacitor_SMD:C_0805_2012Metric, F.Cu at (392.4, 88.6)
- added C96: 2.7n, Capacitor_SMD:C_0805_2012Metric, F.Cu at (392.4, 91.6)
- added C98: 100nF, Capacitor_SMD:C_0805_2012Metric, F.Cu at (396.8, 85.6)
- added C99: 100nF, Capacitor_SMD:C_0805_2012Metric, F.Cu at (396.8, 88.6)
- added H1: MountingHole_Pad, MountingHole:MountingHole_3.5mm_Pad_Via, F.Cu at (308.8, 25.7)
- added H2: MountingHole_Pad, MountingHole:MountingHole_3.5mm_Pad_Via, F.Cu at (308.8, 34.3)
- added H3: MountingHole_Pad, MountingHole:MountingHole_3.5mm_Pad_Via, F.Cu at (317.4, 25.7)
- added H4: MountingHole_Pad, MountingHole:MountingHole_3.5mm_Pad_Via, F.Cu at (317.4, 34.3)
- added H5: MountingHole_Pad, MountingHole:MountingHole_3.5mm_Pad_Via, F.Cu at (325.9, 25.7)
- added H6: MountingHole_Pad, MountingHole:MountingHole_3.5mm_Pad_Via, F.Cu at (325.9, 34.3)
- added H7: MountingHole_Pad, MountingHole:MountingHole_3.5mm_Pad_Via, F.Cu at (334.4, 25.7)
- added H8: MountingHole_Pad, MountingHole:MountingHole_3.5mm_Pad_Via, F.Cu at (334.4, 34.3)
- added J10: GPIO 0, Connector_PinHeader_2.54mm:PinHeader_2x20_P2.54mm_Vertical, F.Cu at (369.4, 71.6)
- added J11: GPIO 1, Connector_PinHeader_2.54mm:PinHeader_2x20_P2.54mm_Vertical, F.Cu at (376.6, 71.6)
- added J6: Conn_01x03, Connector_JST:JST_PH_B3B-PH-K_1x03_P2.00mm_Vertical, F.Cu at (297.6, 43.8)
- added J7: Conn_01x03, Connector_JST:JST_PH_B3B-PH-K_1x03_P2.00mm_Vertical, F.Cu at (297.6, 50.4)
- added J8: Conn_01x03, Connector_JST:JST_PH_B3B-PH-K_1x03_P2.00mm_Vertical, F.Cu at (297.6, 56.9)
- added J9: Conn_01x03, Connector_JST:JST_PH_B3B-PH-K_1x03_P2.00mm_Vertical, F.Cu at (297.6, 63.5)
- added R1: 22R, Resistor_SMD:R_0805_2012Metric, F.Cu at (342.9, 22.9)
- added R100: 10, Resistor_SMD:R_0805_2012Metric, F.Cu at (303.4, 128.2)
- added R101: 10, Resistor_SMD:R_0805_2012Metric, F.Cu at (303.4, 131.1)
- added R106: 1k, Resistor_SMD:R_0805_2012Metric, F.Cu at (392.4, 70.8)
- added R107: 270, Resistor_SMD:R_0805_2012Metric, F.Cu at (392.4, 73.7)
- added R110: 39, Resistor_SMD:R_0805_2012Metric, F.Cu at (392.4, 76.7)
- added R111: 39, Resistor_SMD:R_0805_2012Metric, F.Cu at (392.4, 79.6)
- added R119: 10, Resistor_SMD:R_0805_2012Metric, F.Cu at (392.4, 82.6)
- added R120: 10, Resistor_SMD:R_0805_2012Metric, F.Cu at (396.8, 70.8)
- added R121: 10, Resistor_SMD:R_0805_2012Metric, F.Cu at (396.8, 73.7)
- added R122: 10, Resistor_SMD:R_0805_2012Metric, F.Cu at (396.8, 76.7)
- added R123: 10, Resistor_SMD:R_0805_2012Metric, F.Cu at (396.8, 79.6)
- added R124: 10, Resistor_SMD:R_0805_2012Metric, F.Cu at (396.8, 82.6)
- added R18: 10K, Resistor_SMD:R_0805_2012Metric, F.Cu at (351.8, 25.9)
- added R19: 10K, Resistor_SMD:R_0805_2012Metric, F.Cu at (351.8, 28.8)
- added R20: 1k, Resistor_SMD:R_0805_2012Metric, F.Cu at (351.8, 31.8)
- added R21: 1k, Resistor_SMD:R_0805_2012Metric, F.Cu at (351.8, 34.7)
- added R22: 4.7k, Resistor_SMD:R_0805_2012Metric, F.Cu at (351.8, 37.7)
- added R23: 4.7k, Resistor_SMD:R_0805_2012Metric, F.Cu at (351.8, 40.6)
- added R24: 10, Resistor_SMD:R_0805_2012Metric, F.Cu at (351.8, 43.6)
- added R25: 820, Resistor_SMD:R_0805_2012Metric, F.Cu at (356.2, 22.9)
- added R26: 820, Resistor_SMD:R_0805_2012Metric, F.Cu at (356.2, 25.9)
- added R27: 4.3K, Resistor_SMD:R_0805_2012Metric, F.Cu at (356.2, 28.8)
- added R28: 4.3k, Resistor_SMD:R_0805_2012Metric, F.Cu at (356.2, 31.8)
- added R29: 22, Resistor_SMD:R_0805_2012Metric, F.Cu at (356.2, 34.7)
- added R30: 39, Resistor_SMD:R_0805_2012Metric, F.Cu at (356.2, 37.7)
- added R39: 10, Resistor_SMD:R_0805_2012Metric, F.Cu at (296.8, 70.8)
- added R40: 10, Resistor_SMD:R_0805_2012Metric, F.Cu at (296.8, 73.7)
- added R41: 22R, Resistor_SMD:R_0805_2012Metric, F.Cu at (296.8, 76.7)
- added R42: 22R, Resistor_SMD:R_0805_2012Metric, F.Cu at (296.8, 79.6)
- added R43: 22R, Resistor_SMD:R_0805_2012Metric, F.Cu at (296.8, 82.6)
- added R44: 22R, Resistor_SMD:R_0805_2012Metric, F.Cu at (296.8, 85.5)
- added R45: 10, Resistor_SMD:R_0805_2012Metric, F.Cu at (296.8, 88.5)
- added R46: 10, Resistor_SMD:R_0805_2012Metric, F.Cu at (301.2, 70.8)
- added R47: 10, Resistor_SMD:R_0805_2012Metric, F.Cu at (301.2, 73.7)
- added R48: 10, Resistor_SMD:R_0805_2012Metric, F.Cu at (301.2, 76.7)
- added R49: 10, Resistor_SMD:R_0805_2012Metric, F.Cu at (301.2, 79.6)
- added R50: 10, Resistor_SMD:R_0805_2012Metric, F.Cu at (301.2, 82.6)
- added R51: 22R, Resistor_SMD:R_0805_2012Metric, F.Cu at (91.6, 104.4)
- added R52: 22R, Resistor_SMD:R_0805_2012Metric, F.Cu at (91.6, 107.3)
- added R53: 1k, Resistor_SMD:R_0805_2012Metric, F.Cu at (301.2, 85.5)
- added R54: 1k, Resistor_SMD:R_0805_2012Metric, F.Cu at (301.2, 88.5)
- added R55: 10, Resistor_SMD:R_0805_2012Metric, F.Cu at (91.6, 110.3)
- added R56: 10, Resistor_SMD:R_0805_2012Metric, F.Cu at (91.6, 113.2)
- added R57: 1k, Resistor_SMD:R_0805_2012Metric, F.Cu at (305.6, 70.8)
- added R58: 1k, Resistor_SMD:R_0805_2012Metric, F.Cu at (305.6, 73.7)
- added R59: 4.7k, Resistor_SMD:R_0805_2012Metric, F.Cu at (305.6, 76.7)
- added R60: 4.7k, Resistor_SMD:R_0805_2012Metric, F.Cu at (305.6, 79.6)
- added R61: 4.7k, Resistor_SMD:R_0805_2012Metric, F.Cu at (305.6, 82.6)
- added R62: 4.7k, Resistor_SMD:R_0805_2012Metric, F.Cu at (305.6, 85.5)
- added R63: 22R, Resistor_SMD:R_0805_2012Metric, F.Cu at (91.6, 116.2)
- added R64: 22R, Resistor_SMD:R_0805_2012Metric, F.Cu at (91.6, 119.1)
- added R65: 10, Resistor_SMD:R_0805_2012Metric, F.Cu at (91.6, 122.1)
- added R66: 10, Resistor_SMD:R_0805_2012Metric, F.Cu at (96.1, 104.4)
- added R67: 10, Resistor_SMD:R_0805_2012Metric, F.Cu at (96.1, 107.3)
- added R68: 10, Resistor_SMD:R_0805_2012Metric, F.Cu at (96.1, 110.3)
- added R69: 10, Resistor_SMD:R_0805_2012Metric, F.Cu at (96.1, 113.2)
- added R70: 10, Resistor_SMD:R_0805_2012Metric, F.Cu at (96.1, 116.2)
- added R71: 1k, Resistor_SMD:R_0805_2012Metric, F.Cu at (96.1, 119.1)
- added R72: 1k, Resistor_SMD:R_0805_2012Metric, F.Cu at (96.1, 122.1)
- added R73: 39, Resistor_SMD:R_0805_2012Metric, F.Cu at (305.6, 88.5)
- added R74: 39, Resistor_SMD:R_0805_2012Metric, F.Cu at (310.0, 70.8)
- added R75: 39, Resistor_SMD:R_0805_2012Metric, F.Cu at (310.0, 73.7)
- added R76: 39, Resistor_SMD:R_0805_2012Metric, F.Cu at (310.0, 76.7)
- added R77: 1k, Resistor_SMD:R_0805_2012Metric, F.Cu at (100.5, 104.4)
- added R78: 1k, Resistor_SMD:R_0805_2012Metric, F.Cu at (100.5, 107.3)
- added R79: 4.7k, Resistor_SMD:R_0805_2012Metric, F.Cu at (100.5, 110.3)
- added R80: 4.7k, Resistor_SMD:R_0805_2012Metric, F.Cu at (100.5, 113.2)
- added R81: 4.7k, Resistor_SMD:R_0805_2012Metric, F.Cu at (100.5, 116.2)
- added R82: 4.7k, Resistor_SMD:R_0805_2012Metric, F.Cu at (100.5, 119.1)
- added R83: 39, Resistor_SMD:R_0805_2012Metric, F.Cu at (100.5, 122.1)
- added R84: 39, Resistor_SMD:R_0805_2012Metric, F.Cu at (104.9, 104.4)
- added R85: 39, Resistor_SMD:R_0805_2012Metric, F.Cu at (104.9, 107.3)
- added R86: 39, Resistor_SMD:R_0805_2012Metric, F.Cu at (104.9, 110.3)
- added R87: 1k, Resistor_SMD:R_0805_2012Metric, F.Cu at (303.4, 110.5)
- added R88: 10, Resistor_SMD:R_0805_2012Metric, F.Cu at (303.4, 113.4)
- added R89: 2.7k, Resistor_SMD:R_0805_2012Metric, F.Cu at (303.4, 116.4)
- added R90: 10, Resistor_SMD:R_0805_2012Metric, F.Cu at (303.4, 119.3)
- added R91: 39, Resistor_SMD:R_0805_2012Metric, F.Cu at (303.4, 122.3)
- added R92: 39, Resistor_SMD:R_0805_2012Metric, F.Cu at (303.4, 125.2)
- added U1: PCM1789-Q1, Package_SO:TSSOP-24_4.4x7.8mm_P0.65mm, F.Cu at (345.1, 49.7)
- added U11: PCM1789-Q1, Package_SO:TSSOP-24_4.4x7.8mm_P0.65mm, F.Cu at (113.7, 87.9)
- added U18: 12V, Audio-DSP:BUCK_MAX17634C, F.Cu at (394.2, 25.0)
- added U19: 5V, Audio-DSP:BUCK_MAX17634C, F.Cu at (394.2, 32.0)
- added U2: LM4562, Package_SO:SOIC-8_3.9x4.9mm_P1.27mm, F.Cu at (344.9, 57.6)
- added U20: 8V, Audio-DSP:BUCK_MAX17634C, F.Cu at (394.2, 39.1)
- added U21: 15V, Audio-DSP:BUCK_MAX17634C, F.Cu at (394.2, 46.1)
- added U7: PCM1789-Q1, Package_SO:TSSOP-24_4.4x7.8mm_P0.65mm, F.Cu at (298.9, 94.6)
- added U9: LM4562, Package_SO:SOIC-8_3.9x4.9mm_P1.27mm, F.Cu at (113.6, 95.8)
- C13: value 5.6n -> 1n5
- C14, C8: value 2.2n -> 1n5
- C16, C26: value 22uF -> 100nF; footprint Capacitor_THT:CP_Radial_D5.0mm_P2.00mm -> Capacitor_SMD:C_0805_2012Metric
- C17: value 1N -> 680p
- C18: value 680p -> 680
- C19, C2, C3: value 100nF -> 100n
- C23, C28: value 100nF -> 22uF; footprint Capacitor_SMD:C_0805_2012Metric -> Capacitor_THT:CP_Radial_D5.0mm_P2.00mm
- C27: value 680 -> 2.2n
- C29: value 2.2n -> 100n
- C6: value 100nF -> 4n7
- C7: value 5.6n -> 4n7
- C9: value 1N -> 1n5
- moved R17 344.2 mm to (351.8, 22.9)
- moved R10 344.0 mm to (347.3, 25.9)
- moved R11 344.0 mm to (347.3, 28.8)
- moved R12 344.0 mm to (347.3, 31.8)
- moved R9 344.0 mm to (347.3, 22.9)
- moved R2 343.9 mm to (342.9, 25.9)
- moved R3 343.9 mm to (342.9, 28.8)
- moved R4 343.9 mm to (342.9, 31.8)
- moved R5 343.9 mm to (342.9, 34.7)
- moved R6 343.9 mm to (342.9, 37.7)
- moved R7 339.7 mm to (342.9, 40.6)
- moved R8 339.7 mm to (342.9, 43.6)
- moved R13 339.5 mm to (347.3, 34.7)
- moved R14 339.5 mm to (347.3, 37.7)
- moved R15 339.5 mm to (347.3, 40.6)
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Connections:
- net /DAC CH1_2/BCK renamed /DAC_CH1_2/BCK
- net /DAC CH1_2/DIN renamed /DAC_CH1_2/DIN
- net /DAC CH1_2/RCA JACK CH1 renamed /DAC_CH1_2/RCA JACK CH1
- net /DAC CH1_2/SCKI renamed /DAC_CH1_2/SCKI
- C12 pad 1: /DAC CH1_2/VOUT CH1(-) -> /DAC_CH1_2/VOUT CH1(-)
- C12 pad 2: /DAC CH1_2/VOUT CH1(+) -> /DAC_CH1_2/VOUT CH1(+)
- C15 pad 1: GND -> Net-(U3B-V+)
- C15 pad 2: Net-(C15-Pad2) -> GND
- C16 pad 2: Net-(C15-Pad2) -> Net-(U3B-V-)
- C18 pad 2: Net-(IC3-VOUT-) -> Net-(U4A-VOUT+)
- C23 pad 1: Net-(C23-Pad1) -> Net-(U3B-V+)
- C24 pad 1: Net-(C23-Pad1) -> GND
- C24 pad 2: GND -> Net-(U3B-V-)
- C25 pad 1: GND -> Net-(U4B-V+)
- C25 pad 2: Net-(C25-Pad2) -> GND
- C26 pad 2: Net-(C25-Pad2) -> Net-(U4B-V-)
- C27 pad 1: Net-(IC3-VIN-) -> /DAC_CH1_2/VOUT CH2(-)
- C27 pad 2: Net-(IC3-VOUT+) -> /DAC_CH1_2/VOUT CH2(+)
- C28 pad 1: Net-(C28-Pad1) -> Net-(U4B-V+)
- C29 pad 1: /DAC CH1_2/VOUT CH1(-) -> Net-(C29-Pad1)
- C29 pad 2: /DAC CH1_2/VOUT CH1(+) -> GND
- C30 pad 1: Net-(C28-Pad1) -> GND
- C30 pad 2: GND -> Net-(U4B-V-)
- C4 pad 1: Net-(U1C-V+) -> Net-(U2C-V+)
- C6 pad 1: Net-(U1C-V+) -> Net-(C6-Pad1)
- C6 pad 2: GND -> Net-(C6-Pad2)
- J2 pad 1: /DAC CH1_2/VOUT CH1(+) -> /DAC_CH1_2/VOUT CH1(+)
- J2 pad 3: /DAC CH1_2/VOUT CH1(-) -> /DAC_CH1_2/VOUT CH1(-)
- J4 pad 1: /VOUT CH2(-) -> /DAC_CH1_2/VOUT CH2(-)
- J4 pad 3: /VOUT CH2(+) -> /DAC_CH1_2/VOUT CH2(+)
- R13 pad 2: /DAC CH1_2/VOUT CH1(-) -> /DAC_CH1_2/VOUT CH1(-)
- R14 pad 2: /DAC CH1_2/VOUT CH1(-) -> /DAC_CH1_2/VOUT CH1(-)
- R15 pad 2: /DAC CH1_2/VOUT CH1(+) -> /DAC_CH1_2/VOUT CH1(+)
- R17 pad 2: /DAC CH1_2/VOUT CH1(+) -> /DAC_CH1_2/VOUT CH1(+)
- R32 pad 1: Net-(U1C-V+) -> Net-(U2C-V+)
- R35 pad 1: Net-(C23-Pad1) -> -12V
- R35 pad 2: +12V -> Net-(U3B-V-)
- R36 pad 1: -12V -> Net-(U4B-V+)
- R36 pad 2: Net-(C25-Pad2) -> +12V
- R37 pad 1: Net-(IC3-VOUT+) -> Net-(U4A-VOUT+)
- R37 pad 2: /DAC CH1_2/VOUT CH1(+) -> /DAC_CH1_2/VOUT CH2(+)
- R38 pad 1: Net-(C28-Pad1) -> -12V
- R38 pad 2: +12V -> Net-(U4B-V-)
Other:
- board outline added: 100 x 150 mm
- board text added: "Update stackup and constrain manager"

Commit message: Worked on main board
Parts:
- moved H3 341.9 mm to (55.0, 245.0)
- moved J10 329.3 mm to (57.5, 177.1)
- moved J11 324.6 mm to (69.7, 177.1)
- moved U19 313.6 mm to (145.0, 222.5), turned to -90 degrees
- moved U20 297.5 mm to (160.0, 222.5), turned to -90 degrees
- moved U18 295.0 mm to (175.0, 222.5), turned to -90 degrees
- moved U21 269.8 mm to (190.0, 222.4), turned to -90 degrees
- moved H1 253.9 mm to (56.9, 56.9)
- moved H4 243.7 mm to (195.0, 245.0)
- moved U11 208.6 mm to (321.7, 104.8)
- moved C44 208.6 mm to (291.1, 103.5)
- moved C47 208.6 mm to (317.2, 121.3)
- moved C48 208.6 mm to (317.2, 124.3)
- moved C49 208.6 mm to (291.1, 110.0)
- moved C50 208.6 mm to (291.1, 116.5)
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Connections:
- net /VOUT CH1(+) renamed /VOUT CH1(+)_1
- net /VOUT CH1(-) renamed /VOUT CH1(-)_1
Other:
- board size 100 x 150 mm -> 150 x 200 mm

Commit message: Worked a bit on the main board
Parts:
- removed R4, R41, R42, R43, R44, R51, R52, R63, R64: 22R, Resistor_SMD:R_0805_2012Metric
- added J12: Conn_01x03, Connector_JST:JST_PH_B3B-PH-K_1x03_P2.00mm_Vertical, F.Cu at (158.0, 57.0)
- added J13: Conn_01x02, Connector_JST:JST_PH_B2B-PH-K_1x02_P2.00mm_Vertical, F.Cu at (187.0, 56.0)
- added J14: Conn_01x02, Connector_JST:JST_PH_B2B-PH-K_1x02_P2.00mm_Vertical, F.Cu at (181.0, 56.0)
- added NT1: NetTie_2, NetTie:NetTie-2_SMD_Pad0.5mm, F.Cu at (266.5, 79.2)
- added NT2: NetTie_2, NetTie:NetTie-2_SMD_Pad0.5mm, F.Cu at (266.5, 81.2)
- added R200: 22R, Resistor_SMD:R_Array_Convex_2x0402, F.Cu at (96.0, 145.0)
- added U23: LIN_REG_±5V, Audio_DSP:LIN_REG_±xxV, F.Cu at (149.0, 76.3)
- added U24: LIN_REG_±12V, Audio_DSP:LIN_REG_±xxV, F.Cu at (131.0, 76.3)
- added U25: LIN_REG_±5V, Audio_DSP:LIN_REG_±xxV, F.Cu at (122.0, 96.3)
- added U26: LIN_REG_±12V, Audio_DSP:LIN_REG_±xxV, F.Cu at (140.0, 95.3)
- added U27: PCM1804, Package_SO:SSOP-28_5.3x10.2mm_P0.65mm, F.Cu at (184.4, 68.0)
- added U28: PCM1804, Package_SO:SSOP-28_5.3x10.2mm_P0.65mm, F.Cu at (162.0, 68.0)
- C15, C16, C19, C2, C25, C26, C3: footprint Capacitor_SMD:C_0805_2012Metric -> Capacitor_SMD:C_0402_1005Metric
- C21, C35: footprint Capacitor_SMD:C_0805_2012Metric -> Capacitor_SMD:C_0402_1005Metric; moved to B.Cu
- R1, R2, R3: footprint Resistor_SMD:R_0805_2012Metric -> Resistor_SMD:R_Array_Convex_4x0402
- U1, U11, U7: value PCM1789-Q1 -> PCM1789
- moved U11 260.8 mm to (61.0, 96.0), turned to 180 degrees
- moved H7 243.2 mm to (80.0, 165.0)
- moved R2 242.8 mm to (80.0, 145.0), turned to -90 degrees
- moved H8 242.5 mm to (135.0, 245.0)
- moved C3 235.0 mm to (96.0, 93.0), turned to 90 degrees
- moved R1 234.6 mm to (90.0, 145.0), turned to -90 degrees
- moved C21 234.6 mm to (103.0, 74.0), turned to -90 degrees
- moved C35 234.2 mm to (103.0, 70.0), turned to -90 degrees
- moved C22 230.7 mm to (105.0, 66.0)
- moved C19 230.3 mm to (110.0, 95.0), turned to 90 degrees
- moved C4 228.0 mm to (101.0, 66.0), turned to 180 degrees
- moved R3 224.1 mm to (99.0, 145.0), turned to 90 degrees
- moved R29 223.5 mm to (96.0, 61.0), turned to 90 degrees
- moved C2 221.4 mm to (110.0, 91.0), turned to 90 degrees
- moved U1 206.9 mm to (102.0, 95.7), turned to 180 degrees
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Connections:
- net /DAC_CH1_2/AMUTEI renamed /DAC_CH1_2/AMUTEI_CH1_2
- net /DAC_CH1_2/DIN renamed /DAC_CH1_2/LRCK_CH1_2
- net /DAC_CH1_2/RCA JACK CH1 renamed /DAC_CH1_2/RCA_JACK_CH1(+)
- net /DAC_CH1_2/RST renamed /DAC_CH1_2/RST_CH1_2
- net /DAC_CH1_2/VOUT CH1(+) renamed /DAC_CH1_2/VOUT_CH1(+)
- net /DAC_CH1_2/VOUT CH1(-) renamed /DAC_CH1_2/VOUT_CH1(-)
- net /VOUT CH1(+)_1 renamed /VOUT CH1(+)
- net /VOUT CH1(-)_1 renamed /VOUT CH1(-)
- net /VOUT CH2(+)_1 renamed /VOUT CH2(+)
- net /VOUT CH2(-)_1 renamed /VOUT CH2(-)
- C14 pad 2: GND -> /DAC_CH1_2/RCA_JACK_CH2(REF)
- C27 pad 1: /DAC_CH1_2/VOUT CH2(-) -> /DAC_CH1_2/VOUT_CH2(-)
- C27 pad 2: /DAC_CH1_2/VOUT CH2(+) -> /DAC_CH1_2/VOUT_CH2(+)
- C8 pad 2: GND -> /DAC_CH1_2/RCA_JACK_CH1(REF)
- H1 pad 1: unconnected-(H1-Pad1) -> GND
- H2 pad 1: unconnected-(H2-Pad1) -> GND
- H3 pad 1: unconnected-(H3-Pad1) -> GND
- H4 pad 1: unconnected-(H4-Pad1) -> GND
- H5 pad 1: unconnected-(H5-Pad1) -> GND
- H6 pad 1: unconnected-(H6-Pad1) -> GND
- H7 pad 1: unconnected-(H7-Pad1) -> GND
- H8 pad 1: unconnected-(H8-Pad1) -> GND
- J3 pad 2: GND -> /DAC_CH1_2/RCA_JACK_CH1(REF)
- J4 pad 1: /DAC_CH1_2/VOUT CH2(-) -> /DAC_CH1_2/VOUT_CH2(+)
- J4 pad 3: /DAC_CH1_2/VOUT CH2(+) -> /DAC_CH1_2/VOUT_CH2(-)
- J5 pad 1: /RCA/JACK CH2 -> /DAC_CH1_2/RCA_JACK_CH2(+)
- J5 pad 2: GND -> /DAC_CH1_2/RCA_JACK_CH2(REF)
- R1 pad 1: /DAC_CH1_2/LRCK -> Net-(R1-R1.1)
- R1 pad 2: Net-(U1-LRCK) -> Net-(R1-R2.1)
- R2 pad 1: /DAC_CH1_2/BCK -> Net-(R2-R1.1)
- R2 pad 2: Net-(U1-BCK) -> Net-(R2-R2.1)
- R22 pad 2: /DAC_CH1_2/VOUT CH2(-) -> /DAC_CH1_2/VOUT_CH2(-)
- R23 pad 2: /DAC_CH1_2/VOUT CH2(+) -> /DAC_CH1_2/VOUT_CH2(+)
- R28 pad 2: GND -> /DAC_CH1_2/RCA_JACK_CH2(REF)
- R29 pad 2: /DAC_CH1_2/RCA JACK CH2 -> /DAC_CH1_2/RCA_JACK_CH2(+)
- R3 pad 2: Net-(U1-DIN) -> /DAC_CH1_2/BCK_CH1_2
- R30 pad 2: /DAC_CH1_2/VOUT CH2(-) -> /DAC_CH1_2/VOUT_CH2(-)
- R37 pad 2: /DAC_CH1_2/VOUT CH2(+) -> /DAC_CH1_2/VOUT_CH2(+)
- R9 pad 2: GND -> /DAC_CH1_2/RCA_JACK_CH1(REF)
- U1 pad 1: Net-(U1-LRCK) -> Net-(R3-R1.2)
- U1 pad 2: Net-(U1-BCK) -> Net-(R3-R2.2)
- U1 pad 20: /DAC_CH1_2/MODE -> GND
- U1 pad 21: /DAC_CH1_2/MD/SDA/DEMP -> Net-(R200-R1.2)
- U1 pad 22: /DAC_CH1_2/MC/SCL/FMT -> Net-(R200-R2.2)
- U1 pad 3: Net-(U1-DIN) -> Net-(R3-R3.2)
- U1 pad 5: Net-(U1-SCKI) -> Net-(R3-R4.2)
- U11 pad 1: Net-(U11-LRCK) -> Net-(R2-R4.1)
- U11 pad 2: Net-(U11-BCK) -> Net-(R2-R3.1)
- U11 pad 20: /DAC_CH5_6/MODE -> /DAC_CH5_6/MC/SCL/FMT
- U11 pad 21: /DAC_CH5_6/MD/SDA/DEMP -> /DAC_CH5_6/MODE
- U11 pad 22: /DAC_CH5_6/MC/SCL/FMT -> /DAC_CH5_6/MD/SDA/DEMP
- U11 pad 3: Net-(U11-DIN) -> Net-(R2-R2.1)
- U11 pad 5: Net-(U11-SCKI) -> Net-(R2-R1.1)
- U7 pad 1: Net-(U7-LRCK) -> Net-(R1-R4.1)
- U7 pad 2: Net-(U7-BCK) -> Net-(R1-R3.1)
- U7 pad 20: /DAC_CH3_4/MODE -> /DAC_CH3_4/MC/SCL/FMT
- U7 pad 21: /DAC_CH3_4/MD/SDA/DEMP -> /DAC_CH3_4/MODE
- U7 pad 22: /DAC_CH3_4/MC/SCL/FMT -> /DAC_CH3_4/MD/SDA/DEMP
- U7 pad 3: Net-(U7-DIN) -> Net-(R1-R2.1)
- U7 pad 5: Net-(U7-SCKI) -> Net-(R1-R1.1)
Routing:
- added copper zone on F.Cu, net GND
Other:
- board text added: "+12V"
- board text added: "+15V"
- board text added: "+5V"
- board text added: "+8V"
- board text added: "GPIO 0"
- board text added: "GPIO 1"

Commit message: Worked on main board
Parts:
- U18, U19, U20, U21: footprint Audio-DSP:BUCK_MAX17634C -> Audio-DSP:BUCK_MAX17634C_xxV
- moved C18 60.2 mm to (290.3, 106.6)
- moved C12 57.2 mm to (285.8, 106.6)
- moved C11 57.2 mm to (285.8, 103.5)
- moved C13 57.2 mm to (285.8, 109.6)
- moved C42 49.8 mm to (292.5, 40.5)
- moved C55 49.8 mm to (292.5, 49.6)
- moved C44 49.8 mm to (281.5, 42.3)
- moved C45 49.8 mm to (292.5, 43.5)
- moved C46 49.8 mm to (292.5, 46.6)
- moved C49 49.8 mm to (281.5, 48.9)
- moved C50 49.8 mm to (281.5, 55.4)
- moved C56 49.8 mm to (292.5, 52.6)
- moved C57 49.8 mm to (292.5, 55.6)
- moved R39 49.8 mm to (268.1, 60.2)
- moved R40 49.8 mm to (268.1, 63.1)
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