File: KiCAD/Main board/Main board.kicad_pcb (KiCad board)
At the start: 2 copper layers, 150 x 200 mm, 239 parts, among them J1 Conn_01x03, J10 GPIO 0, J11 GPIO 1, J12 Conn_01x03, J13 Conn_01x02, J14 Conn_01x02, J2 Conn_01x03, J3 Conn_01x02, J4 Conn_01x03, J5 Conn_01x02, J6 Conn_01x03, J7 Conn_01x03, J8 Conn_01x03, J9 Conn_01x03, U1 PCM1789, U11 PCM1789, U18 12V, U19 5V, U2 LM4562, U20 8V, U21 15V, U23 LIN_REG_±5V, U24 LIN_REG_±12V, U25 LIN_REG_±5V, U26 LIN_REG_±12V, U27 PCM1804, U28 PCM1804, U7 PCM1789, U9 LM4562

Commit message: fixed 3D viewer
Parts:
- U23, U24, U25, U26: footprint Audio_DSP:LIN_REG_±xxV -> Audio DSP:LIN_REG_±xxV
Changed lines of the file:
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@@
     )
   )
-  (footprint "Audio_DSP:LIN_REG_±xxV" (layer "F.Cu")
+  (footprint "Audio DSP:LIN_REG_±xxV" (layer "F.Cu")
     (at 131 76.35 90)
     (property "Sheetfile" "POWER_SUPPLIES.kicad_sch")
@@
     (pad "6" thru_hole oval (at -6.35 0) (size 1.7 1.7) (drill 1) (layers "*.Cu" "*.Mask")
       (net 266 "unconnected-(U24--15V-Pad6)") (pinfunction "-15V") (pintype "power_in"))
-    (model "C:/Users/PC/OneDrive/Documenten/School/Fontys/Minor/Be creative minor/Git/Audio-DSP/KiCAD/Discrete_linear_regulator/Discrete_linear_regulator.step"
+    (model "${CUSTOM_3D_MODELS}/Discrete_linear_regulator.step"
       (offset (xyz -75 3 80.1))
       (scale (xyz 1 1 1))
@@
       (net 2 "GND") (pinfunction "1") (pintype "input"))
   )
-  (footprint "Audio_DSP:LIN_REG_±xxV" (layer "F.Cu")
+  (footprint "Audio DSP:LIN_REG_±xxV" (layer "F.Cu")
     (at 140 95.35 90)
     (property "Sheetfile" "POWER_SUPPLIES.kicad_sch")
@@
     (pad "6" thru_hole oval (at -6.35 0) (size 1.7 1.7) (drill 1) (layers "*.Cu" "*.Mask")
       (net 274 "unconnected-(U26--15V-Pad6)") (pinfunction "-15V") (pintype "power_in"))
-    (model "C:/Users/PC/OneDrive/Documenten/School/Fontys/Minor/Be creative minor/Git/Audio-DSP/KiCAD/Discrete_linear_regulator/Discrete_linear_regulator.step"
+    (model "${CUSTOM_3D_MODELS}/Discrete_linear_regulator.step"
       (offset (xyz -75 3 80.1))
       (scale (xyz 1 1 1))
@@
     )
   )
-  (footprint "Audio_DSP:LIN_REG_±xxV" (layer "F.Cu")
+  (footprint "Audio DSP:LIN_REG_±xxV" (layer "F.Cu")
     (at 122 96.35 90)
     (property "Sheetfile" "POWER_SUPPLIES.kicad_sch")
@@
     (pad "6" thru_hole oval (at -6.35 0) (size 1.7 1.7) (drill 1) (layers "*.Cu" "*.Mask")
       (net 267 "unconnected-(U25--8V-Pad6)") (pinfunction "-8V") (pintype "power_in"))
-    (model "C:/Users/PC/OneDrive/Documenten/School/Fontys/Minor/Be creative minor/Git/Audio-DSP/KiCAD/Discrete_linear_regulator/Discrete_linear_regulator.step"
+    (model "${CUSTOM_3D_MODELS}/Discrete_linear_regulator.step"
       (offset (xyz -75 3 80.1))
       (scale (xyz 1 1 1))
@@
     )
   )
-  (footprint "Audio_DSP:LIN_REG_±xxV" (layer "F.Cu")
+  (footprint "Audio DSP:LIN_REG_±xxV" (layer "F.Cu")
     (at 149 76.35 90)
     (property "Sheetfile" "POWER_SUPPLIES.kicad_sch")
@@
         (effects (font (size 1 1) (thickness 0.15)))
     )
-    (fp_text user "${REFERENCE}" (at 0 0 90) (layer "F.Fab")
+    (fp_text user "${REFERENCE}" (at 0 -4 90 unlocked) (layer "F.Fab")
         (effects (font (size 1 1) (thickness 0.15)))
     )
-    (fp_text user "${REFERENCE}" (at 0 -4 90 unlocked) (layer "F.Fab")
+    (fp_text user "${REFERENCE}" (at 0 0 90) (layer "F.Fab")
         (effects (font (size 1 1) (thickness 0.15)))
     )
@@
     (pad "6" thru_hole oval (at -6.35 0) (size 1.7 1.7) (drill 1) (layers "*.Cu" "*.Mask")
       (net 263 "unconnected-(U23--8V-Pad6)") (pinfunction "-8V") (pintype "power_in"))
-    (model "C:/Users/PC/OneDrive/Documenten/School/Fontys/Minor/Be creative minor/Git/Audio-DSP/KiCAD/Discrete_linear_regulator/Discrete_linear_regulator.step"
+    (model "${CUSTOM_3D_MODELS}/Discrete_linear_regulator.step"
       (offset (xyz -75 3 80.1))
       (scale (xyz 1 1 1))
