File: KiCAD/Main board/Main board.kicad_pcb (KiCad board)
At the start: 2 copper layers, 150 x 200 mm, 239 parts, among them J1 Conn_01x03, J10 GPIO 0, J11 GPIO 1, J12 Conn_01x03, J13 Conn_01x02, J14 Conn_01x02, J2 Conn_01x03, J3 Conn_01x02, J4 Conn_01x03, J5 Conn_01x02, J6 Conn_01x03, J7 Conn_01x03, J8 Conn_01x03, J9 Conn_01x03, U1 PCM1789, U11 PCM1789, U18 12V, U19 5V, U2 LM4562, U20 8V, U21 15V, U23 LIN_REG_±5V, U24 LIN_REG_±12V, U25 LIN_REG_±5V, U26 LIN_REG_±12V, U27 PCM1804, U28 PCM1804, U7 PCM1789, U9 LM4562

Commit message: Updated main step
Parts:
- moved C19 30.0 mm to (110.0, 125.0)
- moved C2 30.0 mm to (110.0, 121.0)
- moved C21 30.0 mm to (103.0, 104.0)
- moved C22 30.0 mm to (105.0, 96.0)
- moved C3 30.0 mm to (96.0, 123.0)
- moved C35 30.0 mm to (103.0, 100.0)
- moved C4 30.0 mm to (101.0, 96.0)
- moved H1 30.0 mm to (56.9, 86.9)
- moved H2 30.0 mm to (195.0, 85.0)
- moved H5 30.0 mm to (140.0, 85.0)
- moved H6 30.0 mm to (195.0, 165.0)
- moved J1 30.0 mm to (165.0, 87.0)
- moved J12 30.0 mm to (158.0, 87.0)
- moved J13 30.0 mm to (187.0, 86.0)
- moved J14 30.0 mm to (181.0, 86.0)
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Other:
- board size 150 x 200 mm -> 150 x 170 mm

Commit message: Updated main board
Parts:
- moved H4 47.2 mm to (235.0, 220.0)
- moved H2 44.7 mm to (235.0, 105.0)
- moved H6 40.0 mm to (235.0, 165.0)
- moved J1 38.6 mm to (198.0, 107.0)
- moved J12 38.6 mm to (191.0, 107.0)
- moved J13 38.6 mm to (220.0, 106.0)
- moved J14 38.6 mm to (214.0, 106.0)
- moved U27 38.6 mm to (217.4, 118.0)
- moved U28 38.6 mm to (195.0, 118.0)
- moved C19 32.0 mm to (135.0, 145.0)
- moved C2 32.0 mm to (135.0, 141.0)
- moved C3 32.0 mm to (121.0, 143.0)
- moved H5 32.0 mm to (165.0, 105.0)
- moved U1 32.0 mm to (127.0, 145.7)
- moved U11 32.0 mm to (86.0, 146.0)
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Other:
- board size 150 x 170 mm -> 190 x 125 mm

Commit message: Worked on main board
Parts:
- removed C29, C36, C39, C42, C47, C54, C61, C64: 100n, Capacitor_SMD:C_0805_2012Metric
- removed C31, C37, C38, C45, C46, C48, C62, C63, C69, C70: 100nF, Capacitor_SMD:C_0805_2012Metric
- removed C32, C33, C34, C40, C41, C43, C44, C49, C50, C51, C52, C53, C65, C66, C67, C68, C71, C72: 22uF, Capacitor_THT:CP_Radial_D5.0mm_P2.00mm
- removed C35: 100n, Capacitor_SMD:C_0402_1005Metric
- removed C55, C57, C73, C75: 680p, Capacitor_SMD:C_0805_2012Metric
- removed C56, C58, C74, C76: 680, Capacitor_SMD:C_0805_2012Metric
- removed C59, C60, C77, C78: 2.2n, Capacitor_SMD:C_0805_2012Metric
- removed R200: 22R, Resistor_SMD:R_Array_Convex_2x0402
- removed R36, R38, R39, R40, R45, R46, R47, R48, R49, R50, R55, R56, R65, R66, R67, R68, R69, R70: 10, Resistor_SMD:R_0805_2012Metric
- removed R53, R54, R57, R58, R71, R72, R77, R78: 1k, Resistor_SMD:R_0805_2012Metric
- removed R59, R60, R61, R62, R79, R80, R81, R82: 4.7k, Resistor_SMD:R_0805_2012Metric
- removed R73, R74, R75, R76, R83, R84, R85, R86: 39, Resistor_SMD:R_0805_2012Metric
- removed U11, U7: PCM1789, Package_SO:TSSOP-24_4.4x7.8mm_P0.65mm
- removed U9: LM4562, Package_SO:SOIC-8_3.9x4.9mm_P1.27mm
- added C110: 100n, Capacitor_SMD:C_0402_1005Metric, F.Cu at (319.5, 120.0)
- added R4: 22R, Resistor_SMD:R_Array_Convex_4x0402, F.Cu at (99.0, 152.0)
- C15, C16, C25, C26: value 100nF -> 100n
- C19: value 100n -> 1n5
- C21: value 100nF -> 100n; moved to F.Cu
- C7, C8: footprint Capacitor_SMD:C_0805_2012Metric -> Capacitor_SMD:C_0402_1005Metric
- C9: value 1n5 -> 100n; footprint Capacitor_SMD:C_0805_2012Metric -> Capacitor_SMD:C_0402_1005Metric
- J10, J11: footprint Connector_PinHeader_2.54mm:PinHeader_2x20_P2.54mm_Vertical -> Connector_IDC:IDC-Header_2x20_P2.54mm_Vertical
- R1, R2: value 22R -> 10R; footprint Resistor_SMD:R_Array_Convex_4x0402 -> Resistor_SMD:R_0805_2012Metric
- R24, R31, R32, R33, R34, R35: value 10 -> 10R
- moved R2 237.6 mm to (293.1, 70.0), turned to 0 degrees
- moved R1 230.0 mm to (293.1, 67.0), turned to 0 degrees
- moved C21 204.8 mm to (319.5, 114.1), turned to 0 degrees
- moved C3 194.7 mm to (313.8, 116.1), turned to 0 degrees
- moved C19 183.4 mm to (316.6, 120.0), turned to 0 degrees
- moved C2 180.8 mm to (313.8, 114.1), turned to 0 degrees
- moved C9 35.5 mm to (316.6, 114.1)
- moved C7 35.5 mm to (313.8, 118.0)
- moved C8 35.1 mm to (313.8, 120.0)
- moved C25 28.3 mm to (319.5, 116.1)
- moved C26 28.3 mm to (319.5, 118.0)
- moved C15 27.8 mm to (316.6, 116.1)
- moved C16 27.8 mm to (316.6, 118.0)
- moved R3 23.2 mm to (96.0, 152.0)
- moved U28 21.1 mm to (184.0, 136.0)
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Connections:
- C19 pad 1: +3.3V -> Net-(U2A-+)
- C19 pad 2: GND -> Net-(C19-Pad2)
- C9 pad 1: Net-(U2A-+) -> Net-(U2C-V+)
- C9 pad 2: Net-(C9-Pad2) -> GND
- J7 pad 1: /DAC_CH5_6/VOUT CH5(-) -> /VOUT CH5(-)
- J7 pad 3: /DAC_CH5_6/VOUT CH5(+) -> /VOUT CH5(+)
- J9 pad 1: /DAC_CH5_6/VOUT CH6(-) -> /VOUT CH6(-)
- J9 pad 3: /DAC_CH5_6/VOUT CH6(+) -> /VOUT CH6(+)
- R1 pad 1: Net-(R1-R1.1) -> +12V
- R1 pad 2: Net-(R1-R2.1) -> Net-(U2C-V+)
- R10 pad 1: Net-(C9-Pad2) -> Net-(C19-Pad2)
- R11 pad 2: Net-(C9-Pad2) -> Net-(C19-Pad2)
- R2 pad 1: Net-(R2-R1.1) -> Net-(U2C-V-)
- R2 pad 2: Net-(R2-R2.1) -> -12V
- R24 pad 1: Net-(U3B-V+) -> +12V
- R24 pad 2: +12V -> Net-(U3B-V+)
- R31 pad 1: -12V -> Net-(U3B-V-)
- R31 pad 2: Net-(U2C-V-) -> -12V
- R32 pad 1: Net-(U2C-V+) -> +12V
- R32 pad 2: +12V -> Net-(U4B-V+)
- R33 pad 1: Net-(U1-VCC1) -> +5V
- R33 pad 2: +5V -> Net-(U1-VCC1)
- R34 pad 1: Net-(U1-VCC2) -> +5V
- R34 pad 2: +5V -> Net-(U1-VCC2)
- R35 pad 1: -12V -> Net-(U4B-V-)
- R35 pad 2: Net-(U3B-V-) -> -12V
- U1 pad 17: /DAC_CH1_2/AMUTEI_CH1_2 -> Net-(R4-R1.2)
- U1 pad 4: /DAC_CH1_2/RST_CH1_2 -> +3.3V
- U2 pad 1: Net-(C9-Pad2) -> Net-(C19-Pad2)

Commit message: Worked on main board
Parts:
- moved C110 37.8 mm to (283.4, 130.9)
- moved C15 37.8 mm to (280.5, 127.0)
- moved C16 37.8 mm to (280.5, 129.0)
- moved C19 37.8 mm to (280.5, 130.9)
- moved C2 37.8 mm to (277.6, 125.0)
- moved C21 37.8 mm to (283.4, 125.0)
- moved C25 37.8 mm to (283.4, 127.0)
- moved C26 37.8 mm to (283.4, 129.0)
- moved C3 37.8 mm to (277.6, 127.0)
- moved C7 37.8 mm to (277.6, 129.0)
- moved C8 37.8 mm to (277.6, 130.9)
- moved C9 37.8 mm to (280.5, 125.0)
Changed lines of the file:
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@@
   )
   (footprint "Capacitor_SMD:C_0402_1005Metric" (layer "F.Cu")
-    (at 316.65 114.09)
+    (at 280.48 125.03)
     (descr "Capacitor SMD 0402 (1005 Metric), square (rectangular) end terminal, IPC_7351 nominal, (Body size source: IPC-SM-782 page 76, https://www.pcb-3d.com/wordpress/wp-content/uploads/ipc-sm-782a_amendment_1_and_2.pdf), generated with kicad-footprint-generator")
     (tags "capacitor")
@@
   )
   (footprint "Capacitor_SMD:C_0402_1005Metric" (layer "F.Cu")
-    (at 313.78 114.09)
+    (at 277.61 125.03)
     (descr "Capacitor SMD 0402 (1005 Metric), square (rectangular) end terminal, IPC_7351 nominal, (Body size source: IPC-SM-782 page 76, https://www.pcb-3d.com/wordpress/wp-content/uploads/ipc-sm-782a_amendment_1_and_2.pdf), generated with kicad-footprint-generator")
     (tags "capacitor")
@@
   )
   (footprint "Capacitor_SMD:C_0402_1005Metric" (layer "F.Cu")
-    (at 313.78 120)
+    (at 277.61 130.94)
     (descr "Capacitor SMD 0402 (1005 Metric), square (rectangular) end terminal, IPC_7351 nominal, (Body size source: IPC-SM-782 page 76, https://www.pcb-3d.com/wordpress/wp-content/uploads/ipc-sm-782a_amendment_1_and_2.pdf), generated with kicad-footprint-generator")
     (tags "capacitor")
@@
   )
   (footprint "Capacitor_SMD:C_0402_1005Metric" (layer "F.Cu")
-    (at 319.52 120)
+    (at 283.35 130.94)
     (descr "Capacitor SMD 0402 (1005 Metric), square (rectangular) end terminal, IPC_7351 nominal, (Body size source: IPC-SM-782 page 76, https://www.pcb-3d.com/wordpress/wp-content/uploads/ipc-sm-782a_amendment_1_and_2.pdf), generated with kicad-footprint-generator")
     (tags "capacitor")
@@
   )
   (footprint "Capacitor_SMD:C_0402_1005Metric" (layer "F.Cu")
-    (at 313.78 116.06)
+    (at 277.61 127)
     (descr "Capacitor SMD 0402 (1005 Metric), square (rectangular) end terminal, IPC_7351 nominal, (Body size source: IPC-SM-782 page 76, https://www.pcb-3d.com/wordpress/wp-content/uploads/ipc-sm-782a_amendment_1_and_2.pdf), generated with kicad-footprint-generator")
     (tags "capacitor")
@@
   )
   (footprint "Capacitor_SMD:C_0402_1005Metric" (layer "F.Cu")
-    (at 319.52 118.03)
+    (at 283.35 128.97)
     (descr "Capacitor SMD 0402 (1005 Metric), square (rectangular) end terminal, IPC_7351 nominal, (Body size source: IPC-SM-782 page 76, https://www.pcb-3d.com/wordpress/wp-content/uploads/ipc-sm-782a_amendment_1_and_2.pdf), generated with kicad-footprint-generator")
     (tags "capacitor")
@@
   )
   (footprint "Capacitor_SMD:C_0402_1005Metric" (layer "F.Cu")
-    (at 316.65 116.06)
+    (at 280.48 127)
     (descr "Capacitor SMD 0402 (1005 Metric), square (rectangular) end terminal, IPC_7351 nominal, (Body size source: IPC-SM-782 page 76, https://www.pcb-3d.com/wordpress/wp-content/uploads/ipc-sm-782a_amendment_1_and_2.pdf), generated with kicad-footprint-generator")
     (tags "capacitor")
@@
   )
   (footprint "Capacitor_SMD:C_0402_1005Metric" (layer "F.Cu")
-    (at 319.52 114.09)
+    (at 283.35 125.03)
     (descr "Capacitor SMD 0402 (1005 Metric), square (rectangular) end terminal, IPC_7351 nominal, (Body size source: IPC-SM-782 page 76, https://www.pcb-3d.com/wordpress/wp-content/uploads/ipc-sm-782a_amendment_1_and_2.pdf), generated with kicad-footprint-generator")
     (tags "capacitor")
@@
   )
   (footprint "Capacitor_SMD:C_0402_1005Metric" (layer "F.Cu")
-    (at 313.78 118.03)
+    (at 277.61 128.97)
     (descr "Capacitor SMD 0402 (1005 Metric), square (rectangular) end terminal, IPC_7351 nominal, (Body size source: IPC-SM-782 page 76, https://www.pcb-3d.com/wordpress/wp-content/uploads/ipc-sm-782a_amendment_1_and_2.pdf), generated with kicad-footprint-generator")
     (tags "capacitor")
@@
   )
   (footprint "Capacitor_SMD:C_0402_1005Metric" (layer "F.Cu")
-    (at 316.65 118.03)
+    (at 280.48 128.97)
     (descr "Capacitor SMD 0402 (1005 Metric), square (rectangular) end terminal, IPC_7351 nominal, (Body size source: IPC-SM-782 page 76, https://www.pcb-3d.com/wordpress/wp-content/uploads/ipc-sm-782a_amendment_1_and_2.pdf), generated with kicad-footprint-generator")
     (tags "capacitor")
@@
   )
   (footprint "Capacitor_SMD:C_0402_1005Metric" (layer "F.Cu")
-    (at 319.52 116.06)
+    (at 283.35 127)
     (descr "Capacitor SMD 0402 (1005 Metric), square (rectangular) end terminal, IPC_7351 nominal, (Body size source: IPC-SM-782 page 76, https://www.pcb-3d.com/wordpress/wp-content/uploads/ipc-sm-782a_amendment_1_and_2.pdf), generated with kicad-footprint-generator")
     (tags "capacitor")
@@
   )
   (footprint "Capacitor_SMD:C_0402_1005Metric" (layer "F.Cu")
-    (at 316.65 120)
+    (at 280.48 130.94)
     (descr "Capacitor SMD 0402 (1005 Metric), square (rectangular) end terminal, IPC_7351 nominal, (Body size source: IPC-SM-782 page 76, https://www.pcb-3d.com/wordpress/wp-content/uploads/ipc-sm-782a_amendment_1_and_2.pdf), generated with kicad-footprint-generator")
     (tags "capacitor")

Commit message: Worked on main board
Parts:
- U23, U24, U25, U26: footprint Audio DSP:LIN_REG_±xxV -> Audio_DSP:LIN_REG_±xxV
Changed lines of the file:
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@@
     )
   )
-  (footprint "Audio DSP:LIN_REG_±xxV" (layer "F.Cu")
+  (footprint "Audio_DSP:LIN_REG_±xxV" (layer "F.Cu")
     (at 141 126.35 90)
     (property "Sheetfile" "POWER_SUPPLIES.kicad_sch")
@@
     (property "ki_description" "LIN_REG_±12V")
     (attr smd)
-    (fp_text reference "U24" (at 0 -4.55 90 unlocked) (layer "F.SilkS") hide
+    (fp_text reference "U24" (at 0 -10.62 90 unlocked) (layer "F.SilkS") hide
         (effects (font (size 1 1) (thickness 0.1)))
     )
@@
         (effects (font (size 1 1) (thickness 0.15)))
     )
-    (fp_text user "${REFERENCE}" (at 0 -4 90 unlocked) (layer "F.Fab")
+    (fp_text user "${REFERENCE}" (at 0 0 90) (layer "F.Fab")
         (effects (font (size 1 1) (thickness 0.15)))
     )
-    (fp_text user "${REFERENCE}" (at 0 0 90) (layer "F.Fab")
+    (fp_text user "${REFERENCE}" (at 0 -4 90 unlocked) (layer "F.Fab")
         (effects (font (size 1 1) (thickness 0.15)))
     )
@@
       (net 2 "GND") (pinfunction "1") (pintype "input"))
   )
-  (footprint "Audio DSP:LIN_REG_±xxV" (layer "F.Cu")
+  (footprint "Audio_DSP:LIN_REG_±xxV" (layer "F.Cu")
     (at 150 145.35 90)
     (property "Sheetfile" "POWER_SUPPLIES.kicad_sch")
@@
     (property "ki_description" "LIN_REG_±12V")
     (attr smd)
-    (fp_text reference "U26" (at 0 -4.7 90 unlocked) (layer "F.SilkS") hide
+    (fp_text reference "U26" (at 0 -10.62 90 unlocked) (layer "F.SilkS") hide
         (effects (font (size 1 1) (thickness 0.1)))
     )
@@
         (effects (font (size 1 1) (thickness 0.15)))
     )
-    (fp_text user "${REFERENCE}" (at 0 0 90) (layer "F.Fab")
+    (fp_text user "${REFERENCE}" (at 0 -4 90 unlocked) (layer "F.Fab")
         (effects (font (size 1 1) (thickness 0.15)))
     )
-    (fp_text user "${REFERENCE}" (at 0 -4 90 unlocked) (layer "F.Fab")
+    (fp_text user "${REFERENCE}" (at 0 0 90) (layer "F.Fab")
         (effects (font (size 1 1) (thickness 0.15)))
     )
@@
     )
   )
-  (footprint "Audio DSP:LIN_REG_±xxV" (layer "F.Cu")
+  (footprint "Audio_DSP:LIN_REG_±xxV" (layer "F.Cu")
     (at 132 146.35 90)
     (property "Sheetfile" "POWER_SUPPLIES.kicad_sch")
@@
     (property "ki_description" "LIN_REG_±5V")
     (attr smd)
-    (fp_text reference "U25" (at 0 -4 90 unlocked) (layer "F.SilkS") hide
+    (fp_text reference "U25" (at 0 -10.62 90 unlocked) (layer "F.SilkS") hide
         (effects (font (size 1 1) (thickness 0.1)))
     )
@@
         (effects (font (size 1 1) (thickness 0.15)))
     )
-    (fp_text user "${REFERENCE}" (at 0 -4 90 unlocked) (layer "F.Fab")
+    (fp_text user "${REFERENCE}" (at 0 0 90) (layer "F.Fab")
         (effects (font (size 1 1) (thickness 0.15)))
     )
-    (fp_text user "${REFERENCE}" (at 0 0 90) (layer "F.Fab")
+    (fp_text user "${REFERENCE}" (at 0 -4 90 unlocked) (layer "F.Fab")
         (effects (font (size 1 1) (thickness 0.15)))
     )
@@
     )
   )
-  (footprint "Audio DSP:LIN_REG_±xxV" (layer "F.Cu")
+  (footprint "Audio_DSP:LIN_REG_±xxV" (layer "F.Cu")
     (at 159 126.35 90)
     (property "Sheetfile" "POWER_SUPPLIES.kicad_sch")
@@
     (property "ki_description" "LIN_REG_±5V")
     (attr smd)
-    (fp_text reference "U23" (at 0 -4.35 90 unlocked) (layer "F.SilkS") hide
+    (fp_text reference "U23" (at 0 -10.62 90 unlocked) (layer "F.SilkS") hide
         (effects (font (size 1 1) (thickness 0.1)))
     )
@@
         (effects (font (size 1 1) (thickness 0.15)))
     )
-    (fp_text user "${REFERENCE}" (at 0 -4 90 unlocked) (layer "F.Fab")
+    (fp_text user "${REFERENCE}" (at 0 0 90) (layer "F.Fab")
         (effects (font (size 1 1) (thickness 0.15)))
     )
-    (fp_text user "${REFERENCE}" (at 0 0 90) (layer "F.Fab")
+    (fp_text user "${REFERENCE}" (at 0 -4 90 unlocked) (layer "F.Fab")
         (effects (font (size 1 1) (thickness 0.15)))
     )

Commit message: Worked on main board
Parts:
- renumbered C9 to C1, C23 to C10, C24 to C11, C3 to C12, C5 to C13, C1 to C14, C25 to C15, C26 to C16, C7 to C17, C6 to C18, C28 to C19, C21 to C2, C30 to C20, C19 to C21, C8 to C22, C13 to C23, C14 to C24, C10 to C25, C11 to C26, C17 to C27, C18 to C28, C12 to C29, C4 to C3, C27 to C30, C88 to C31, C89 to C32, C90 to C33, C91 to C34, C84 to C36, C85 to C37, C86 to C38, C87 to C39, C22 to C4, C79 to C41, C80 to C42, C81 to C43, C98 to C44, C99 to C45, C100 to C46, C101 to C47, C20 to C5, C102 to C50, C103 to C51, C104 to C52, C105 to C53, C106 to C55, C107 to C56, C94 to C57, C95 to C58, C108 to C59, C110 to C6, C109 to C60, C96 to C61, C15 to C7, C16 to C8, C2 to C9, J8 to J10, J7 to J11, J9 to J12, J10 to J13, J11 to J14, J12 to J2, J13 to J3, J14 to J4, J2 to J5, J3 to J6, J4 to J7, J5 to J8, J6 to J9, R6 to R10, R12 to R11, R16 to R12, R18 to R13, R19 to R14, R20 to R15, R21 to R16, R13 to R17, R17 to R18, R22 to R19, R23 to R20, R25 to R21, R26 to R22, R7 to R23, R8 to R24, R11 to R25, R9 to R26, R10 to R29, R24 to R3, R29 to R30, R14 to R31, R15 to R32, R30 to R33, R37 to R34, R100 to R35, R101 to R36, R88 to R38, R90 to R39, R31 to R4, R87 to R42, R89 to R43, R91 to R46, R92 to R47, R33 to R5, R119 to R50, R120 to R51, R121 to R57, R122 to R58, R32 to R6, R106 to R62, R123 to R64, R124 to R65, R107 to R66, R110 to R69, R35 to R7, R111 to R70, R34 to R8, R5 to R9, R3 to RN1, R4 to RN2, U27 to U11, U23 to U12, U25 to U13, U24 to U14, U26 to U15, U28 to U7

Commit message: Worked on main board
Parts:
- added U3: OPA1632DR, Audio-DSP:VSSOP-8_3.0x3.0mm_P0.65_TP1.8x1.5, F.Cu at (336.8, 76.9)
- added U4: OPA1632DR, Audio-DSP:VSSOP-8_3.0x3.0mm_P0.65_TP1.8x1.5, F.Cu at (336.8, 81.5)
- added U5: OPA1632DR, Audio-DSP:VSSOP-8_3.0x3.0mm_P0.65_TP1.8x1.5, F.Cu at (336.8, 88.0)
- moved R17 82.5 mm to (337.7, 37.3)
- moved R25 81.5 mm to (342.1, 37.3)
- moved R26 77.7 mm to (342.1, 40.2)
- moved C17 77.1 mm to (320.6, 65.0)
- moved C16 75.7 mm to (320.6, 63.0)
- moved C8 75.7 mm to (317.7, 63.0)
- moved C21 75.5 mm to (320.6, 67.0)
- moved C22 75.4 mm to (320.6, 68.9)
- moved R11 73.1 mm to (333.3, 43.2)
- moved C12 72.2 mm to (317.7, 67.0)
- moved C9 72.2 mm to (317.7, 65.0)
- moved C6 71.3 mm to (314.8, 67.0)
- moved R27 71.0 mm to (342.1, 43.2)
- moved R28 71.0 mm to (342.1, 46.1)
- moved C10 70.9 mm to (315.7, 45.6)
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
Commit message: Added 3D model 744871004
Connections:
- H3 pad 1: GND -> unconnected-(H3-Pad1)
Changed lines of the file:
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@@
   (net 257 "unconnected-(U15--15V-Pad6)")
   (net 258 "Net-(U5A-VOCM)")
+  (net 259 "unconnected-(H3-Pad1)")
   (footprint "Connector_JST:JST_PH_B3B-PH-K_1x03_P2.00mm_Vertical" (layer "F.Cu")
     (at 105 103)
@@
     (property "Sheetfile" "Main board.kicad_sch")
     (property "Sheetname" "")
+    (property "exclude_from_bom" "")
     (property "ki_description" "Mounting Hole with connection")
     (property "ki_keywords" "mounting hole")
-    (attr exclude_from_pos_files)
+    (attr exclude_from_pos_files exclude_from_bom)
     (fp_text reference "H3" (at 0 -4.5) (layer "F.SilkS")
         (effects (font (size 1 1) (thickness 0.15)))
@@
       (stroke (width 0.05) (type solid)) (fill none) (layer "F.CrtYd"))
     (pad "1" thru_hole circle (at -2.625 0) (size 0.8 0.8) (drill 0.5) (layers "*.Cu" "*.Mask")
-      (net 2 "GND") (pinfunction "1") (pintype "input"))
+      (net 259 "unconnected-(H3-Pad1)") (pinfunction "1") (pintype "input"))
     (pad "1" thru_hole circle (at -1.856155 -1.856155) (size 0.8 0.8) (drill 0.5) (layers "*.Cu" "*.Mask")
-      (net 2 "GND") (pinfunction "1") (pintype "input"))
+      (net 259 "unconnected-(H3-Pad1)") (pinfunction "1") (pintype "input"))
     (pad "1" thru_hole circle (at -1.856155 1.856155) (size 0.8 0.8) (drill 0.5) (layers "*.Cu" "*.Mask")
-      (net 2 "GND") (pinfunction "1") (pintype "input"))
+      (net 259 "unconnected-(H3-Pad1)") (pinfunction "1") (pintype "input"))
     (pad "1" thru_hole circle (at 0 -2.625) (size 0.8 0.8) (drill 0.5) (layers "*.Cu" "*.Mask")
-      (net 2 "GND") (pinfunction "1") (pintype "input"))
+      (net 259 "unconnected-(H3-Pad1)") (pinfunction "1") (pintype "input"))
     (pad "1" thru_hole circle (at 0 0) (size 7 7) (drill 3.5) (layers "*.Cu" "*.Mask")
-      (net 2 "GND") (pinfunction "1") (pintype "input"))
+      (net 259 "unconnected-(H3-Pad1)") (pinfunction "1") (pintype "input"))
     (pad "1" thru_hole circle (at 0 2.625) (size 0.8 0.8) (drill 0.5) (layers "*.Cu" "*.Mask")
-      (net 2 "GND") (pinfunction "1") (pintype "input"))
+      (net 259 "unconnected-(H3-Pad1)") (pinfunction "1") (pintype "input"))
     (pad "1" thru_hole circle (at 1.856155 -1.856155) (size 0.8 0.8) (drill 0.5) (layers "*.Cu" "*.Mask")
-      (net 2 "GND") (pinfunction "1") (pintype "input"))
+      (net 259 "unconnected-(H3-Pad1)") (pinfunction "1") (pintype "input"))
     (pad "1" thru_hole circle (at 1.856155 1.856155) (size 0.8 0.8) (drill 0.5) (layers "*.Cu" "*.Mask")
-      (net 2 "GND") (pinfunction "1") (pintype "input"))
+      (net 259 "unconnected-(H3-Pad1)") (pinfunction "1") (pintype "input"))
     (pad "1" thru_hole circle (at 2.625 0) (size 0.8 0.8) (drill 0.5) (layers "*.Cu" "*.Mask")
-      (net 2 "GND") (pinfunction "1") (pintype "input"))
+      (net 259 "unconnected-(H3-Pad1)") (pinfunction "1") (pintype "input"))
   )
   (footprint "Capacitor_THT:CP_Radial_D5.0mm_P2.00mm" (layer "F.Cu")
