File: KiCAD/Main board/Main board.kicad_sch (KiCad schematic)
At the start: 2 parts, among them J1 Conn_01x03, J2 Conn_01x03

Commit message: KICAD
Parts:
- added J3, J5: Conn_01x02, Connector_JST:JST_PH_B2B-PH-K_1x02_P2.00mm_Vertical, symbol Connector_Generic:Conn_01x02
- added J4: Conn_01x03, Connector_JST:JST_PH_B3B-PH-K_1x03_P2.00mm_Vertical, symbol Connector_Generic:Conn_01x03
Connections:
- net DAC CH1_2/VOUT CH1(+): now reaches J2.1 (Pin_1)
- net GND: now reaches J2.2 (Pin_2)
- net GND: now also J3.2 (Pin_2), J4.2 (Pin_2), J5.2 (Pin_2)
- net DAC CH1_2/VOUT CH1(-): now reaches J2.3 (Pin_3)
- new net DAC CH1_2/RCA JACK CH1: J3.1 (Pin_1)
- new net DAC CH1_2/RCA/JACK CH2: J5.1 (Pin_1)
- new net DAC CH1_2/VOUT CH2(+): J4.3 (Pin_3)
- new net DAC CH1_2/VOUT CH2(-): J4.1 (Pin_1)
Other:
- sheet DAC CH1_2 ports: added RCA JACK CH1, RCA/JACK CH2, VOUT CH1(+), VOUT CH1(-), VOUT CH2(+), VOUT CH2(-); removed RCA JACK L, RCA/JACK R, VOUTL+, VOUTL-, VOUTR+, VOUTR-
- moved on the sheet: J2
Changed lines of the file:
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@@
 (kicad_sch (version 20230121) (generator eeschema)
   (paper "A4")
+  (wire (pts (xy 222.25 48.26) (xy 243.84 48.26))
+    (stroke (width 0) (type default))
+  )
+  (wire (pts (xy 222.25 74.93) (xy 243.84 74.93))
+    (stroke (width 0) (type default))
+  )
+  (wire (pts (xy 222.25 58.42) (xy 243.84 58.42))
+    (stroke (width 0) (type default))
+  )
+  (wire (pts (xy 222.25 64.77) (xy 243.84 64.77))
+    (stroke (width 0) (type default))
+  )
+  (wire (pts (xy 222.25 53.34) (xy 243.84 53.34))
+    (stroke (width 0) (type default))
+  )
+  (wire (pts (xy 222.25 69.85) (xy 243.84 69.85))
+    (stroke (width 0) (type default))
+  )
   (text "POWER SUPPLIES" (at 143.51 116.84 0)
     (effects (font (size 1.27 1.27)) (justify left bottom))
@@
     )
   )
-  (symbol (lib_id "Connector_Generic:Conn_01x03") (at 257.81 44.45 0) (unit 1)
-    (in_bom yes) (on_board yes) (dnp no)
-    (property "Reference" "J2" (at 255.7272 36.3982 0)
-      (effects (font (size 1.27 1.27)))
-    )
-    (property "Value" "Conn_01x03" (at 255.7272 38.7096 0)
-      (effects (font (size 1.27 1.27)))
-    )
-    (property "Footprint" "Connector_JST:JST_PH_B3B-PH-K_1x03_P2.00mm_Vertical" (at 257.81 44.45 0)
-      (effects (font (size 1.27 1.27)) hide)
-    )
-    (property "Datasheet" "~" (at 257.81 44.45 0)
+  (symbol (lib_id "power:GND") (at 243.84 77.47 270) (unit 1)
+    (in_bom yes) (on_board yes) (dnp no) (fields_autoplaced)
+    (property "Reference" "#PWR027" (at 237.49 77.47 0)
+      (effects (font (size 1.27 1.27)) hide)
+    )
+    (property "Value" "GND" (at 240.6651 77.7868 90)
+      (effects (font (size 1.27 1.27)) (justify right))
+    )
+    (property "Footprint" "" (at 243.84 77.47 0)
+      (effects (font (size 1.27 1.27)) hide)
+    )
+    (property "Datasheet" "" (at 243.84 77.47 0)
+      (effects (font (size 1.27 1.27)) hide)
+    )
+    (pin "1")
+    (instances
+      (project "Main board"
+        (path "/2f8cbac6-fd11-4240-8e40-3bb6952a0324"
+          (reference "#PWR027") (unit 1)
+        )
+      )
+    )
+  )
+  (symbol (lib_id "Connector_Generic:Conn_01x02") (at 248.92 58.42 0) (unit 1)
+    (in_bom yes) (on_board yes) (dnp no) (fields_autoplaced)
+    (property "Reference" "J3" (at 250.952 59.0463 0)
+      (effects (font (size 1.27 1.27)) (justify left))
+    )
+    (property "Value" "Conn_01x02" (at 250.952 60.9673 0)
+      (effects (font (size 1.27 1.27)) (justify left))
+    )
+    (property "Footprint" "Connector_JST:JST_PH_B2B-PH-K_1x02_P2.00mm_Vertical" (at 248.92 58.42 0)
+      (effects (font (size 1.27 1.27)) hide)
+    )
+    (property "Datasheet" "~" (at 248.92 58.42 0)
+      (effects (font (size 1.27 1.27)) hide)
+    )
+    (pin "1")
+    (pin "2")
+    (instances
+      (project "Main board"
+        (path "/2f8cbac6-fd11-4240-8e40-3bb6952a0324"
+          (reference "J3") (unit 1)
+        )
+      )
+    )
+  )
+  (symbol (lib_id "power:GND") (at 243.84 60.96 270) (unit 1)
+    (in_bom yes) (on_board yes) (dnp no) (fields_autoplaced)
+    (property "Reference" "#PWR024" (at 237.49 60.96 0)
+      (effects (font (size 1.27 1.27)) hide)
+    )
+    (property "Value" "GND" (at 240.6651 61.2768 90)
+      (effects (font (size 1.27 1.27)) (justify right))
+    )
+    (property "Footprint" "" (at 243.84 60.96 0)
+      (effects (font (size 1.27 1.27)) hide)
+    )
+    (property "Datasheet" "" (at 243.84 60.96 0)
+      (effects (font (size 1.27 1.27)) hide)
+    )
+    (pin "1")
+    (instances
+      (project "Main board"
+        (path "/2f8cbac6-fd11-4240-8e40-3bb6952a0324"
+          (reference "#PWR024") (unit 1)
+        )
+      )
+    )
+  )
+  (symbol (lib_id "Connector_Generic:Conn_01x03") (at 248.92 67.31 0) (unit 1)
+    (in_bom yes) (on_board yes) (dnp no)
+    (property "Reference" "J4" (at 252.73 66.04 0)
+      (effects (font (size 1.27 1.27)))
+    )
+    (property "Value" "Conn_01x03" (at 257.81 67.31 0)
+      (effects (font (size 1.27 1.27)))
+    )
+    (property "Footprint" "Connector_JST:JST_PH_B3B-PH-K_1x03_P2.00mm_Vertical" (at 248.92 67.31 0)
+      (effects (font (size 1.27 1.27)) hide)
+    )
+    (property "Datasheet" "~" (at 248.92 67.31 0)
       (effects (font (size 1.27 1.27)) hide)
     )
@@
       (project "Main board"
         (path "/2f8cbac6-fd11-4240-8e40-3bb6952a0324"
+          (reference "J4") (unit 1)
+        )
+      )
+    )
+  )
+  (symbol (lib_id "Connector_Generic:Conn_01x02") (at 248.92 74.93 0) (unit 1)
+    (in_bom yes) (on_board yes) (dnp no) (fields_autoplaced)
+    (property "Reference" "J5" (at 250.952 75.5563 0)
+      (effects (font (size 1.27 1.27)) (justify left))
+    )
+    (property "Value" "Conn_01x02" (at 250.952 77.4773 0)
+      (effects (font (size 1.27 1.27)) (justify left))
+    )
+    (property "Footprint" "Connector_JST:JST_PH_B2B-PH-K_1x02_P2.00mm_Vertical" (at 248.92 74.93 0)
+      (effects (font (size 1.27 1.27)) hide)
+    )
+    (property "Datasheet" "~" (at 248.92 74.93 0)
+      (effects (font (size 1.27 1.27)) hide)
+    )
+    (pin "1")
+    (pin "2")
+    (instances
+      (project "Main board"
+        (path "/2f8cbac6-fd11-4240-8e40-3bb6952a0324"
+          (reference "J5") (unit 1)
+        )
+      )
+    )
+  )
+  (symbol (lib_id "power:GND") (at 243.84 67.31 270) (unit 1)
+    (in_bom yes) (on_board yes) (dnp no)
+    (property "Reference" "#PWR026" (at 237.49 67.31 0)
+      (effects (font (size 1.27 1.27)) hide)
+    )
+    (property "Value" "GND" (at 240.03 67.31 90)
+      (effects (font (size 1.27 1.27)) (justify right))
+    )
+    (property "Footprint" "" (at 243.84 67.31 0)
+      (effects (font (size 1.27 1.27)) hide)
+    )
+    (property "Datasheet" "" (at 243.84 67.31 0)
+      (effects (font (size 1.27 1.27)) hide)
+    )
+    (pin "1")
+    (instances
+      (project "Main board"
+        (path "/2f8cbac6-fd11-4240-8e40-3bb6952a0324"
+          (reference "#PWR026") (unit 1)
+        )
+      )
+    )
+  )
+  (symbol (lib_id "Connector_Generic:Conn_01x03") (at 248.92 50.8 0) (unit 1)
+    (in_bom yes) (on_board yes) (dnp no)
+    (property "Reference" "J2" (at 251.46 49.53 0)
+      (effects (font (size 1.27 1.27)))
+    )
+    (property "Value" "Conn_01x03" (at 256.54 52.07 0)
+      (effects (font (size 1.27 1.27)))
+    )
+    (property "Footprint" "Connector_JST:JST_PH_B3B-PH-K_1x03_P2.00mm_Vertical" (at 248.92 50.8 0)
+      (effects (font (size 1.27 1.27)) hide)
+    )
+    (property "Datasheet" "~" (at 248.92 50.8 0)
+      (effects (font (size 1.27 1.27)) hide)
+    )
+    (pin "1")
+    (pin "2")
+    (pin "3")
+    (instances
+      (project "Main board"
+        (path "/2f8cbac6-fd11-4240-8e40-3bb6952a0324"
           (reference "J2") (unit 1)
         )
@@
     )
   )
-  (sheet (at 186.69 43.18) (size 35.56 38.1) (fields_autoplaced)
+  (symbol (lib_id "power:GND") (at 243.84 50.8 270) (unit 1)
+    (in_bom yes) (on_board yes) (dnp no)
+    (property "Reference" "#PWR025" (at 237.49 50.8 0)
+      (effects (font (size 1.27 1.27)) hide)
+    )
+    (property "Value" "GND" (at 240.03 50.8 90)
+      (effects (font (size 1.27 1.27)) (justify right))
+    )
+    (property "Footprint" "" (at 243.84 50.8 0)
+      (effects (font (size 1.27 1.27)) hide)
+    )
+    (property "Datasheet" "" (at 243.84 50.8 0)
+      (effects (font (size 1.27 1.27)) hide)
+    )
+    (pin "1")
+    (instances
+      (project "Main board"
+        (path "/2f8cbac6-fd11-4240-8e40-3bb6952a0324"
+          (reference "#PWR025") (unit 1)
+        )
+      )
+    )
+  )
+  (sheet (at 186.69 43.18) (size 35.56 38.1)
     (stroke (width 0.1524) (type solid))
     (fill (color 0 0 0 0.0000))
-    (property "Sheetname" "DAC CH1_2" (at 186.69 42.4684 0)
+    (property "Sheetname" "DAC CH1_2" (at 198.12 43.18 0)
       (effects (font (size 1.27 1.27)) (justify left bottom))
     )
-    (property "Sheetfile" "DAC CH 1_2.kicad_sch" (at 186.69 81.8646 0)
+    (property "Sheetfile" "DAC CH 1_2.kicad_sch" (at 190.5 81.28 0)
       (effects (font (size 1.27 1.27)) (justify left top))
     )
@@
       (effects (font (size 1.27 1.27)) (justify left))
     )
-    (pin "VOUTL-" input (at 222.25 54.61 0)
-      (effects (font (size 1.27 1.27)) (justify right))
-    )
-    (pin "VOUTL+" input (at 222.25 58.42 0)
-      (effects (font (size 1.27 1.27)) (justify right))
-    )
     (pin "ADR1" input (at 186.69 78.74 180)
       (effects (font (size 1.27 1.27)) (justify left))
@@
       (effects (font (size 1.27 1.27)) (justify left))
     )
-    (pin "RCA JACK L" input (at 222.25 50.8 0)
-      (effects (font (size 1.27 1.27)) (justify right))
-    )
-    (pin "VOUTR-" input (at 222.25 69.85 0)
-      (effects (font (size 1.27 1.27)) (justify right))
-    )
-    (pin "VOUTR+" input (at 222.25 72.39 0)
-      (effects (font (size 1.27 1.27)) (justify right))
-    )
-    (pin "RCA{slash}JACK R" input (at 222.25 74.93 0)
-      (effects (font (size 1.27 1.27)) (justify right))
-    )
+    (pin "VOUT CH1(+)" input (at 222.25 48.26 0)
+      (effects (font (size 1.27 1.27)) (justify right))
+    )
+    (pin "RCA{slash}JACK CH2" input (at 222.25 74.93 0)
+      (effects (font (size 1.27 1.27)) (justify right))
+    )
+    (pin "VOUT CH2(-)" input (at 222.25 64.77 0)
+      (effects (font (size 1.27 1.27)) (justify right))
+    )
+    (pin "VOUT CH2(+)" input (at 222.25 69.85 0)
+      (effects (font (size 1.27 1.27)) (justify right))
+    )
+    (pin "RCA JACK CH1" input (at 222.25 58.42 0)
+      (effects (font (size 1.27 1.27)) (justify right))
+    )
+    (pin "VOUT CH1(-)" input (at 222.25 53.34 0)
+      (effects (font (size 1.27 1.27)) (justify right))
+    )

Commit message: Updated BACK-END
Parts:
- added J6, J7, J8, J9: Conn_01x03, Connector_JST:JST_PH_B3B-PH-K_1x03_P2.00mm_Vertical, symbol Connector_Generic:Conn_01x03
Connections:
- net GND: now also J6.2 (Pin_2), J7.2 (Pin_2), J8.2 (Pin_2), J9.2 (Pin_2)
- new net DAC CH 5_6/VOUT CH5(+): J7.3 (Pin_3)
- new net DAC CH 5_6/VOUT CH5(-): J7.1 (Pin_1)
- new net DAC CH 5_6/VOUT CH6(+): J9.3 (Pin_3)
- new net DAC CH 5_6/VOUT CH6(-): J9.1 (Pin_1)
- new net DAC CH3_4/VOUT CH1(+): J8.3 (Pin_3)
- new net DAC CH3_4/VOUT CH1(-): J8.1 (Pin_1)
- new net DAC CH3_4/VOUT CH2(+): J6.3 (Pin_3)
- new net DAC CH3_4/VOUT CH2(-): J6.1 (Pin_1)
Other:
- sheet DAC CH 5_6 ports: added AMUTEI, BCK, DIN, LRCK, MC/SCL/FMT, MD/SDA/DEMP, MODE, RST, SCKI, VOUT CH5(+), VOUT CH5(-), VOUT CH6(+), VOUT CH6(-); removed none
- sheet DAC CH1_2 ports: added none; removed ADR0, ADR1
- sheet DAC CH3_4 ports: added AMUTEI, BCK, DIN, LRCK, MC/SCL/FMT, MD/SDA/DEMP, MODE, RST, SCKI, VOUT CH1(+), VOUT CH1(-), VOUT CH2(+), VOUT CH2(-); removed none
- moved on the sheet: J2, J3, J4, J5

Commit message: Started on Front-END
Other:
- added sheet ADC CH 1_2 (ADC CH1_2.kicad_sch)
- added sheet ADC CH 3_4 (untitled.kicad_sch)
- note removed: "ADC CH 1_2"
- note removed: "ADC CH 3_4"
- note removed: "ADC CH 5_6"
- moved on the sheet: J1
Changed lines of the file:
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@@
     (stroke (width 0) (type default))
   )
-  (text "POWER SUPPLIES" (at 143.51 116.84 0)
+  (text "POWER SUPPLIES" (at 219.71 207.01 0)
     (effects (font (size 1.27 1.27)) (justify left bottom))
   )
-  (text "ADC CH 1_2" (at 83.82 40.64 0)
+  (text "FPGA" (at 220.98 39.37 0)
     (effects (font (size 1.27 1.27)) (justify left bottom))
   )
-  (text "ADC CH 3_4" (at 83.82 66.04 0)
-    (effects (font (size 1.27 1.27)) (justify left bottom))
-  )
-  (text "ADC CH 5_6\n" (at 83.82 93.98 0)
-    (effects (font (size 1.27 1.27)) (justify left bottom))
-  )
-  (text "FPGA" (at 152.4 74.93 0)
-    (effects (font (size 1.27 1.27)) (justify left bottom))
-  )
-  (symbol (lib_id "Connector_Generic:Conn_01x03") (at 40.64 31.75 0) (mirror y) (unit 1)
-    (in_bom yes) (on_board yes) (dnp no)
-    (property "Reference" "J1" (at 42.7228 23.6982 0)
-      (effects (font (size 1.27 1.27)))
-    )
-    (property "Value" "Conn_01x03" (at 42.7228 26.0096 0)
-      (effects (font (size 1.27 1.27)))
-    )
-    (property "Footprint" "Connector_JST:JST_PH_B3B-PH-K_1x03_P2.00mm_Vertical" (at 40.64 31.75 0)
-      (effects (font (size 1.27 1.27)) hide)
-    )
-    (property "Datasheet" "~" (at 40.64 31.75 0)
+  (symbol (lib_id "Connector_Generic:Conn_01x03") (at 43.18 41.91 0) (mirror y) (unit 1)
+    (in_bom yes) (on_board yes) (dnp no)
+    (property "Reference" "J1" (at 45.2628 33.8582 0)
+      (effects (font (size 1.27 1.27)))
+    )
+    (property "Value" "Conn_01x03" (at 45.2628 36.1696 0)
+      (effects (font (size 1.27 1.27)))
+    )
+    (property "Footprint" "Connector_JST:JST_PH_B3B-PH-K_1x03_P2.00mm_Vertical" (at 43.18 41.91 0)
+      (effects (font (size 1.27 1.27)) hide)
+    )
+    (property "Datasheet" "~" (at 43.18 41.91 0)
       (effects (font (size 1.27 1.27)) hide)
     )
@@
     )
   )
+  (sheet (at 64.77 33.02) (size 48.26 58.42) (fields_autoplaced)
+    (stroke (width 0.1524) (type solid))
+    (fill (color 0 0 0 0.0000))
+    (property "Sheetname" "ADC CH 1_2" (at 64.77 32.3084 0)
+      (effects (font (size 1.27 1.27)) (justify left bottom))
+    )
+    (property "Sheetfile" "ADC CH1_2.kicad_sch" (at 64.77 92.0246 0)
+      (effects (font (size 1.27 1.27)) (justify left top))
+    )
+    (property "Field2" "" (at 64.77 33.02 0)
+      (effects (font (size 1.27 1.27)) hide)
+    )
+    (pin "RCA JACK CH1" input (at 64.77 45.72 180)
+      (effects (font (size 1.27 1.27)) (justify left))
+    )
+    (pin "RCA JACK CH2" input (at 64.77 49.53 180)
+      (effects (font (size 1.27 1.27)) (justify left))
+    )
+    (instances
+      (project "Main board"
+        (path "/2f8cbac6-fd11-4240-8e40-3bb6952a0324" (page "5"))
+      )
+    )
+  )
   (sheet (at 321.31 144.78) (size 35.56 50.8) (fields_autoplaced)
     (stroke (width 0.1524) (type solid))
@@
       )
     )
+  )
+  (sheet (at 64.77 99.06) (size 48.26 59.69) (fields_autoplaced)
+    (stroke (width 0.1524) (type solid))
+    (fill (color 0 0 0 0.0000))
+    (property "Sheetname" "ADC CH 3_4" (at 64.77 98.3484 0)
+      (effects (font (size 1.27 1.27)) (justify left bottom))
+    )
+    (property "Sheetfile" "untitled.kicad_sch" (at 64.77 159.3346 0)
+      (effects (font (size 1.27 1.27)) (justify left top))
+    )
+    (pin "VIN CH3(-)" input (at 64.77 109.22 180)
+      (effects (font (size 1.27 1.27)) (justify left))
+    )
+    (pin "VIN CH3(+)" input (at 64.77 113.03 180)
+      (effects (font (size 1.27 1.27)) (justify left))
+    )
+    (pin "VIN CH4(+)" input (at 64.77 120.65 180)
+      (effects (font (size 1.27 1.27)) (justify left))
+    )
+    (pin "VIN CH4(-)" input (at 64.77 124.46 180)
+      (effects (font (size 1.27 1.27)) (justify left))
+    )
+    (instances
+      (project "Main board"
+        (path "/2f8cbac6-fd11-4240-8e40-3bb6952a0324" (page "6"))
+      )
+    )

Commit message: Worked on main board
Other:
- sheet ADC CH 1_2 renamed ADC_CH1_2
- sheet ADC CH 3_4 renamed ADC_CH3_4
- sheet DAC CH 5_6 renamed DAC_CH5_6
- sheet DAC CH1_2 renamed DAC_CH1_2
- sheet DAC CH3_4 renamed DAC_CH3_4
- added sheet FPGA (FPGA.kicad_sch)
- added sheet POWER_SUPPLIES (POWER_SUPPLIES.kicad_sch)
- sheet ADC_CH1_2: file ADC CH1_2.kicad_sch -> ADC_CH1_2.kicad_sch
- sheet ADC_CH3_4: file untitled.kicad_sch -> ADC_CH3_4.kicad_sch
- sheet DAC_CH1_2: file DAC CH 1_2.kicad_sch -> DAC_CH1_2.kicad_sch
- sheet DAC_CH3_4: file DAC CH3_4.kicad_sch -> DAC_CH3_4.kicad_sch
- sheet DAC_CH5_6: file DAC CH 5_6.kicad_sch -> DAC_CH5_6.kicad_sch
- note removed: "FPGA"
- note removed: "POWER SUPPLIES"
Changed lines of the file:
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@@
     (stroke (width 0) (type default))
-  )
-  (text "POWER SUPPLIES" (at 219.71 207.01 0)
-    (effects (font (size 1.27 1.27)) (justify left bottom))
-  )
-  (text "FPGA" (at 220.98 39.37 0)
-    (effects (font (size 1.27 1.27)) (justify left bottom))
   )
   (symbol (lib_id "Connector_Generic:Conn_01x03") (at 43.18 41.91 0) (mirror y) (unit 1)
@@
     (stroke (width 0.1524) (type solid))
     (fill (color 0 0 0 0.0000))
-    (property "Sheetname" "DAC CH1_2" (at 332.74 25.4 0)
+    (property "Sheetname" "DAC_CH1_2" (at 332.74 25.4 0)
       (effects (font (size 1.27 1.27)) (justify left bottom))
     )
-    (property "Sheetfile" "DAC CH 1_2.kicad_sch" (at 326.39 76.2 0)
+    (property "Sheetfile" "DAC_CH1_2.kicad_sch" (at 326.39 76.2 0)
       (effects (font (size 1.27 1.27)) (justify left top))
     )
@@
     (stroke (width 0.1524) (type solid))
     (fill (color 0 0 0 0.0000))
-    (property "Sheetname" "DAC CH3_4" (at 321.31 83.1084 0)
+    (property "Sheetname" "DAC_CH3_4" (at 321.31 83.1084 0)
       (effects (font (size 1.27 1.27)) (justify left bottom))
     )
-    (property "Sheetfile" "DAC CH3_4.kicad_sch" (at 321.31 132.6646 0)
+    (property "Sheetfile" "DAC_CH3_4.kicad_sch" (at 321.31 132.6646 0)
       (effects (font (size 1.27 1.27)) (justify left top))
     )
@@
       (project "Main board"
         (path "/2f8cbac6-fd11-4240-8e40-3bb6952a0324" (page "3"))
+      )
+    )
+  )
+  (sheet (at 193.04 27.94) (size 58.42 39.37) (fields_autoplaced)
+    (stroke (width 0.1524) (type solid))
+    (fill (color 0 0 0 0.0000))
+    (property "Sheetname" "FPGA" (at 193.04 27.2284 0)
+      (effects (font (size 1.27 1.27)) (justify left bottom))
+    )
+    (property "Sheetfile" "FPGA.kicad_sch" (at 193.04 67.8946 0)
+      (effects (font (size 1.27 1.27)) (justify left top))
+    )
+    (instances
+      (project "Main board"
+        (path "/2f8cbac6-fd11-4240-8e40-3bb6952a0324" (page "8"))
       )
     )
@@
     (stroke (width 0.1524) (type solid))
     (fill (color 0 0 0 0.0000))
-    (property "Sheetname" "ADC CH 1_2" (at 64.77 32.3084 0)
+    (property "Sheetname" "ADC_CH1_2" (at 64.77 32.3084 0)
       (effects (font (size 1.27 1.27)) (justify left bottom))
     )
-    (property "Sheetfile" "ADC CH1_2.kicad_sch" (at 64.77 92.0246 0)
+    (property "Sheetfile" "ADC_CH1_2.kicad_sch" (at 64.77 92.0246 0)
       (effects (font (size 1.27 1.27)) (justify left top))
-    )
-    (property "Field2" "" (at 64.77 33.02 0)
-      (effects (font (size 1.27 1.27)) hide)
     )
     (pin "RCA JACK CH1" input (at 64.77 45.72 180)
@@
     (stroke (width 0.1524) (type solid))
     (fill (color 0 0 0 0.0000))
-    (property "Sheetname" "DAC CH 5_6" (at 321.31 144.0684 0)
+    (property "Sheetname" "DAC_CH5_6" (at 321.31 144.0684 0)
       (effects (font (size 1.27 1.27)) (justify left bottom))
     )
-    (property "Sheetfile" "DAC CH 5_6.kicad_sch" (at 321.31 196.1646 0)
+    (property "Sheetfile" "DAC_CH5_6.kicad_sch" (at 321.31 196.1646 0)
       (effects (font (size 1.27 1.27)) (justify left top))
     )
@@
     (stroke (width 0.1524) (type solid))
     (fill (color 0 0 0 0.0000))
-    (property "Sheetname" "ADC CH 3_4" (at 64.77 98.3484 0)
+    (property "Sheetname" "ADC_CH3_4" (at 64.77 98.3484 0)
       (effects (font (size 1.27 1.27)) (justify left bottom))
     )
-    (property "Sheetfile" "untitled.kicad_sch" (at 64.77 159.3346 0)
+    (property "Sheetfile" "ADC_CH3_4.kicad_sch" (at 64.77 159.3346 0)
       (effects (font (size 1.27 1.27)) (justify left top))
     )
@@
       )
     )
+  )
+  (sheet (at 160.02 176.53) (size 77.47 36.83) (fields_autoplaced)
+    (stroke (width 0.1524) (type solid))
+    (fill (color 0 0 0 0.0000))
+    (property "Sheetname" "POWER_SUPPLIES" (at 160.02 175.8184 0)
+      (effects (font (size 1.27 1.27)) (justify left bottom))
+    )
+    (property "Sheetfile" "POWER_SUPPLIES.kicad_sch" (at 160.02 213.9446 0)
+      (effects (font (size 1.27 1.27)) (justify left top))
+    )
+    (instances
+      (project "Main board"
+        (path "/2f8cbac6-fd11-4240-8e40-3bb6952a0324" (page "7"))
+      )
+    )
