File: KiCAD/Main board/Main board.kicad_sch (KiCad schematic)
At the start: 9 parts, among them J1 Conn_01x03, J2 Conn_01x03, J3 Conn_01x02, J4 Conn_01x03, J5 Conn_01x02, J6 Conn_01x03, J7 Conn_01x03, J8 Conn_01x03, J9 Conn_01x03

Commit message: Worked on KiCAD
Parts:
- added H1, H2, H3, H4, H5, H6, H7, H8: MountingHole_Pad, MountingHole:MountingHole_3.5mm_Pad_Via, symbol Mechanical:MountingHole_Pad
Changed lines of the file:
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@@
+    )
+  )
+  (symbol (lib_id "Mechanical:MountingHole_Pad") (at 342.9 237.49 0) (unit 1)
+    (in_bom yes) (on_board yes) (dnp no) (fields_autoplaced)
+    (property "Reference" "H7" (at 345.44 235.585 0)
+      (effects (font (size 1.27 1.27)) (justify left))
+    )
+    (property "Value" "MountingHole_Pad" (at 345.44 238.125 0)
+      (effects (font (size 1.27 1.27)) (justify left))
+    )
+    (property "Footprint" "MountingHole:MountingHole_3.5mm_Pad_Via" (at 342.9 237.49 0)
+      (effects (font (size 1.27 1.27)) hide)
+    )
+    (property "Datasheet" "NA" (at 342.9 237.49 0)
+      (effects (font (size 1.27 1.27)) hide)
+    )
+    (pin "1")
+    (instances
+      (project "Main board"
+        (path "/2f8cbac6-fd11-4240-8e40-3bb6952a0324"
+          (reference "H7") (unit 1)
+        )
+      )
+    )
+  )
+  (symbol (lib_id "Mechanical:MountingHole_Pad") (at 317.5 227.33 0) (unit 1)
+    (in_bom yes) (on_board yes) (dnp no) (fields_autoplaced)
+    (property "Reference" "H2" (at 320.04 225.425 0)
+      (effects (font (size 1.27 1.27)) (justify left))
+    )
+    (property "Value" "MountingHole_Pad" (at 320.04 227.965 0)
+      (effects (font (size 1.27 1.27)) (justify left))
+    )
+    (property "Footprint" "MountingHole:MountingHole_3.5mm_Pad_Via" (at 317.5 227.33 0)
+      (effects (font (size 1.27 1.27)) hide)
+    )
+    (property "Datasheet" "NA" (at 317.5 227.33 0)
+      (effects (font (size 1.27 1.27)) hide)
+    )
+    (pin "1")
+    (instances
+      (project "Main board"
+        (path "/2f8cbac6-fd11-4240-8e40-3bb6952a0324"
+          (reference "H2") (unit 1)
+        )
+      )
     )
   )
@@
     )
   )
+  (symbol (lib_id "Mechanical:MountingHole_Pad") (at 342.9 247.65 0) (unit 1)
+    (in_bom yes) (on_board yes) (dnp no) (fields_autoplaced)
+    (property "Reference" "H8" (at 345.44 245.745 0)
+      (effects (font (size 1.27 1.27)) (justify left))
+    )
+    (property "Value" "MountingHole_Pad" (at 345.44 248.285 0)
+      (effects (font (size 1.27 1.27)) (justify left))
+    )
+    (property "Footprint" "MountingHole:MountingHole_3.5mm_Pad_Via" (at 342.9 247.65 0)
+      (effects (font (size 1.27 1.27)) hide)
+    )
+    (property "Datasheet" "NA" (at 342.9 247.65 0)
+      (effects (font (size 1.27 1.27)) hide)
+    )
+    (pin "1")
+    (instances
+      (project "Main board"
+        (path "/2f8cbac6-fd11-4240-8e40-3bb6952a0324"
+          (reference "H8") (unit 1)
+        )
+      )
+    )
+  )
   (symbol (lib_id "power:GND") (at 375.92 154.94 270) (unit 1)
     (in_bom yes) (on_board yes) (dnp no)
@@
     )
   )
+  (symbol (lib_id "Mechanical:MountingHole_Pad") (at 342.9 217.17 0) (unit 1)
+    (in_bom yes) (on_board yes) (dnp no) (fields_autoplaced)
+    (property "Reference" "H5" (at 345.44 215.265 0)
+      (effects (font (size 1.27 1.27)) (justify left))
+    )
+    (property "Value" "MountingHole_Pad" (at 345.44 217.805 0)
+      (effects (font (size 1.27 1.27)) (justify left))
+    )
+    (property "Footprint" "MountingHole:MountingHole_3.5mm_Pad_Via" (at 342.9 217.17 0)
+      (effects (font (size 1.27 1.27)) hide)
+    )
+    (property "Datasheet" "NA" (at 342.9 217.17 0)
+      (effects (font (size 1.27 1.27)) hide)
+    )
+    (pin "1")
+    (instances
+      (project "Main board"
+        (path "/2f8cbac6-fd11-4240-8e40-3bb6952a0324"
+          (reference "H5") (unit 1)
+        )
+      )
+    )
+  )
   (symbol (lib_id "Connector_Generic:Conn_01x03") (at 382.27 121.92 0) (unit 1)
     (in_bom yes) (on_board yes) (dnp no)
@@
     )
   )
+  (symbol (lib_id "Mechanical:MountingHole_Pad") (at 317.5 237.49 0) (unit 1)
+    (in_bom yes) (on_board yes) (dnp no) (fields_autoplaced)
+    (property "Reference" "H3" (at 320.04 235.585 0)
+      (effects (font (size 1.27 1.27)) (justify left))
+    )
+    (property "Value" "MountingHole_Pad" (at 320.04 238.125 0)
+      (effects (font (size 1.27 1.27)) (justify left))
+    )
+    (property "Footprint" "MountingHole:MountingHole_3.5mm_Pad_Via" (at 317.5 237.49 0)
+      (effects (font (size 1.27 1.27)) hide)
+    )
+    (property "Datasheet" "NA" (at 317.5 237.49 0)
+      (effects (font (size 1.27 1.27)) hide)
+    )
+    (pin "1")
+    (instances
+      (project "Main board"
+        (path "/2f8cbac6-fd11-4240-8e40-3bb6952a0324"
+          (reference "H3") (unit 1)
+        )
+      )
+    )
+  )
   (symbol (lib_id "power:GND") (at 381 62.23 270) (unit 1)
     (in_bom yes) (on_board yes) (dnp no)
@@
     )
   )
+  (symbol (lib_id "Mechanical:MountingHole_Pad") (at 342.9 227.33 0) (unit 1)
+    (in_bom yes) (on_board yes) (dnp no) (fields_autoplaced)
+    (property "Reference" "H6" (at 345.44 225.425 0)
+      (effects (font (size 1.27 1.27)) (justify left))
+    )
+    (property "Value" "MountingHole_Pad" (at 345.44 227.965 0)
+      (effects (font (size 1.27 1.27)) (justify left))
+    )
+    (property "Footprint" "MountingHole:MountingHole_3.5mm_Pad_Via" (at 342.9 227.33 0)
+      (effects (font (size 1.27 1.27)) hide)
+    )
+    (property "Datasheet" "NA" (at 342.9 227.33 0)
+      (effects (font (size 1.27 1.27)) hide)
+    )
+    (pin "1")
+    (instances
+      (project "Main board"
+        (path "/2f8cbac6-fd11-4240-8e40-3bb6952a0324"
+          (reference "H6") (unit 1)
+        )
+      )
+    )
+  )
   (symbol (lib_id "Connector_Generic:Conn_01x03") (at 381 185.42 0) (unit 1)
     (in_bom yes) (on_board yes) (dnp no)
@@
         )
       )
+    )
+  )
+  (symbol (lib_id "Mechanical:MountingHole_Pad") (at 317.5 247.65 0) (unit 1)
+    (in_bom yes) (on_board yes) (dnp no) (fields_autoplaced)
+    (property "Reference" "H4" (at 320.04 245.745 0)
+      (effects (font (size 1.27 1.27)) (justify left))
+    )
+    (property "Value" "MountingHole_Pad" (at 320.04 248.285 0)
+      (effects (font (size 1.27 1.27)) (justify left))
+    )
+    (property "Footprint" "MountingHole:MountingHole_3.5mm_Pad_Via" (at 317.5 247.65 0)
+      (effects (font (size 1.27 1.27)) hide)
+    )
+    (property "Datasheet" "NA" (at 317.5 247.65 0)
+      (effects (font (size 1.27 1.27)) hide)
+    )
+    (pin "1")
+    (instances
+      (project "Main board"
+        (path "/2f8cbac6-fd11-4240-8e40-3bb6952a0324"
+          (reference "H4") (unit 1)
+        )
+      )
+    )
+  )
+  (symbol (lib_id "Mechanical:MountingHole_Pad") (at 317.5 217.17 0) (unit 1)
+    (in_bom yes) (on_board yes) (dnp no) (fields_autoplaced)
+    (property "Reference" "H1" (at 320.04 215.265 0)
+      (effects (font (size 1.27 1.27)) (justify left))
+    )
+    (property "Value" "MountingHole_Pad" (at 320.04 217.805 0)
+      (effects (font (size 1.27 1.27)) (justify left))
+    )
+    (property "Footprint" "MountingHole:MountingHole_3.5mm_Pad_Via" (at 317.5 217.17 0)
+      (effects (font (size 1.27 1.27)) hide)
+    )
+    (property "Datasheet" "NA" (at 317.5 217.17 0)
+      (effects (font (size 1.27 1.27)) hide)
+    )
+    (pin "1")
+    (instances
+      (project "Main board"
+        (path "/2f8cbac6-fd11-4240-8e40-3bb6952a0324"
+          (reference "H1") (unit 1)
+        )
+      )

Commit message: Worked a bit on the main board
Parts:
- added J12: Conn_01x03, Connector_JST:JST_PH_B3B-PH-K_1x03_P2.00mm_Vertical, symbol Connector_Generic:Conn_01x03
- added J13, J14: Conn_01x02, Connector_JST:JST_PH_B2B-PH-K_1x02_P2.00mm_Vertical, symbol Connector_Generic:Conn_01x02
Connections:
- net GND: now also H1.1, H2.1, H3.1, H4.1, H5.1, H6.1, H7.1, H8.1; no longer J3.2 (Pin_2), J5.2 (Pin_2)
- net DAC_CH1_2/RCA JACK CH1 renamed DAC_CH1_2/RCA_JACK_CH1(+)
- net DAC_CH1_2/RCA/JACK CH2 renamed DAC_CH1_2/RCA_JACK_CH2(+)
- net DAC_CH1_2/VOUT CH1(+) renamed DAC_CH1_2/VOUT_CH1(+)
- net DAC_CH1_2/VOUT CH1(-) renamed DAC_CH1_2/VOUT_CH1(-)
- net DAC_CH1_2/VOUT CH2(+) renamed DAC_CH1_2/VOUT_CH2(-)
- net DAC_CH1_2/VOUT CH2(-) renamed DAC_CH1_2/VOUT_CH2(+)
- new net DAC_CH1_2/RCA_JACK_CH1(REF): J3.2 (Pin_2)
- new net DAC_CH1_2/RCA_JACK_CH2(REF): J5.2 (Pin_2)
Other:
- sheet DAC_CH1_2 ports: added AMUTEI_CH1_2, BCK_CH1_2, DIN_CH1_2, LRCK_CH1_2, RCA_JACK_CH1(+), RCA_JACK_CH1(REF), RCA_JACK_CH2(+), RCA_JACK_CH2(REF), RST_CH1_2, SCKI_CH1_2, SCL_CH1_2, SDA_CH1_2, VOUT_CH1(+), VOUT_CH1(-), VOUT_CH2(+), VOUT_CH2(-); removed AMUTEI, BCK, DIN, LRCK, MC/SCL/FMT, MD/SDA/DEMP, MODE, RCA JACK CH1, RCA/JACK CH2, RST, SCKI, VOUT CH1(+), VOUT CH1(-), VOUT CH2(+), VOUT CH2(-)
- sheet FPGA ports: added AMUTEI_CH1_2, BCK_CH1_2, DIN_CH1_2, LRCK_CH1_2, RST_CH1_2, SCKI_CH1_2, SCL_CH1_2, SDA_CH1_2; removed none
- note added: "LEAVE INTERNALS FOR NOW"
- title: (none) -> AUDIO-DSP_MAIN_BOARD
- moved on the sheet: H1, H2, H3, H4, H5, H6, H7, H8, J1, J2, J3, J4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

Commit message: Worked on main board
Other:
- moved on the sheet: J2, J3, J4, J5, J6, J7, J8, J9

Commit message: Worked on main board
Parts:
- renumbered J8 to J10, J7 to J11, J9 to J12, J12 to J2, J13 to J3, J14 to J4, J2 to J5, J3 to J6, J4 to J7, J5 to J8, J6 to J9
