File: KiCAD/Main board/Main board.kicad_sch (KiCad schematic)
At the start: 29 parts, among them J1 Conn_01x03, J10 Conn_01x03, J11 Conn_01x03, J12 Conn_01x03, J13 Conn_01x02, J14 Conn_01x02, J15 Conn_01x06, J16 Conn_01x02, J17 Conn_01x02, J18 Conn_01x05, J2 Conn_01x03, J3 Conn_01x02, J4 Conn_01x02, J5 Conn_01x03, J6 Conn_01x02, J7 Conn_01x03, J8 Conn_01x02, J9 Conn_01x03

Commit message: Worked on main board schematic
Connections:
- net ADC_CH1_2/VU_LED1_CH1 renamed ADC_CH1_2/VU_G1_CH1
- net ADC_CH1_2/VU_LED1_CH2 renamed ADC_CH1_2/VU_G1_CH2
- net ADC_CH1_2/VU_LED2_CH1 renamed ADC_CH1_2/VU_G2_CH1
- net ADC_CH1_2/VU_LED2_CH2 renamed ADC_CH1_2/VU_G2_CH2
- net ADC_CH1_2/VU_LED3_CH1 renamed ADC_CH1_2/VU_O1_CH1
- net ADC_CH1_2/VU_LED3_CH2 renamed ADC_CH1_2/VU_O1_CH2
- net ADC_CH1_2/VU_LED4_CH1 renamed ADC_CH1_2/VU_R1_CH1
- net ADC_CH1_2/VU_LED4_CH2 renamed ADC_CH1_2/VU_R1_CH2
Other:
- sheet ADC_CH1_2 ports: added VU_G1_CH1, VU_G1_CH2, VU_G2_CH1, VU_G2_CH2, VU_O1_CH1, VU_O1_CH2, VU_R1_CH1, VU_R1_CH2; removed VU_LED1_CH1, VU_LED1_CH2, VU_LED2_CH1, VU_LED2_CH2, VU_LED3_CH1, VU_LED3_CH2, VU_LED4_CH1, VU_LED4_CH2
Changed lines of the file:
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@@
-      (effects (font (size 1.27 1.27)) (justify left))
-    )
-    (pin "VU_LED4_CH2" output (at 137.16 83.82 180)
-      (effects (font (size 1.27 1.27)) (justify left))
-    )
-    (pin "VU_LED3_CH2" output (at 137.16 81.28 180)
-      (effects (font (size 1.27 1.27)) (justify left))
-    )
-    (pin "VU_LED2_CH2" output (at 137.16 78.74 180)
-      (effects (font (size 1.27 1.27)) (justify left))
-    )
-    (pin "VU_LED1_CH2" output (at 137.16 76.2 180)
-      (effects (font (size 1.27 1.27)) (justify left))
-    )
-    (pin "VU_LED4_CH1" output (at 137.16 68.58 180)
-      (effects (font (size 1.27 1.27)) (justify left))
-    )
-    (pin "VU_LED3_CH1" output (at 137.16 66.04 180)
-      (effects (font (size 1.27 1.27)) (justify left))
-    )
-    (pin "VU_LED2_CH1" output (at 137.16 63.5 180)
-      (effects (font (size 1.27 1.27)) (justify left))
-    )
-    (pin "VU_LED1_CH1" output (at 137.16 60.96 180)
       (effects (font (size 1.27 1.27)) (justify left))
     )
@@
       (effects (font (size 1.27 1.27)) (justify right))
     )
+    (pin "VU_G1_CH1" output (at 137.16 60.96 180)
+      (effects (font (size 1.27 1.27)) (justify left))
+    )
+    (pin "VU_G2_CH1" output (at 137.16 63.5 180)
+      (effects (font (size 1.27 1.27)) (justify left))
+    )
+    (pin "VU_O1_CH1" output (at 137.16 66.04 180)
+      (effects (font (size 1.27 1.27)) (justify left))
+    )
+    (pin "VU_R1_CH1" output (at 137.16 68.58 180)
+      (effects (font (size 1.27 1.27)) (justify left))
+    )
+    (pin "VU_G1_CH2" output (at 137.16 76.2 180)
+      (effects (font (size 1.27 1.27)) (justify left))
+    )
+    (pin "VU_G2_CH2" output (at 137.16 78.74 180)
+      (effects (font (size 1.27 1.27)) (justify left))
+    )
+    (pin "VU_O1_CH2" output (at 137.16 81.28 180)
+      (effects (font (size 1.27 1.27)) (justify left))
+    )
+    (pin "VU_R1_CH2" output (at 137.16 83.82 180)
+      (effects (font (size 1.27 1.27)) (justify left))
+    )
     (instances

Commit message: Worked on main board schematic
Other:
- moved on the sheet: J1, J10, J11, J12, J15, J16, J17, J18, J2, J3, J4, J5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
