File: KiCAD/Main board/ADC_CH1_2.kicad_sch (KiCad schematic)
At the start: 31 parts, among them U13 OPA1632DR, U15 OPA1632DR, U16 LM4562

Commit message: Worked a bit on the main board
Parts:
- removed unit 3 of U16
- added U22: LM4562, symbol Amplifier_Operational:LM4562
- added U27: PCM1804, Package_SO:SSOP-28_5.3x10.2mm_P0.65mm, symbol Audio-DSP:PCM1804
Connections:
- net at C35.1, C4.1, R32.1: now also U22.8 (V+)
- net at C21.2, C22.2, R31.2: now also U22.4 (V-)
Changed lines of the file:
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@@
 (kicad_sch (version 20230121) (generator eeschema)
-  (paper "A4")
+  (paper "A3")
   (junction (at 106.68 97.79) (diameter 0) (color 0 0 0 0)
   )
@@
   (junction (at 76.2 100.33) (diameter 0) (color 0 0 0 0)
   )
+  (junction (at 66.04 182.88) (diameter 0) (color 0 0 0 0)
+  )
   (junction (at 78.74 175.26) (diameter 0) (color 0 0 0 0)
   )
@@
   (junction (at 158.75 104.14) (diameter 0) (color 0 0 0 0)
   )
+  (junction (at 39.37 181.61) (diameter 0) (color 0 0 0 0)
+  )
+  (junction (at 123.19 127) (diameter 0) (color 0 0 0 0)
+  )
+  (junction (at 152.4 104.14) (diameter 0) (color 0 0 0 0)
+  )
+  (junction (at 21.59 181.61) (diameter 0) (color 0 0 0 0)
+  )
+  (junction (at 152.4 124.46) (diameter 0) (color 0 0 0 0)
+  )
+  (junction (at 90.17 175.26) (diameter 0) (color 0 0 0 0)
+  )
+  (junction (at 172.72 114.3) (diameter 0) (color 0 0 0 0)
+  )
+  (junction (at 50.8 173.99) (diameter 0) (color 0 0 0 0)
+  )
+  (junction (at 66.04 90.17) (diameter 0) (color 0 0 0 0)
+  )
+  (junction (at 39.37 173.99) (diameter 0) (color 0 0 0 0)
+  )
   (junction (at 66.04 167.64) (diameter 0) (color 0 0 0 0)
-  )
-  (junction (at 39.37 181.61) (diameter 0) (color 0 0 0 0)
-  )
-  (junction (at 123.19 127) (diameter 0) (color 0 0 0 0)
-  )
-  (junction (at 152.4 104.14) (diameter 0) (color 0 0 0 0)
-  )
-  (junction (at 21.59 181.61) (diameter 0) (color 0 0 0 0)
-  )
-  (junction (at 152.4 124.46) (diameter 0) (color 0 0 0 0)
-  )
-  (junction (at 90.17 175.26) (diameter 0) (color 0 0 0 0)
-  )
-  (junction (at 172.72 114.3) (diameter 0) (color 0 0 0 0)
-  )
-  (junction (at 50.8 173.99) (diameter 0) (color 0 0 0 0)
-  )
-  (junction (at 66.04 90.17) (diameter 0) (color 0 0 0 0)
-  )
-  (junction (at 39.37 173.99) (diameter 0) (color 0 0 0 0)
-  )
-  (junction (at 66.04 182.88) (diameter 0) (color 0 0 0 0)
   )
   (junction (at 106.68 92.71) (diameter 0) (color 0 0 0 0)
@@
     )
   )
+  (symbol (lib_id "Audio-DSP:PCM1804") (at 146.05 49.53 0) (unit 1)
+    (in_bom yes) (on_board yes) (dnp no) (fields_autoplaced)
+    (property "Reference" "U27" (at 150.5459 25.4 0)
+      (effects (font (size 1.27 1.27)) (justify left))
+    )
+    (property "Value" "PCM1804" (at 150.5459 27.94 0)
+      (effects (font (size 1.27 1.27)) (justify left))
+    )
+    (property "Footprint" "Package_SO:SSOP-28_5.3x10.2mm_P0.65mm" (at 113.03 81.28 0)
+      (effects (font (size 1.27 1.27)) (justify left) hide)
+    )
+    (property "Datasheet" "https://nl.mouser.com/ProductDetail/Texas-Instruments/PCM1804DBR?qs=wgAEGBTxy7lnBW3YYZcxMA%3D%3D" (at 113.03 83.82 0)
+      (effects (font (size 1.27 1.27)) (justify left) hide)
+    )
+    (pin "1")
+    (pin "10")
+    (pin "11")
+    (pin "12")
+    (pin "13")
+    (pin "14")
+    (pin "15")
+    (pin "16")
+    (pin "17")
+    (pin "18")
+    (pin "19")
+    (pin "2")
+    (pin "20")
+    (pin "21")
+    (pin "22")
+    (pin "23")
+    (pin "24")
+    (pin "25")
+    (pin "26")
+    (pin "27")
+    (pin "28")
+    (pin "3")
+    (pin "4")
+    (pin "5")
+    (pin "6")
+    (pin "7")
+    (pin "8")
+    (pin "9")
+    (instances
+      (project "Main board"
+        (path "/2f8cbac6-fd11-4240-8e40-3bb6952a0324/b7530516-5ab1-4afa-9366-b30c4f029458"
+          (reference "U27") (unit 1)
+        )
+        (path "/2f8cbac6-fd11-4240-8e40-3bb6952a0324/4e10d7ae-7c54-4ac5-ac67-e4842ffdf025"
+          (reference "U28") (unit 1)
+        )
+      )
+    )
+  )
   (symbol (lib_id "Device:R") (at 85.09 138.43 90) (unit 1)
     (in_bom yes) (on_board yes) (dnp no)
@@
     )
   )
-  (symbol (lib_id "Amplifier_Operational:LM4562") (at 63.5 175.26 180) (unit 3)
+  (symbol (lib_id "Device:R") (at 21.59 162.56 180) (unit 1)
+    (in_bom yes) (on_board yes) (dnp no)
+    (property "Reference" "R36" (at 19.05 162.56 90)
+      (effects (font (size 1.27 1.27)))
+    )
+    (property "Value" "10" (at 21.59 162.56 90)
+      (effects (font (size 1.27 1.27)))
+    )
+    (property "Footprint" "Resistor_SMD:R_0805_2012Metric" (at 23.368 162.56 90)
+      (effects (font (size 1.27 1.27)) hide)
+    )
+    (property "Datasheet" "~" (at 21.59 162.56 0)
+      (effects (font (size 1.27 1.27)) hide)
+    )
+    (pin "1")
+    (pin "2")
+    (instances
+      (project "Main board"
+        (path "/2f8cbac6-fd11-4240-8e40-3bb6952a0324/03c234da-ad6d-41dc-b0ec-5880e5376fd2"
+          (reference "R36") (unit 1)
+        )
+        (path "/2f8cbac6-fd11-4240-8e40-3bb6952a0324/4e10d7ae-7c54-4ac5-ac67-e4842ffdf025"
+          (reference "R100") (unit 1)
+        )
+      )
+    )
+  )
+  (symbol (lib_id "power:+12V") (at 66.04 158.75 0) (unit 1)
     (in_bom yes) (on_board yes) (dnp no) (fields_autoplaced)
-    (property "Reference" "U16" (at 66.675 174.6163 0)
-      (effects (font (size 1.27 1.27)) (justify right) hide)
-    )
-    (property "Value" "LM4562" (at 66.675 176.5373 0)
-      (effects (font (size 1.27 1.27)) (justify right) hide)
-    )
-    (property "Footprint" "" (at 63.5 175.26 0)
-      (effects (font (size 1.27 1.27)) hide)
-    )
-    (property "Datasheet" "http://www.ti.com/lit/ds/symlink/lm4562.pdf" (at 63.5 175.26 0)
+    (property "Reference" "#PWR014" (at 66.04 162.56 0)
+      (effects (font (size 1.27 1.27)) hide)
+    )
+    (property "Value" "+12V" (at 66.04 155.2481 0)
+      (effects (font (size 1.27 1.27)))
+    )
+    (property "Footprint" "" (at 66.04 158.75 0)
+      (effects (font (size 1.27 1.27)) hide)
+    )
+    (property "Datasheet" "" (at 66.04 158.75 0)
+      (effects (font (size 1.27 1.27)) hide)
+    )
+    (pin "1")
+    (instances
+      (project "Main board"
+        (path "/2f8cbac6-fd11-4240-8e40-3bb6952a0324/03c234da-ad6d-41dc-b0ec-5880e5376fd2"
+          (reference "#PWR014") (unit 1)
+        )
+        (path "/2f8cbac6-fd11-4240-8e40-3bb6952a0324/05d59304-dfac-45e1-85e6-83cda4d81484"
+          (reference "#PWR013") (unit 1)
+        )
+        (path "/2f8cbac6-fd11-4240-8e40-3bb6952a0324/4e10d7ae-7c54-4ac5-ac67-e4842ffdf025"
+          (reference "#PWR078") (unit 1)
+        )
+      )
+    )
+  )
+  (symbol (lib_id "Amplifier_Operational:LM4562") (at 68.58 175.26 0) (unit 3)
+    (in_bom yes) (on_board yes) (dnp no)
+    (property "Reference" "U22" (at 69.85 177.181 0)
+      (effects (font (size 1.27 1.27)))
+    )
+    (property "Value" "LM4562" (at 69.85 175.26 0)
+      (effects (font (size 1.27 1.27)))
+    )
+    (property "Footprint" "" (at 68.58 175.26 0)
+      (effects (font (size 1.27 1.27)) hide)
+    )
+    (property "Datasheet" "http://www.ti.com/lit/ds/symlink/lm4562.pdf" (at 68.58 175.26 0)
       (effects (font (size 1.27 1.27)) hide)
     )
@@
       (project "Main board"
         (path "/2f8cbac6-fd11-4240-8e40-3bb6952a0324/4e10d7ae-7c54-4ac5-ac67-e4842ffdf025"
-          (reference "U16") (unit 3)
-        )
-      )
-    )
-  )
-  (symbol (lib_id "Device:R") (at 21.59 162.56 180) (unit 1)
-    (in_bom yes) (on_board yes) (dnp no)
-    (property "Reference" "R36" (at 19.05 162.56 90)
-      (effects (font (size 1.27 1.27)))
-    )
-    (property "Value" "10" (at 21.59 162.56 90)
-      (effects (font (size 1.27 1.27)))
-    )
-    (property "Footprint" "Resistor_SMD:R_0805_2012Metric" (at 23.368 162.56 90)
-      (effects (font (size 1.27 1.27)) hide)
-    )
-    (property "Datasheet" "~" (at 21.59 162.56 0)
-      (effects (font (size 1.27 1.27)) hide)
-    )
-    (pin "1")
-    (pin "2")
-    (instances
-      (project "Main board"
-        (path "/2f8cbac6-fd11-4240-8e40-3bb6952a0324/03c234da-ad6d-41dc-b0ec-5880e5376fd2"
-          (reference "R36") (unit 1)
-        )
-        (path "/2f8cbac6-fd11-4240-8e40-3bb6952a0324/4e10d7ae-7c54-4ac5-ac67-e4842ffdf025"
-          (reference "R100") (unit 1)
-        )
-      )
-    )
-  )
-  (symbol (lib_id "power:+12V") (at 66.04 158.75 0) (unit 1)
-    (in_bom yes) (on_board yes) (dnp no) (fields_autoplaced)
-    (property "Reference" "#PWR014" (at 66.04 162.56 0)
-      (effects (font (size 1.27 1.27)) hide)
-    )
-    (property "Value" "+12V" (at 66.04 155.2481 0)
-      (effects (font (size 1.27 1.27)))
-    )
-    (property "Footprint" "" (at 66.04 158.75 0)
-      (effects (font (size 1.27 1.27)) hide)
-    )
-    (property "Datasheet" "" (at 66.04 158.75 0)
-      (effects (font (size 1.27 1.27)) hide)
-    )
-    (pin "1")
-    (instances
-      (project "Main board"
-        (path "/2f8cbac6-fd11-4240-8e40-3bb6952a0324/03c234da-ad6d-41dc-b0ec-5880e5376fd2"
-          (reference "#PWR014") (unit 1)
-        )
-        (path "/2f8cbac6-fd11-4240-8e40-3bb6952a0324/05d59304-dfac-45e1-85e6-83cda4d81484"
-          (reference "#PWR013") (unit 1)
-        )
-        (path "/2f8cbac6-fd11-4240-8e40-3bb6952a0324/4e10d7ae-7c54-4ac5-ac67-e4842ffdf025"
-          (reference "#PWR078") (unit 1)
+          (reference "U22") (unit 3)
         )
       )
@@
   (symbol (lib_id "Device:C") (at 158.75 113.03 0) (unit 1)
     (in_bom yes) (on_board yes) (dnp no)
-    (property "Reference" "C12" (at 171.831 112.3863 0)
-      (effects (font (size 1.27 1.27)) (justify left))
-    )
-    (property "Value" "2.7n" (at 171.831 114.3073 0)
-      (effects (font (size 1.27 1.27)) (justify left))
-    )
+    (property "Reference" "C12" (at 162.56 111.76 0)
+      (effects (font (size 1.27 1.27)) (justify left))
+    )
+    (property "Value" "2.7n" (at 162.56 114.3 0)
+      (effects (font (size 1.27 1.27)) (justify left))
+    )

Commit message: Worked on main board
Parts:
- U5: renamed from U15; now in the parts list
- U5: renamed from U13; now in the parts list
- renumbered C83 to C35, C82 to C40, R94 to R37, R95 to R40, R96 to R41, R97 to R44, R93 to R45, R98 to R48, R99 to R49, U22 to U6, U16 to U6

Commit message: Worked on main board
Parts:
- U5: footprint Audio_DSP:VSSOP-8_3.0x3.0mm_P0.65_TP1.8x1.5 -> Audio-DSP:VSSOP-8_3.0x3.0mm_P0.65_TP1.8x1.5
Other:
- moved on the sheet: U27
