File: KiCAD/Main board/ADC_CH1_2.kicad_sch (KiCad schematic)
At the start: 114 parts, among them K1 EA2-12NU, K2 EA2-12NU, Q1 BC847, Q2 BC847, Q3 BC847, Q4 BC857, U24 LM4562, U25 OPA1632DR, U34 TL072, U35 TL072, U36 LM339, U38 PGA2311P, U39 TXS0102, U4 OPA1632DR, U5 OPA1632DR, U6 LM4562, U7 PCM1804

Commit message: Worked on main board schematic
Parts:
- added C1 (x2): 10u, Capacitor_SMD:C_1210_3225Metric, symbol Device:C
- added C9 (x2): 47p, Capacitor_SMD:C_0402_1005Metric, symbol Device:C
- added D10, D7, D8, D9: 1N4148WS, Diode_SMD:D_SOD-323, symbol Diode:1N4148WS
- added R1 (x6): 2k, Resistor_SMD:R_0805_2012Metric, symbol Device:R
- added R1 (x2): 24k, Resistor_SMD:R_0805_2012Metric, symbol Device:R
- added R1 (x6): 1k, Resistor_SMD:R_0805_2012Metric, symbol Device:R
- added R20 (x4): 10k, Resistor_SMD:R_0805_2012Metric, symbol Device:R
- added R20 (x8): 330, Resistor_SMD:R_0805_2012Metric, symbol Device:R
- added R20: 100k, Resistor_SMD:R_0805_2012Metric, symbol Device:R
Connections:
- net +5VD1: now also C1.1, C1.1, U36.3 (V+), U36.3 (V+), R1.2, R1.2
- net GND: now also C1.2, C1.2, R1.1, R1.1, R1.1, R1.1, R1.1, R1.1
- net at U36.10 (-): now also R1.1, R1.2 (x2)
- net at U36.11 (+): now also U36.5 (+), U36.7 (+), U36.9 (+), C1.1, R1.1, R1.2
- net at C30.1, D4.2 (A2), R19.2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: no longer U35.3 (+)
- net at U36.6 (-): now also R1.1, R1.2 (x2)
- net at U36.7 (+): now also U36.11 (+), U36.5 (+), U36.9 (+), C1.1, R1.1, R1.2
- net at U36.8 (-): now also R1.1, R1.2 (x2)
- net at U35.5 (+): now also D10.1 (K), R1.2
- net at U35.6 (-): now also R20.1, R20.2
- net at U35.7: now also U36.4 (-), R1.2, R20.1
- net at C30.1, D3.2 (A2), R19.2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: no longer U34.3 (+)
- net at U34.5 (+): now also D8.1 (K), R1.2
- net at U34.6 (-): now also R20.1, R20.2
- net at U34.7: now also U36.4 (-), R1.2, R20.1
- net at U35.1: now also C9.2, D10.2 (A), D9.1 (K); no longer U35.2 (-)
- net at U34.1: now also C9.2, D7.1 (K), D8.2 (A); no longer U34.2 (-)
- net at R20.1: now also U34.3 (+)
- net VU_LED1_CH1: no longer names the net of U36.2
- net VU_LED1_CH1: now also R20.2
- net VU_LED1_CH2: no longer names the net of U36.2
- net VU_LED1_CH2: now also R20.2
- net VU_LED2_CH1: no longer names the net of U36.1
- net VU_LED2_CH1: now also R20.2
- net VU_LED2_CH2: no longer names the net of U36.1
- net VU_LED2_CH2: now also R20.2
- net VU_LED3_CH1: no longer names the net of U36.13
- net VU_LED3_CH1: now also R20.2
- net VU_LED3_CH2: no longer names the net of U36.13
- net VU_LED3_CH2: now also R20.2
- net VU_LED4_CH1: no longer names the net of U36.14
- net VU_LED4_CH1: now also R20.2
- net VU_LED4_CH2: no longer names the net of U36.14
- net VU_LED4_CH2: now also R20.2
- new net: C9.1, D9.2 (A), R20.2, U35.2 (-)
- new net: C9.1, D7.2 (A), R20.2, U34.2 (-)
- new net: R20.1, U35.3 (+)
- new net VU_G1_CH1: R20.1
- new net VU_G1_CH2: R20.1
- new net VU_G2_CH1: R20.1
- new net VU_G2_CH2: R20.1
- new net VU_O1_CH1: R20.1
- new net VU_O1_CH2: R20.1
- new net VU_R1_CH1: R20.1
- new net VU_R1_CH2: R20.1
- no-connect marks 5 -> 3
Other:
- note added: "Block diagram updaten adv plaatsing VU-meter"
- note added: "Weerstandswaarden verhogen? Waarde afronden naar E24"
- note removed: "+12V or +5V? ADC en VU-meter position"
- note removed: "DC-offset creëren voor comparator?"
- moved on the sheet: R20, U34A, U34B, U35A, U35B, U36A, U36B, U36C, U36D
