File: KiCAD/Main board/ADC_CH1_2.kicad_sch (KiCad schematic)
At the start: 149 parts, among them K1 EA2-12NU, K2 EA2-12NU, Q1 BC847, Q2 BC847, Q3 BC847, Q4 BC857, U24 LM4562, U25 OPA1632DR, U34 TL072, U35 TL072, U36 LM339, U38 PGA2311P, U39 TXS0102, U4 OPA1632DR, U5 OPA1632DR, U6 LM4562, U7 PCM1804

Commit message: Worked on main board schematic
Parts:
- removed NT1 (x2): NetTie_2, Audio-DSP:NetTie-2_SMD_Pad0.3mm, symbol Device:NetTie_2
- removed R20 (x2): 100k, Resistor_SMD:R_0805_2012Metric, symbol Device:R
- added NT1 (x2): NetTie_2, Audio-DSP:NetTie-2_SMD_Pad0.3mm, symbol Device:NetTie_2
- added R1 (x2): 100k, Resistor_SMD:R_0805_2012Metric, symbol Device:R
Connections:
- net ~{RST_ADC_CH1_2} is gone; now on net +3V3D1: U7.19 (~{RST})
- net GND: now also NT1.1, NT1.1
- net at C30.2, R20.2, R34.2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: now also NT1.2 (x2)
- net at U38.14 (VOUTL), U6.3 (+): now also R1.2
- net AGND_CH1: now reaches C30.2, D3.1 (A1), K1.8, NT1.2, R1.2, U38.15 (AGNDL)
- net AGND_CH1: now also R16.1
- net AGND_CH2: now reaches C30.2, D4.1 (A1), K2.8, NT1.2, R1.2, U38.10 (AGNDR)
- net AGND_CH2: now also R16.1
- net at U24.3 (+), U38.11 (VOUTR): now also R1.1
- net at U35.3 (+): now also R1.2
- net at U34.3 (+): now also R1.1
Other:
- note added: "Place nettie at ADC input"
- note added: "RST aan +3V3D1"
- note added: "RST inactive"
- note removed: "Check output impedance of PGA2311 Misschien kan deze buffer weg"
- note removed: "RST kan ook aan +3V3D1"
- moved on the sheet: C1, C13, C27, C28, C3, C30, C39, C5, C9, D1, D10, D2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

Commit message: Worked on main board
Other:
- note removed: "Block diagram updaten adv plaatsing VU-meter"
- note removed: "RST aan +3V3D1"
Changed lines of the file:
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@@
     (effects (font (size 1.27 1.27)) (justify left bottom))
-  )
-  (text "RST aan +3V3D1" (at 426.72 85.09 0)
-    (effects (font (size 1.27 1.27) (color 200 0 200 1)) (justify left bottom))
   )
   (text "Bidirectional level translator" (at 130.81 133.35 0)
@@
     (effects (font (size 1.27 1.27) (color 200 0 200 1)) (justify left bottom))
   )
-  (text "Block diagram updaten adv plaatsing VU-meter" (at 91.44 67.31 0)
-    (effects (font (size 1.27 1.27) (color 200 0 200 1)) (justify left bottom))
-  )

Commit message: Main board, ordering of PCBs and LTspice simulations
Parts:
- removed NT1 (x2): NetTie_2, Audio-DSP:NetTie-2_SMD_Pad0.3mm, symbol Device:NetTie_2
- R1: value 2k -> 3k9
Other:
- note added: "1.74V clipping 870mV -6dB 435mV -12dB 218mV -18dB"
- note added: "Add 0R resistors to be able to change some settings? -Sample freq -bits"
- note removed: "Place nettie at ADC input"
- note removed: "Weerstandswaarden verhogen? Waarde afronden naar E24"
Changed lines of the file:
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@@
   (junction (at 243.84 157.48) (diameter 0) (color 0 0 0 0)
   )
-  (junction (at 363.22 138.43) (diameter 0) (color 0 0 0 0)
-  )
   (junction (at 143.51 182.88) (diameter 0) (color 0 0 0 0)
   )
@@
   (junction (at 109.22 175.26) (diameter 0) (color 0 0 0 0)
   )
-  (junction (at 360.68 72.39) (diameter 0) (color 0 0 0 0)
-  )
   (junction (at 184.15 115.57) (diameter 0) (color 0 0 0 0)
   )
@@
     (stroke (width 0) (type default))
   )
-  (text "Place nettie at ADC input" (at 358.14 77.47 0)
-    (effects (font (size 1.27 1.27)) (justify left bottom))
-  )
-  (text "Weerstandswaarden verhogen?\nWaarde afronden naar E24"
-    (at 191.77 54.61 0)
-    (effects (font (size 1.27 1.27) (color 200 0 200 1)) (justify left bottom))
-  )
   (text "QUAD mode" (at 431.8 103.505 0)
     (effects (font (size 1.27 1.27)) (justify left bottom))
@@
     (effects (font (size 1.27 1.27)) (justify left bottom))
   )
-  (text "Weerstandswaarden verhogen?\nWaarde afronden naar E24"
-    (at 222.25 160.02 0)
-    (effects (font (size 1.27 1.27) (color 200 0 200 1)) (justify right bottom))
-  )
   (text "INPUT_SELECTOR_RELAY\nLOW=RCA\nHIGH-Jack" (at 132.08 43.18 0)
     (effects (font (size 1.27 1.27)) (justify left bottom))
@@
     (effects (font (size 1.27 1.27)) (justify left bottom))
   )
-  (text "Place nettie at ADC input" (at 367.03 142.24 0)
+  (text "1.74V     clipping\n870mV   -6dB\n435mV  -12dB\n218mV  -18dB"
+    (at 205.74 57.15 0)
     (effects (font (size 1.27 1.27)) (justify left bottom))
   )
+  (text "Add 0R resistors to be able to change some settings?\n-Sample freq\n-bits"
+    (at 401.32 114.3 0)
+    (effects (font (size 1.27 1.27) (color 200 0 200 1)) (justify left bottom))
+  )
   (text "Unmuted" (at 137.16 100.965 0)
     (effects (font (size 1.27 1.27)) (justify left bottom))
@@
     (effects (font (size 1.27 1.27) (color 200 0 200 1)) (justify left bottom))
   )
+  (text "1.74V     clipping\n870mV   -6dB\n435mV  -12dB\n218mV  -18dB"
+    (at 205.74 137.16 0)
+    (effects (font (size 1.27 1.27)) (justify left bottom))
+  )
   (label "AGND_CH1" (at 288.29 63.5 0) (fields_autoplaced)
     (effects (font (size 1.27 1.27)) (justify left bottom))
@@
       (effects (font (size 1.27 1.27)) (justify left))
     )
-    (property "Value" "2k" (at 227.33 115.57 0)
+    (property "Value" "3k9" (at 227.33 115.57 0)
       (effects (font (size 1.27 1.27)) (justify left))
     )
@@
     )
   )
-  (symbol (lib_id "power:GND") (at 355.6 72.39 270) (unit 1)
-    (in_bom yes) (on_board yes) (dnp no)
-    (property "Reference" "#PWR0128" (at 349.25 72.39 0)
-      (effects (font (size 1.27 1.27)) hide)
-    )
-    (property "Value" "GND" (at 353.06 72.39 90)
-      (effects (font (size 1.27 1.27)) (justify right))
-    )
-    (property "Footprint" "" (at 355.6 72.39 0)
-      (effects (font (size 1.27 1.27)) hide)
-    )
-    (property "Datasheet" "" (at 355.6 72.39 0)
-      (effects (font (size 1.27 1.27)) hide)
-    )
-    (pin "1")
-    (instances
-      (project "Main board"
-        (path "/2f8cbac6-fd11-4240-8e40-3bb6952a0324/03c234da-ad6d-41dc-b0ec-5880e5376fd2"
-          (reference "#PWR0128") (unit 1)
-        )
-        (path "/2f8cbac6-fd11-4240-8e40-3bb6952a0324/4e10d7ae-7c54-4ac5-ac67-e4842ffdf025"
-          (reference "#PWR0191") (unit 1)
-        )
-      )
-    )
-  )
   (symbol (lib_id "Device:R") (at 234.95 161.29 0) (mirror x) (unit 1)
     (in_bom yes) (on_board yes) (dnp no)
@@
     )
   )
-  (symbol (lib_id "power:GND") (at 363.22 143.51 0) (unit 1)
-    (in_bom yes) (on_board yes) (dnp no)
-    (property "Reference" "#PWR0117" (at 363.22 149.86 0)
-      (effects (font (size 1.27 1.27)) hide)
-    )
-    (property "Value" "GND" (at 363.22 147.32 0)
-      (effects (font (size 1.27 1.27)))
-    )
-    (property "Footprint" "" (at 363.22 143.51 0)
-      (effects (font (size 1.27 1.27)) hide)
-    )
-    (property "Datasheet" "" (at 363.22 143.51 0)
-      (effects (font (size 1.27 1.27)) hide)
-    )
-    (pin "1")
-    (instances
-      (project "Main board"
-        (path "/2f8cbac6-fd11-4240-8e40-3bb6952a0324/03c234da-ad6d-41dc-b0ec-5880e5376fd2"
-          (reference "#PWR0117") (unit 1)
-        )
-        (path "/2f8cbac6-fd11-4240-8e40-3bb6952a0324/4e10d7ae-7c54-4ac5-ac67-e4842ffdf025"
-          (reference "#PWR085") (unit 1)
-        )
-      )
-    )
-  )
   (symbol (lib_id "Audio-DSP:TXS0102") (at 149.86 123.19 0) (unit 1)
     (in_bom yes) (on_board yes) (dnp no)
@@
       (effects (font (size 1.27 1.27)) (justify left))
     )
-    (property "Value" "2k" (at 227.33 35.56 0)
+    (property "Value" "3k9" (at 227.33 35.56 0)
       (effects (font (size 1.27 1.27)) (justify left))
     )
@@
     )
   )
-  (symbol (lib_id "Device:NetTie_2") (at 363.22 140.97 90) (unit 1)
-    (in_bom no) (on_board yes) (dnp no)
-    (property "Reference" "NT1" (at 361.95 140.97 0)
-      (effects (font (size 1.27 1.27)))
-    )
-    (property "Value" "NetTie_2" (at 351.79 142.24 90)
-      (effects (font (size 1.27 1.27)) (justify right))
-    )
-    (property "Footprint" "Audio-DSP:NetTie-2_SMD_Pad0.3mm" (at 363.22 140.97 0)
-      (effects (font (size 1.27 1.27)) hide)
-    )
-    (property "Datasheet" "~" (at 363.22 140.97 0)
-      (effects (font (size 1.27 1.27)) hide)
-    )
-    (pin "1")
-    (pin "2")
-    (instances
-      (project "Main board"
-        (path "/2f8cbac6-fd11-4240-8e40-3bb6952a0324/03c234da-ad6d-41dc-b0ec-5880e5376fd2"
-          (reference "NT1") (unit 1)
-        )
-        (path "/2f8cbac6-fd11-4240-8e40-3bb6952a0324/4e10d7ae-7c54-4ac5-ac67-e4842ffdf025"
-          (reference "NT4") (unit 1)
-        )
-      )
-    )
-  )
   (symbol (lib_id "Transistor_BJT:BC847") (at 54.61 46.99 0) (mirror y) (unit 1)
     (in_bom yes) (on_board yes) (dnp no) (fields_autoplaced)
@@
         )
       )
-    )
-  )
-  (symbol (lib_id "Device:NetTie_2") (at 358.14 72.39 0) (unit 1)
-    (in_bom no) (on_board yes) (dnp no)
-    (property "Reference" "NT1" (at 358.14 71.12 0)
-      (effects (font (size 1.27 1.27)))
-    )
-    (property "Value" "NetTie_2" (at 362.585 73.66 0)
-      (effects (font (size 1.27 1.27)) (justify right))
-    )
-    (property "Footprint" "Audio-DSP:NetTie-2_SMD_Pad0.3mm" (at 358.14 72.39 0)
-      (effects (font (size 1.27 1.27)) hide)
-    )
-    (property "Datasheet" "~" (at 358.14 72.39 0)
-      (effects (font (size 1.27 1.27)) hide)
-    )
-    (pin "1")
-    (pin "2")
-    (instances
-      (project "Main board"
-        (path "/2f8cbac6-fd11-4240-8e40-3bb6952a0324/03c234da-ad6d-41dc-b0ec-5880e5376fd2"
-          (reference "NT1") (unit 1)
-        )
-        (path "/2f8cbac6-fd11-4240-8e40-3bb6952a0324/4e10d7ae-7c54-4ac5-ac67-e4842ffdf025"
-          (reference "NT3") (unit 1)
-        )
-      )

Commit message: Ad good as finilized the main board schematic
Parts:
- R19, R20: value 270 -> 2k7
Other:
- note added: "Add 0R resistors to be able to change some settings? -Sample freq->OSRX -bits->OSRX"
- note added: "Place this isolation resistors as close to the audio signal as possible."
- note removed: "Add 0R resistors to be able to change some settings? -Sample freq -bits"
- title: (none) -> AUDIO-DSP_MAIN_BOARD
Changed lines of the file:
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@@
 (kicad_sch (version 20230121) (generator eeschema)
   (paper "User" 464.998 215.011)
+  (title_block
+    (title "AUDIO-DSP_MAIN_BOARD")
+    (rev "R01")
+  )
   (junction (at 210.82 175.26) (diameter 0) (color 0 0 0 0)
   )
@@
     (effects (font (size 1.27 1.27)) (justify left bottom))
   )
-  (text "Precision rectifier" (at 185.42 21.59 0)
+  (text "Precision rectifier" (at 194.31 22.86 0)
     (effects (font (size 1.27 1.27)) (justify left bottom))
   )
@@
     (effects (font (size 1.27 1.27)) (justify left bottom))
   )
+  (text "Place this isolation\nresistors as close to\nthe audio signal\nas possible."
+    (at 173.99 101.6 0)
+    (effects (font (size 1.27 1.27)) (justify left bottom))
+  )
   (text "1.74V     clipping\n870mV   -6dB\n435mV  -12dB\n218mV  -18dB"
     (at 205.74 57.15 0)
     (effects (font (size 1.27 1.27)) (justify left bottom))
   )
-  (text "Add 0R resistors to be able to change some settings?\n-Sample freq\n-bits"
+  (text "Add 0R resistors to be able to change some settings?\n-Sample freq->OSRX\n-bits->OSRX"
     (at 401.32 114.3 0)
     (effects (font (size 1.27 1.27) (color 200 0 200 1)) (justify left bottom))
@@
     (effects (font (size 1.27 1.27)) (justify left bottom))
   )
-  (text "Precision rectifier" (at 185.42 101.6 0)
+  (text "Precision rectifier" (at 194.31 102.87 0)
     (effects (font (size 1.27 1.27)) (justify left bottom))
   )
@@
     (effects (font (size 1.27 1.27)) (justify left bottom))
   )
+  (text "Place this isolation\nresistors as close to\nthe audio signal\nas possible."
+    (at 168.91 55.88 0)
+    (effects (font (size 1.27 1.27)) (justify left bottom))
+  )
   (text "RST inactive" (at 431.8 88.265 0)
     (effects (font (size 1.27 1.27)) (justify left bottom))
@@
     (effects (font (size 1.27 1.27)) (justify right))
   )
-  (hierarchical_label "SCKI_ADC_CH1_2" (shape output) (at 433.07 69.85 0) (fields_autoplaced)
+  (hierarchical_label "SCKI_ADC_CH1_2" (shape input) (at 433.07 69.85 0) (fields_autoplaced)
     (effects (font (size 1.27 1.27)) (justify left))
   )
@@
       (effects (font (size 1.27 1.27)))
     )
-    (property "Value" "270" (at 318.77 143.51 90)
+    (property "Value" "2k7" (at 318.77 143.51 90)
       (effects (font (size 1.27 1.27)))
     )
@@
       (effects (font (size 1.27 1.27)))
     )
-    (property "Value" "270" (at 318.77 19.05 90)
+    (property "Value" "2k7" (at 318.77 19.05 90)
       (effects (font (size 1.27 1.27)))
     )
@@
       (effects (font (size 1.27 1.27)))
     )
-    (property "Value" "270" (at 318.77 99.06 90)
+    (property "Value" "2k7" (at 318.77 99.06 90)
       (effects (font (size 1.27 1.27)))
     )
@@
       (effects (font (size 1.27 1.27)))
     )
-    (property "Value" "270" (at 318.77 63.5 90)
+    (property "Value" "2k7" (at 318.77 63.5 90)
       (effects (font (size 1.27 1.27)))
     )
