File: KiCAD/Main board/ADC_CH1_2.kicad_sch (KiCad schematic)
At the start: 148 parts, among them K1 EA2-12NU, K2 EA2-12NU, Q1 BC847, Q2 BC847, Q3 BC847, Q4 BC857, U24 LM4562, U25 OPA1632DR, U34 TL072, U35 TL072, U36 LM339, U38 PGA2311P, U39 TXS0102, U4 OPA1632DR, U5 OPA1632DR, U6 LM4562, U7 PCM1804

Commit message: Main board
Other:
- note added: "MISSING"
- note added: "Start-up circuitry"
Changed lines of the file:
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@@
     (effects (font (size 1.27 1.27)) (justify left bottom))
   )
+  (text "MISSING" (at 265.43 46.99 0)
+    (effects (font (size 1.27 1.27) (thickness 0.254) bold (color 200 0 200 1)) (justify left bottom))
+  )
   (text "INPUT_SELECTOR_RELAY\nLOW=RCA\nHIGH-Jack" (at 132.08 43.18 0)
     (effects (font (size 1.27 1.27)) (justify left bottom))
@@
     (effects (font (size 1.27 1.27)) (justify left bottom))
   )
+  (text "MISSING" (at 265.43 143.51 0)
+    (effects (font (size 1.27 1.27) (thickness 0.254) bold (color 200 0 200 1)) (justify left bottom))
+  )
   (text "These resistors make it\nfairly easy to change\nthe mode of the ADC in\ncase this is needed to\ncomply with the firmware.\nThe resistors can be\ndesoldered and the OSRx\npins can be connected\nwith a wire to GND."
     (at 424.18 125.73 0)
     (effects (font (size 1.27 1.27)) (justify left bottom))
   )
+  (text "MISSING" (at 265.43 158.75 0)
+    (effects (font (size 1.27 1.27) (thickness 0.254) bold (color 200 0 200 1)) (justify left bottom))
+  )
   (text "Unmuted" (at 137.16 100.965 0)
     (effects (font (size 1.27 1.27)) (justify left bottom))
@@
     (effects (font (size 1.27 1.27)) (justify left bottom))
   )
+  (text "MISSING" (at 265.43 31.75 0)
+    (effects (font (size 1.27 1.27) (thickness 0.254) bold (color 200 0 200 1)) (justify left bottom))
+  )
+  (text "MISSING" (at 265.43 128.27 0)
+    (effects (font (size 1.27 1.27) (thickness 0.254) bold (color 200 0 200 1)) (justify left bottom))
+  )
   (text "Precision rectifier" (at 194.31 102.87 0)
     (effects (font (size 1.27 1.27)) (justify left bottom))
@@
     (effects (font (size 1.27 1.27)) (justify left bottom))
   )
+  (text "MISSING" (at 265.43 62.23 0)
+    (effects (font (size 1.27 1.27) (thickness 0.254) bold (color 200 0 200 1)) (justify left bottom))
+  )
+  (text "Start-up circuitry" (at 170.18 129.54 0)
+    (effects (font (size 1.27 1.27)) (justify left bottom))
+  )
   (text "Place this isolation\nresistors as close to\nthe audio signal\nas possible."
     (at 168.91 55.88 0)
@@
     (effects (font (size 1.27 1.27)) (justify left bottom))
   )
+  (text "MISSING" (at 265.43 111.76 0)
+    (effects (font (size 1.27 1.27) (thickness 0.254) bold (color 200 0 200 1)) (justify left bottom))
+  )
   (text "Master mode" (at 427.99 98.425 0)
     (effects (font (size 1.27 1.27)) (justify left bottom))
@@
     (effects (font (size 1.27 1.27)) (justify left bottom))
   )
+  (text "MISSING" (at 265.43 77.47 0)
+    (effects (font (size 1.27 1.27) (thickness 0.254) bold (color 200 0 200 1)) (justify left bottom))
+  )
   (label "AGND_CH1" (at 288.29 63.5 0) (fields_autoplaced)
     (effects (font (size 1.27 1.27)) (justify left bottom))
@@
       (effects (font (size 1.27 1.27)) hide)
     )
-    (property "Datasheet" "~" (at 226.06 116.84 0)
+    (property "Datasheet" "https://nl.mouser.com/ProductDetail/Bourns/CR0805-FX-3901ELF?qs=sGAEpiMZZMvdGkrng054t%252BRNGJdg958R%2FWTvjoxzCb0%3D" (at 226.06 116.84 0)
       (effects (font (size 1.27 1.27)) hide)
     )
@@
       (effects (font (size 1.27 1.27) italic) (justify left) hide)
     )
-    (property "Datasheet" "https://www.onsemi.com/pub/Collateral/BC860-D.pdf" (at 170.18 138.43 0)
+    (property "Datasheet" "https://nl.mouser.com/ProductDetail/Micro-Commercial-Components-MCC/BC857B-TP?qs=SdqRYZZ9IxCYF9uJ91hYQg%3D%3D" (at 170.18 138.43 0)
       (effects (font (size 1.27 1.27)) (justify left) hide)
     )
@@
       (effects (font (size 1.27 1.27)) hide)
     )
-    (property "Datasheet" "~" (at 248.92 21.59 0)
+    (property "Datasheet" "https://nl.mouser.com/ProductDetail/YAGEO/RC0805JR-0724KL?qs=sGAEpiMZZMvdGkrng054txdMlaQGj9fixvNEN4DCZoA%3D" (at 248.92 21.59 0)
       (effects (font (size 1.27 1.27)) hide)
     )
@@
       (effects (font (size 1.27 1.27)) hide)
     )
-    (property "Datasheet" "~" (at 226.06 52.07 0)
+    (property "Datasheet" "https://nl.mouser.com/ProductDetail/Bourns/CR0805-FX-2001ELF?qs=sGAEpiMZZMvdGkrng054t%252BRNGJdg958ROajZ6ouhRE4%3D" (at 226.06 52.07 0)
       (effects (font (size 1.27 1.27)) hide)
     )
@@
       (effects (font (size 1.27 1.27) italic) (justify left) hide)
     )
-    (property "Datasheet" "" (at 191.77 143.51 0)
+    (property "Datasheet" "https://nl.mouser.com/ProductDetail/Nexperia/BC847C215?qs=me8TqzrmIYVnv3C18%2Fxa3Q%3D%3D" (at 191.77 143.51 0)
       (effects (font (size 1.27 1.27)) (justify left) hide)
     )
@@
       (effects (font (size 1.27 1.27)) hide)
     )
-    (property "Datasheet" "~" (at 226.06 132.08 0)
+    (property "Datasheet" "https://nl.mouser.com/ProductDetail/Bourns/CR0805-FX-2001ELF?qs=sGAEpiMZZMvdGkrng054t%252BRNGJdg958ROajZ6ouhRE4%3D" (at 226.06 132.08 0)
       (effects (font (size 1.27 1.27)) hide)
     )
@@
       (effects (font (size 1.27 1.27) italic) (justify left) hide)
     )
-    (property "Datasheet" "" (at 116.84 46.99 0)
+    (property "Datasheet" "https://nl.mouser.com/ProductDetail/Nexperia/BC847C215?qs=me8TqzrmIYVnv3C18%2Fxa3Q%3D%3D" (at 116.84 46.99 0)
       (effects (font (size 1.27 1.27)) (justify left) hide)
     )
@@
       (effects (font (size 1.27 1.27)) hide)
     )
-    (property "Datasheet" "~" (at 226.06 36.83 0)
+    (property "Datasheet" "https://nl.mouser.com/ProductDetail/Bourns/CR0805-FX-3901ELF?qs=sGAEpiMZZMvdGkrng054t%252BRNGJdg958R%2FWTvjoxzCb0%3D" (at 226.06 36.83 0)
       (effects (font (size 1.27 1.27)) hide)
     )
@@
       (effects (font (size 1.27 1.27) italic) (justify left) hide)
     )
-    (property "Datasheet" "" (at 54.61 46.99 0)
+    (property "Datasheet" "https://nl.mouser.com/ProductDetail/Nexperia/BC847C215?qs=me8TqzrmIYVnv3C18%2Fxa3Q%3D%3D" (at 54.61 46.99 0)
       (effects (font (size 1.27 1.27)) (justify left) hide)
     )
@@
       (effects (font (size 1.27 1.27)) hide)
     )
-    (property "Datasheet" "~" (at 248.92 101.6 0)
+    (property "Datasheet" "https://nl.mouser.com/ProductDetail/YAGEO/RC0805JR-0724KL?qs=sGAEpiMZZMvdGkrng054txdMlaQGj9fixvNEN4DCZoA%3D" (at 248.92 101.6 0)
       (effects (font (size 1.27 1.27)) hide)
     )
