File: KiCAD/Main board/DAC_CH1_2.kicad_sch (KiCad schematic)
At the start: 73 parts, among them U1 LM4562, U1 PCM1789-Q1, U3 OPA1632DR, U4 OPA1632DR

Commit message: Worked a bit on the main board
Parts:
- removed R1 (x4): 22R, Resistor_SMD:R_0805_2012Metric, symbol Device:R
- removed U1: PCM1789-Q1, Package_SO:TSSOP-24_4.4x7.8mm_P0.65mm, symbol Audio-DSP:PCM1789-Q1
- added NT1, NT2: NetTie_2, NetTie:NetTie-2_SMD_Pad0.5mm, symbol Device:NetTie_2
- added R200: 22R, Resistor_SMD:R_Array_Convex_2x0402, symbol Device:R_Pack02
- added R3: 22R, Resistor_SMD:R_Array_Convex_4x0402, symbol Device:R_Pack04
- added U1: PCM1789, Package_SO:TSSOP-24_4.4x7.8mm_P0.65mm, symbol Audio-DSP:PCM1789
- C15, C16, C19, C2, C21, C25, C26, C3, C35: footprint Capacitor_SMD:C_0805_2012Metric -> Capacitor_SMD:C_0402_1005Metric
Connections:
- net +3.3V: now also U1.6 (VDD)
- net GND: now also NT1.1, NT2.1, U1.10 (AGND1), U1.15 (AGND2), U1.20 (MODE), U1.23 (MS/ADR0/RSV), U1.24 (ADR5/ADR1/RSV), U1.7 (DGND); no longer C14.2, C8.2, R28.2, R9.2
- net at C1.1, C3.1, R34.1: now also U1.16 (VCC2)
- net at R12.1, R6.1: now also U1.12 (VOUTL+)
- net at R16.1, R5.2: now also U1.11 (VOUTL-)
- net at R19.1, R20.1: now also U1.13 (VOUTR+)
- net at R18.2, R21.1: now also U1.14 (VOUTR-)
- net at C2.1, C5.1, R33.1: now also U1.8 (VCC1)
- net RCA JACK CH1 renamed RCA_JACK_CH1(+)
- net RCA JACK CH2 renamed RCA_JACK_CH2(+)
- net VOUT CH1(+) renamed VOUT_CH1(+)
- net VOUT CH1(-) renamed VOUT_CH1(-)
- net VOUT CH2(+) renamed VOUT_CH2(+)
- net VOUT CH2(-) renamed VOUT_CH2(-)
- new net: R3.5 (R4.2), U1.5 (SCKI)
- new net: R3.6 (R3.2), U1.3 (DIN)
- new net: R3.7 (R2.2), U1.2 (BCK)
- new net: R3.8 (R1.2), U1.1 (LRCK)
- new net: R200.3 (R2.2), U1.22 (MC/SCL/FMT)
- new net: R200.4 (R1.2), U1.21 (MD/SDA/DEMP)
- new net AMUTEI_CH1_2: U1.17 (AMUTEI)
- new net BCK_CH1_2: R3.2 (R2.1)
- new net DIN_CH1_2: R3.3 (R3.1)
- new net LRCK_CH1_2: R3.1 (R1.1)
- new net RCA_JACK_CH1(REF): C8.2, NT1.2, R9.2
- new net RCA_JACK_CH2(REF): C14.2, NT2.2, R28.2
- new net RST_CH1_2: U1.4 (RST)
- new net SCKI_CH1_2: R3.4 (R4.1)
- new net SCL_CH1_2: R200.2 (R2.1)
- new net SDA_CH1_2: R200.1 (R1.1)
Other:
- note added: "Location? FPGA/IC?"
- note added: "Update to 0.3mm"
- note removed: "-Below -Update capacitor values -Make it a bit more tidy -Update components text placment and rotation"
- note removed: "Decoupling capacitors (100nF and 22uF)(power supply) -100nF X7R ceremic capacitor-> 0805 mabye we change it to 0402 later -22uF TH electrolytic"
- note removed: "Filter capacitors for with small capacitance -Type C0G - NP0 -Footprint 0805 (mabye we change it to 0402 later)"

Commit message: Worked on main board
Parts:
- removed U3, U4: OPA1632DR, Audio_DSP:VSSOP-8_3.0x3.0mm_P0.65_TP1.8x1.5, symbol Audio-DSP:OPA1632DR
- added U3, U4: OPA1632DR, Audio-DSP:VSSOP-8_3.0x3.0mm_P0.65_TP1.8x1.5, symbol Audio_DSP:OPA1632DR
Connections:
- net GND: now also U3.2 (VOCM), U3.7 (ENABLE), U3.9 (GND), U4.2 (VOCM), U4.7 (ENABLE), U4.9 (GND)
- net at C11.1, R16.2, R17.1: now also U3.1 (VIN-)
- net at C18.1, R21.2, R23.1: now also U4.1 (VIN-)
- net at C25.1, C28.1, R36.1: now also U4.3 (V+)
- net at C16.2, C24.2, R35.2: now also U3.6 (V-)
- net at C10.1, R12.2, R13.1: now also U3.8 (VIN+)
- net at C18.2, R37.1: now also U4.4 (VOUT+)
- net at C15.1, C23.1, R24.1: now also U3.3 (V+)
- net at C17.1, R20.2, R22.1: now also U4.8 (VIN+)
- net at C17.2, R30.1: now also U4.5 (VOUT-)
- net at C10.2, R14.1: now also U3.5 (VOUT-)
- net at C26.2, C30.2, R38.2: now also U4.6 (V-)
- net at C11.2, R15.1: now also U3.4 (VOUT+)

Commit message: Worked on main board
Parts:
- removed C35: 100n, Capacitor_SMD:C_0402_1005Metric, symbol Device:C
- removed R200: 22R, Resistor_SMD:R_Array_Convex_2x0402, symbol Device:R_Pack02
- removed R36, R38: 10, Resistor_SMD:R_0805_2012Metric, symbol Device:R
- removed U1: PCM1789, Package_SO:TSSOP-24_4.4x7.8mm_P0.65mm, symbol Audio-DSP:PCM1789
- added C110: 100n, Capacitor_SMD:C_0402_1005Metric, symbol Device:C
- added R1, R2: 10R, Resistor_SMD:R_0805_2012Metric, symbol Device:R
- added R4: 22R, Resistor_SMD:R_Array_Convex_4x0402, symbol Device:R_Pack04
- added U1: PCM1789, Package_SO:TSSOP-24_4.4x7.8mm_P0.65mm, symbol Audio_DSP:PCM1789
- C15, C16, C21, C25, C26: value 100nF -> 100n
- C19: value 100n -> 1n5
- C7, C8: footprint Capacitor_SMD:C_0805_2012Metric -> Capacitor_SMD:C_0402_1005Metric
- C9: value 1n5 -> 100n; footprint Capacitor_SMD:C_0805_2012Metric -> Capacitor_SMD:C_0402_1005Metric
- R24, R31, R32, R33, R34, R35: value 10 -> 10R
Connections:
- net +12V: now also R24.1, R32.1, R1.1; no longer R24.2, R32.2
- net +3.3V: now also C110.1, U1.4 (RST), U1.6 (VDD); no longer C19.1
- net +5V: now also R33.1, R34.1; no longer R33.2, R34.2
- net -12V: now also R31.2, R35.2, R2.2; no longer R31.1, R35.1
- net AMUTEI_CH1_2: now also R4.1 (R1.1)
- net GND: now also C9.2, C110.2, U1.10 (AGND1), U1.15 (AGND2), U1.20 (MODE), U1.23 (MS/ADR0/RSV), U1.24 (ADR5/ADR1/RSV), U1.7 (DGND); no longer C19.2
- net SCL_CH1_2: now also R4.3 (R3.1)
- net SDA_CH1_2: now also R4.2 (R2.1)
- net at R3.5 (R4.2): now also U1.5 (SCKI)
- net at R3.6 (R3.2): now also U1.3 (DIN)
- net at R3.7 (R2.2): now also U1.2 (BCK)
- net at R3.8 (R1.2): now also U1.1 (LRCK)
- net at C1.1, C3.1: now also R34.2, U1.16 (VCC2); no longer R34.1
- net at R12.1, R6.1: now also U1.12 (VOUTL+)
- net at C4.1, U1.8 (V+): now also C9.1, R1.2; no longer R32.1
- net at C25.1, C28.1, U4.3 (V+): now also R32.2
- net at C2.1, C5.1: now also R33.2, U1.8 (VCC1); no longer R33.1
- net at C16.2, C24.2, U3.6 (V-): now also R31.1; no longer R35.2
- net at R7.2, U1.3 (+): now also C19.1; no longer C9.1
- net at C15.1, C23.1, U3.3 (V+): now also R24.2; no longer R24.1
- net at R10.1, R11.2, U1.1: now also C19.2; no longer C9.2
- net at R16.1, R5.2: now also U1.11 (VOUTL-)
- net at C21.2, C22.2, U1.4 (V-): now also R2.1; no longer R31.2
- net at C26.2, C30.2, U4.6 (V-): now also R35.1
- net at R19.1, R20.1: now also U1.13 (VOUTR+)
- net at R18.2, R21.1: now also U1.14 (VOUTR-)
- new net: R4.6 (R3.2), U1.22 (MC/SCL/FMT)
- new net: R4.7 (R2.2), U1.21 (MD/SDA/DEMP)
- new net: R4.8 (R1.2), U1.17 (AMUTEI)
- no-connect marks 3 -> 5
Other:
- note added: "Place nettie at output connector"
- moved on the sheet: C1, C5, NT1, R10, R11, R7, R8, R9, U1A

Commit message: Worked on main board
Other:
- moved on the sheet: C19, C8, NT1, R10, R11, R9

Commit message: Worked on main board
Parts:
- renumbered C9 to C1, C23 to C10, C24 to C11, C3 to C12, C5 to C13, C1 to C14, C25 to C15, C26 to C16, C7 to C17, C6 to C18, C28 to C19, C21 to C2, C30 to C20, C19 to C21, C8 to C22, C13 to C23, C14 to C24, C10 to C25, C11 to C26, C17 to C27, C18 to C28, C12 to C29, C4 to C3, C27 to C30, C22 to C4, C20 to C5, C110 to C6, C15 to C7, C16 to C8, C2 to C9, R6 to R10, R12 to R11, R16 to R12, R18 to R13, R19 to R14, R20 to R15, R21 to R16, R13 to R17, R17 to R18, R22 to R19, R23 to R20, R25 to R21, R26 to R22, R7 to R23, R8 to R24, R11 to R25, R9 to R26, R10 to R29, R24 to R3, R29 to R30, R14 to R31, R15 to R32, R30 to R33, R37 to R34, R31 to R4, R33 to R5, R32 to R6, R35 to R7, R34 to R8, R5 to R9, R3 to RN1, R4 to RN2

Commit message: Worked on main board
Parts:
- removed U3, U4: OPA1632DR, Audio-DSP:VSSOP-8_3.0x3.0mm_P0.65_TP1.8x1.5, symbol Audio_DSP:OPA1632DR
- added U3, U4: OPA1632DR, Audio-DSP:VSSOP-8_3.0x3.0mm_P0.65_TP1.8x1.5, symbol Audio-DSP:OPA1632DR
Connections:
- net GND: now also U3.2 (VOCM), U3.7 (ENABLE), U3.9 (GND), U4.2 (VOCM), U4.7 (ENABLE), U4.9 (GND)
- net at C28.1, R16.2, R20.1: now also U4.1 (VIN-)
- net at C28.2, R34.1: now also U4.4 (VOUT+)
- net at C27.2, R33.1: now also U4.5 (VOUT-)
- net at C27.1, R15.2, R19.1: now also U4.8 (VIN+)
- net at C26.1, R12.2, R18.1: now also U3.1 (VIN-)
- net at C15.1, C19.1, R6.2: now also U4.3 (V+)
- net at C11.2, C8.2, R4.1: now also U3.6 (V-)
- net at C25.1, R11.2, R17.1: now also U3.8 (VIN+)
- net at C10.1, C7.1, R3.2: now also U3.3 (V+)
- net at C25.2, R31.1: now also U3.5 (VOUT-)
- net at C26.2, R32.1: now also U3.4 (VOUT+)
- net at C16.2, C20.2, R7.1: now also U4.6 (V-)
