File: KiCAD/Main board/DAC_CH1_2.kicad_sch (KiCad schematic)
At the start: 73 parts, among them U1 LM4562, U1 PCM1789, U3 OPA1632DR, U4 OPA1632DR

Commit message: Main board, ordering of PCBs and LTspice simulations
Parts:
- C17, C18, C21, C22: footprint Capacitor_SMD:C_0402_1005Metric -> Capacitor_SMD:C_0805_2012Metric
Changed lines of the file:
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@@
       (effects (font (size 1.27 1.27)))
     )
-    (property "Footprint" "Capacitor_SMD:C_0402_1005Metric" (at 156.21 23.1648 0)
+    (property "Footprint" "Capacitor_SMD:C_0805_2012Metric" (at 156.21 23.1648 0)
       (effects (font (size 1.27 1.27)) hide)
     )
@@
       (effects (font (size 1.27 1.27)) (justify left))
     )
-    (property "Footprint" "Capacitor_SMD:C_0402_1005Metric" (at 134.3152 36.83 0)
+    (property "Footprint" "Capacitor_SMD:C_0805_2012Metric" (at 134.3152 36.83 0)
       (effects (font (size 1.27 1.27)) hide)
     )
@@
       (effects (font (size 1.27 1.27)) (justify left))
     )
-    (property "Footprint" "Capacitor_SMD:C_0402_1005Metric" (at 134.3152 132.08 0)
+    (property "Footprint" "Capacitor_SMD:C_0805_2012Metric" (at 134.3152 132.08 0)
       (effects (font (size 1.27 1.27)) hide)
     )
@@
       (effects (font (size 1.27 1.27)))
     )
-    (property "Footprint" "Capacitor_SMD:C_0402_1005Metric" (at 156.21 43.4848 0)
-      (effects (font (size 1.27 1.27)) hide)
-    )
+    (property "Footprint" "Capacitor_SMD:C_0805_2012Metric" (at 156.21 43.4848 0)
+      (effects (font (size 1.27 1.27)) hide)
+    )
