File: KiCAD/Main board/ADC_CH3_4.kicad_sch (KiCad schematic)
At the start: 44 parts, among them U14 LM4562, U17 LM4562, U5 OPA1632DR

Commit message: Worked on the main board
Parts:
- added U27: PCM1804, Package_SO:SSOP-28_5.3x10.2mm_P0.65mm, symbol Audio-DSP:PCM1804
Changed lines of the file:
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@@
 (kicad_sch (version 20230121) (generator eeschema)
-  (paper "A4")
+  (paper "A3")
   (junction (at 69.85 97.79) (diameter 0) (color 0 0 0 0)
   )
@@
         )
       )
+    )
+  )
+  (symbol (lib_id "Audio-DSP:PCM1804") (at 224.79 72.39 0) (unit 1)
+    (in_bom yes) (on_board yes) (dnp no) (fields_autoplaced)
+    (property "Reference" "U27" (at 229.2859 48.26 0)
+      (effects (font (size 1.27 1.27)) (justify left))
+    )
+    (property "Value" "PCM1804" (at 229.2859 50.8 0)
+      (effects (font (size 1.27 1.27)) (justify left))
+    )
+    (property "Footprint" "Package_SO:SSOP-28_5.3x10.2mm_P0.65mm" (at 191.77 104.14 0)
+      (effects (font (size 1.27 1.27)) (justify left) hide)
+    )
+    (property "Datasheet" "https://nl.mouser.com/ProductDetail/Texas-Instruments/PCM1804DBR?qs=wgAEGBTxy7lnBW3YYZcxMA%3D%3D" (at 191.77 106.68 0)
+      (effects (font (size 1.27 1.27)) (justify left) hide)
+    )
+    (pin "1")
+    (pin "10")
+    (pin "11")
+    (pin "12")
+    (pin "13")
+    (pin "14")
+    (pin "15")
+    (pin "16")
+    (pin "17")
+    (pin "18")
+    (pin "19")
+    (pin "2")
+    (pin "20")
+    (pin "21")
+    (pin "22")
+    (pin "23")
+    (pin "24")
+    (pin "25")
+    (pin "26")
+    (pin "27")
+    (pin "28")
+    (pin "3")
+    (pin "4")
+    (pin "5")
+    (pin "6")
+    (pin "7")
+    (pin "8")
+    (pin "9")
+    (instances
+      (project "Main board"
+        (path "/2f8cbac6-fd11-4240-8e40-3bb6952a0324/b7530516-5ab1-4afa-9366-b30c4f029458"
+          (reference "U27") (unit 1)
+        )
+      )

Commit message: Worked on main board
Parts:
- U8: renamed from U5; now in the parts list
- renumbered C97 to C49, R114 to R53, R115 to R55, R103 to R56, R116 to R59, R117 to R60, R105 to R61, R118 to R63, U17 to U10, U14 to U10, U27 to U11, U14 to U9, U17 to U9

Commit message: fixed symbols excluding from board
Parts:
- C10, C11, C12, C21, C25, C26, C35: footprint Capacitor_SMD:C_0805_2012Metric -> (none)
- C22, C28, C30, C4: footprint Capacitor_THT:CP_Radial_D5.0mm_P2.00mm -> (none)
- R12, R13, R14, R15, R31, R32, R36, R38: footprint Resistor_SMD:R_0805_2012Metric -> (none)
Changed lines of the file:
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@@
       (effects (font (size 1.27 1.27)) (justify left))
     )
-    (property "Footprint" "Capacitor_THT:CP_Radial_D5.0mm_P2.00mm" (at 154.6352 181.61 0)
+    (property "Footprint" "" (at 154.6352 181.61 0)
       (effects (font (size 1.27 1.27)) hide)
     )
@@
       (effects (font (size 1.27 1.27)))
     )
-    (property "Footprint" "Resistor_SMD:R_0805_2012Metric" (at 131.318 162.56 90)
+    (property "Footprint" "" (at 131.318 162.56 90)
       (effects (font (size 1.27 1.27)) hide)
     )
@@
       (effects (font (size 1.27 1.27)) (justify left))
     )
-    (property "Footprint" "Capacitor_SMD:C_0805_2012Metric" (at 143.2052 173.99 0)
+    (property "Footprint" "" (at 143.2052 173.99 0)
       (effects (font (size 1.27 1.27)) hide)
     )
@@
       (effects (font (size 1.27 1.27)) (justify left))
     )
-    (property "Footprint" "Capacitor_THT:CP_Radial_D5.0mm_P2.00mm" (at 102.5652 175.26 0)
+    (property "Footprint" "" (at 102.5652 175.26 0)
       (effects (font (size 1.27 1.27)) hide)
     )
@@
       (effects (font (size 1.27 1.27)))
     )
-    (property "Footprint" "Resistor_SMD:R_0805_2012Metric" (at 18.288 185.42 90)
+    (property "Footprint" "" (at 18.288 185.42 90)
       (effects (font (size 1.27 1.27)) hide)
     )
@@
       (effects (font (size 1.27 1.27)))
     )
-    (property "Footprint" "Resistor_SMD:R_0805_2012Metric" (at 131.318 185.42 90)
+    (property "Footprint" "" (at 131.318 185.42 90)
       (effects (font (size 1.27 1.27)) hide)
     )
@@
       (effects (font (size 1.27 1.27)))
     )
-    (property "Footprint" "Resistor_SMD:R_0805_2012Metric" (at 165.1 95.758 90)
+    (property "Footprint" "" (at 165.1 95.758 90)
       (effects (font (size 1.27 1.27)) hide)
     )
@@
       (effects (font (size 1.27 1.27)))
     )
-    (property "Footprint" "Resistor_SMD:R_0805_2012Metric" (at 18.288 162.56 90)
+    (property "Footprint" "" (at 18.288 162.56 90)
       (effects (font (size 1.27 1.27)) hide)
     )
@@
       (effects (font (size 1.27 1.27)))
     )
-    (property "Footprint" "Capacitor_SMD:C_0805_2012Metric" (at 35.2552 181.61 0)
+    (property "Footprint" "" (at 35.2552 181.61 0)
       (effects (font (size 1.27 1.27)) hide)
     )
@@
       (effects (font (size 1.27 1.27)))
     )
-    (property "Footprint" "Capacitor_SMD:C_0805_2012Metric" (at 157.48 100.6348 0)
+    (property "Footprint" "" (at 157.48 100.6348 0)
       (effects (font (size 1.27 1.27)) hide)
     )
@@
       (effects (font (size 1.27 1.27)))
     )
-    (property "Footprint" "Capacitor_SMD:C_0805_2012Metric" (at 143.2052 181.61 0)
+    (property "Footprint" "" (at 143.2052 181.61 0)
       (effects (font (size 1.27 1.27)) hide)
     )
@@
       (effects (font (size 1.27 1.27)))
     )
-    (property "Footprint" "Resistor_SMD:R_0805_2012Metric" (at 119.38 64.008 90)
+    (property "Footprint" "" (at 119.38 64.008 90)
       (effects (font (size 1.27 1.27)) hide)
     )
@@
       (effects (font (size 1.27 1.27)) (justify left))
     )
-    (property "Footprint" "Capacitor_SMD:C_0805_2012Metric" (at 177.4952 86.36 0)
+    (property "Footprint" "" (at 177.4952 86.36 0)
       (effects (font (size 1.27 1.27)) hide)
     )
@@
       (effects (font (size 1.27 1.27)) (justify left))
     )
-    (property "Footprint" "Capacitor_THT:CP_Radial_D5.0mm_P2.00mm" (at 154.6352 173.99 0)
+    (property "Footprint" "" (at 154.6352 173.99 0)
       (effects (font (size 1.27 1.27)) hide)
     )
@@
       (effects (font (size 1.27 1.27)))
     )
-    (property "Footprint" "Resistor_SMD:R_0805_2012Metric" (at 165.1 75.438 90)
+    (property "Footprint" "" (at 165.1 75.438 90)
       (effects (font (size 1.27 1.27)) hide)
     )
@@
       (effects (font (size 1.27 1.27)) (justify left))
     )
-    (property "Footprint" "Capacitor_THT:CP_Radial_D5.0mm_P2.00mm" (at 46.6852 181.61 0)
+    (property "Footprint" "" (at 46.6852 181.61 0)
       (effects (font (size 1.27 1.27)) hide)
     )
@@
       (effects (font (size 1.27 1.27)))
     )
-    (property "Footprint" "Capacitor_SMD:C_0805_2012Metric" (at 157.48 66.3448 0)
+    (property "Footprint" "" (at 157.48 66.3448 0)
       (effects (font (size 1.27 1.27)) hide)
     )
@@
       (effects (font (size 1.27 1.27)) (justify left))
     )
-    (property "Footprint" "Capacitor_THT:CP_Radial_D5.0mm_P2.00mm" (at 46.6852 173.99 0)
+    (property "Footprint" "" (at 46.6852 173.99 0)
       (effects (font (size 1.27 1.27)) hide)
     )
@@
       (effects (font (size 1.27 1.27)))
     )
-    (property "Footprint" "Capacitor_SMD:C_0805_2012Metric" (at 35.2552 173.99 0)
+    (property "Footprint" "" (at 35.2552 173.99 0)
       (effects (font (size 1.27 1.27)) hide)
     )
@@
       (effects (font (size 1.27 1.27)) (justify left))
     )
-    (property "Footprint" "Capacitor_THT:CP_Radial_D5.0mm_P2.00mm" (at 102.5652 182.88 0)
+    (property "Footprint" "" (at 102.5652 182.88 0)
       (effects (font (size 1.27 1.27)) hide)
     )
@@
       (effects (font (size 1.27 1.27)))
     )
-    (property "Footprint" "Capacitor_SMD:C_0805_2012Metric" (at 91.1352 182.88 0)
+    (property "Footprint" "" (at 91.1352 182.88 0)
       (effects (font (size 1.27 1.27)) hide)
     )
@@
       (effects (font (size 1.27 1.27)))
     )
-    (property "Footprint" "Resistor_SMD:R_0805_2012Metric" (at 79.248 186.69 90)
+    (property "Footprint" "" (at 79.248 186.69 90)
       (effects (font (size 1.27 1.27)) hide)
     )
@@
       (effects (font (size 1.27 1.27)))
     )
-    (property "Footprint" "Resistor_SMD:R_0805_2012Metric" (at 79.248 163.83 90)
+    (property "Footprint" "" (at 79.248 163.83 90)
       (effects (font (size 1.27 1.27)) hide)
     )
@@
       (effects (font (size 1.27 1.27)))
     )
-    (property "Footprint" "Resistor_SMD:R_0805_2012Metric" (at 132.08 64.008 90)
+    (property "Footprint" "" (at 132.08 64.008 90)
       (effects (font (size 1.27 1.27)) hide)
     )
@@
       (effects (font (size 1.27 1.27)) (justify left))
     )
-    (property "Footprint" "Capacitor_SMD:C_0805_2012Metric" (at 91.1352 175.26 0)
-      (effects (font (size 1.27 1.27)) hide)
-    )
+    (property "Footprint" "" (at 91.1352 175.26 0)
+      (effects (font (size 1.27 1.27)) hide)
+    )
