File: KiCAD/Main board/ADC_CH3_4.kicad_sch (KiCad schematic)
At the start: 45 parts, among them U24 LM4562, U4 OPA1632DR, U6 LM4562

Commit message: Worked on main board design
Parts:
- added D4: D_TVS, symbol Device:D_TVS
Other:
- note added: "Niet leverbaar!"
Changed lines of the file:
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@@
   (junction (at 201.93 113.03) (diameter 0) (color 0 0 0 0)
   )
+  (junction (at 238.76 195.58) (diameter 0) (color 0 0 0 0)
+  )
+  (junction (at 203.2 161.29) (diameter 0) (color 0 0 0 0)
+  )
+  (junction (at 165.1 153.67) (diameter 0) (color 0 0 0 0)
+  )
+  (junction (at 190.5 200.66) (diameter 0) (color 0 0 0 0)
+  )
+  (junction (at 219.71 190.5) (diameter 0) (color 0 0 0 0)
+  )
+  (junction (at 232.41 209.55) (diameter 0) (color 0 0 0 0)
+  )
+  (junction (at 163.83 120.65) (diameter 0) (color 0 0 0 0)
+  )
+  (junction (at 250.19 212.09) (diameter 0) (color 0 0 0 0)
+  )
+  (junction (at 153.67 120.65) (diameter 0) (color 0 0 0 0)
+  )
+  (junction (at 189.23 73.66) (diameter 0) (color 0 0 0 0)
+  )
+  (junction (at 201.93 118.11) (diameter 0) (color 0 0 0 0)
+  )
+  (junction (at 172.72 81.28) (diameter 0) (color 0 0 0 0)
+  )
+  (junction (at 153.67 93.98) (diameter 0) (color 0 0 0 0)
+  )
+  (junction (at 153.67 71.12) (diameter 0) (color 0 0 0 0)
+  )
+  (junction (at 237.49 78.74) (diameter 0) (color 0 0 0 0)
+  )
+  (junction (at 248.92 195.58) (diameter 0) (color 0 0 0 0)
+  )
+  (junction (at 163.83 71.12) (diameter 0) (color 0 0 0 0)
+  )
+  (junction (at 154.94 153.67) (diameter 0) (color 0 0 0 0)
+  )
+  (junction (at 189.23 118.11) (diameter 0) (color 0 0 0 0)
+  )
+  (junction (at 237.49 113.03) (diameter 0) (color 0 0 0 0)
+  )
+  (junction (at 203.2 200.66) (diameter 0) (color 0 0 0 0)
+  )
+  (junction (at 172.72 110.49) (diameter 0) (color 0 0 0 0)
+  )
+  (junction (at 248.92 129.54) (diameter 0) (color 0 0 0 0)
+  )
   (junction (at 154.94 203.2) (diameter 0) (color 0 0 0 0)
   )
-  (junction (at 238.76 195.58) (diameter 0) (color 0 0 0 0)
-  )
-  (junction (at 203.2 161.29) (diameter 0) (color 0 0 0 0)
-  )
-  (junction (at 165.1 153.67) (diameter 0) (color 0 0 0 0)
-  )
-  (junction (at 190.5 200.66) (diameter 0) (color 0 0 0 0)
-  )
-  (junction (at 219.71 190.5) (diameter 0) (color 0 0 0 0)
-  )
-  (junction (at 232.41 209.55) (diameter 0) (color 0 0 0 0)
-  )
-  (junction (at 163.83 120.65) (diameter 0) (color 0 0 0 0)
-  )
-  (junction (at 250.19 212.09) (diameter 0) (color 0 0 0 0)
-  )
-  (junction (at 189.23 73.66) (diameter 0) (color 0 0 0 0)
-  )
-  (junction (at 201.93 118.11) (diameter 0) (color 0 0 0 0)
-  )
-  (junction (at 172.72 81.28) (diameter 0) (color 0 0 0 0)
-  )
-  (junction (at 153.67 93.98) (diameter 0) (color 0 0 0 0)
-  )
-  (junction (at 153.67 71.12) (diameter 0) (color 0 0 0 0)
-  )
-  (junction (at 237.49 78.74) (diameter 0) (color 0 0 0 0)
-  )
-  (junction (at 248.92 195.58) (diameter 0) (color 0 0 0 0)
-  )
-  (junction (at 163.83 71.12) (diameter 0) (color 0 0 0 0)
-  )
-  (junction (at 154.94 153.67) (diameter 0) (color 0 0 0 0)
-  )
-  (junction (at 189.23 118.11) (diameter 0) (color 0 0 0 0)
-  )
-  (junction (at 237.49 113.03) (diameter 0) (color 0 0 0 0)
-  )
-  (junction (at 203.2 200.66) (diameter 0) (color 0 0 0 0)
-  )
-  (junction (at 153.67 120.65) (diameter 0) (color 0 0 0 0)
-  )
-  (junction (at 172.72 110.49) (diameter 0) (color 0 0 0 0)
-  )
-  (junction (at 248.92 129.54) (diameter 0) (color 0 0 0 0)
-  )
   (junction (at 173.99 193.04) (diameter 0) (color 0 0 0 0)
   )
@@
     (stroke (width 0) (type default))
   )
+  (wire (pts (xy 154.94 200.66) (xy 154.94 203.2))
+    (stroke (width 0) (type default))
+  )
   (wire (pts (xy 209.55 200.66) (xy 203.2 200.66))
     (stroke (width 0) (type default))
@@
     (stroke (width 0) (type default))
   )
-  (wire (pts (xy 152.4 71.12) (xy 153.67 71.12))
+  (wire (pts (xy 26.67 71.12) (xy 153.67 71.12))
     (stroke (width 0) (type default))
   )
@@
     (stroke (width 0) (type default))
   )
+  (wire (pts (xy 153.67 118.11) (xy 153.67 120.65))
+    (stroke (width 0) (type default))
+  )
   (wire (pts (xy 247.65 195.58) (xy 248.92 195.58))
     (stroke (width 0) (type default))
@@
     (stroke (width 0) (type default))
   )
-  (wire (pts (xy 153.67 153.67) (xy 154.94 153.67))
+  (wire (pts (xy 27.94 153.67) (xy 154.94 153.67))
     (stroke (width 0) (type default))
   )
@@
     (stroke (width 0) (type default))
   )
-  (wire (pts (xy 153.67 120.65) (xy 153.67 118.11))
-    (stroke (width 0) (type default))
-  )
   (wire (pts (xy 172.72 110.49) (xy 172.72 115.57))
     (stroke (width 0) (type default))
@@
     (stroke (width 0) (type default))
   )
-  (wire (pts (xy 152.4 120.65) (xy 153.67 120.65))
+  (wire (pts (xy 26.67 120.65) (xy 153.67 120.65))
     (stroke (width 0) (type default))
   )
@@
     (stroke (width 0) (type default))
   )
-  (wire (pts (xy 154.94 203.2) (xy 154.94 200.66))
-    (stroke (width 0) (type default))
-  )
   (wire (pts (xy 247.65 78.74) (xy 247.65 90.17))
     (stroke (width 0) (type default))
@@
     (stroke (width 0) (type default))
   )
-  (wire (pts (xy 153.67 203.2) (xy 154.94 203.2))
+  (wire (pts (xy 27.94 203.2) (xy 154.94 203.2))
     (stroke (width 0) (type default))
   )
@@
     (effects (font (size 1.27 1.27)) (justify left bottom))
   )
+  (text "Niet leverbaar!" (at 97.79 96.52 0)
+    (effects (font (size 1.27 1.27)) (justify left bottom))
+  )
   (text "NA" (at 175.26 173.99 0)
     (effects (font (size 1.27 1.27)) (justify left bottom))
@@
     (effects (font (size 1.27 1.27)) (justify left bottom))
   )
-  (hierarchical_label "XLR_CH4(+)" (shape input) (at 153.67 153.67 180) (fields_autoplaced)
+  (hierarchical_label "XLR_CH4(+)" (shape input) (at 27.94 153.67 180) (fields_autoplaced)
     (effects (font (size 1.27 1.27)) (justify right))
   )
-  (hierarchical_label "XLR_CH3(+)" (shape input) (at 152.4 71.12 180) (fields_autoplaced)
+  (hierarchical_label "XLR_CH3(+)" (shape input) (at 26.67 71.12 180) (fields_autoplaced)
     (effects (font (size 1.27 1.27)) (justify right))
   )
-  (hierarchical_label "XLR_CH4(-)" (shape input) (at 153.67 203.2 180) (fields_autoplaced)
+  (hierarchical_label "XLR_CH4(-)" (shape input) (at 27.94 203.2 180) (fields_autoplaced)
     (effects (font (size 1.27 1.27)) (justify right))
   )
-  (hierarchical_label "XLR_CH3(-)" (shape input) (at 152.4 120.65 180) (fields_autoplaced)
+  (hierarchical_label "XLR_CH3(-)" (shape input) (at 26.67 120.65 180) (fields_autoplaced)
     (effects (font (size 1.27 1.27)) (justify right))
   )
@@
         )
       )
+    )
+  )
+  (symbol (lib_id "Device:D_TVS") (at 88.9 95.25 90) (unit 1)
+    (in_bom yes) (on_board yes) (dnp no) (fields_autoplaced)
+    (property "Reference" "D4" (at 91.44 94.615 90)
+      (effects (font (size 1.27 1.27)) (justify right))
+    )
+    (property "Value" "D_TVS" (at 91.44 97.155 90)
+      (effects (font (size 1.27 1.27)) (justify right))
+    )
+    (property "Footprint" "" (at 88.9 95.25 0)
+      (effects (font (size 1.27 1.27)) hide)
+    )
+    (property "Datasheet" "" (at 88.9 95.25 0)
+      (effects (font (size 1.27 1.27)) hide)
+    )
+    (pin "1")
+    (pin "2")
+    (instances
+      (project "Main board"
+        (path "/2f8cbac6-fd11-4240-8e40-3bb6952a0324/4e10d7ae-7c54-4ac5-ac67-e4842ffdf025"
+          (reference "D4") (unit 1)
+        )
+        (path "/2f8cbac6-fd11-4240-8e40-3bb6952a0324/b7530516-5ab1-4afa-9366-b30c4f029458"
+          (reference "D5") (unit 1)
+        )
+      )

Commit message: Worked on main board schematic
Parts:
- added D4: CPDT-12V, Package_TO_SOT_SMD:SOT-23, symbol Device:D_TVS
- D4: value D_TVS -> CPDT-12V; footprint (none) -> Package_TO_SOT_SMD:SOT-23
Other:
- note removed: "Niet leverbaar!"
Changed lines of the file:
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@@
-    (effects (font (size 1.27 1.27)) (justify left bottom))
-  )
-  (text "Niet leverbaar!" (at 97.79 96.52 0)
     (effects (font (size 1.27 1.27)) (justify left bottom))
   )
@@
       (effects (font (size 1.27 1.27)) (justify right))
     )
-    (property "Value" "D_TVS" (at 91.44 97.155 90)
+    (property "Value" "CPDT-12V" (at 91.44 97.155 90)
       (effects (font (size 1.27 1.27)) (justify right))
     )
-    (property "Footprint" "" (at 88.9 95.25 0)
-      (effects (font (size 1.27 1.27)) hide)
-    )
-    (property "Datasheet" "" (at 88.9 95.25 0)
+    (property "Footprint" "Package_TO_SOT_SMD:SOT-23" (at 88.9 95.25 0)
+      (effects (font (size 1.27 1.27)) hide)
+    )
+    (property "Datasheet" "https://nl.mouser.com/ProductDetail/Comchip-Technology/CPDT-12V?qs=tw%252BuQ%2FB6PO0KPAaKlo8Fww%3D%3D" (at 88.9 95.25 0)
       (effects (font (size 1.27 1.27)) hide)
     )
@@
         )
       )
+    )
+  )
+  (symbol (lib_id "Device:D_TVS") (at 88.9 176.53 90) (unit 1)
+    (in_bom yes) (on_board yes) (dnp no) (fields_autoplaced)
+    (property "Reference" "D4" (at 91.44 175.895 90)
+      (effects (font (size 1.27 1.27)) (justify right))
+    )
+    (property "Value" "CPDT-12V" (at 91.44 178.435 90)
+      (effects (font (size 1.27 1.27)) (justify right))
+    )
+    (property "Footprint" "Package_TO_SOT_SMD:SOT-23" (at 88.9 176.53 0)
+      (effects (font (size 1.27 1.27)) hide)
+    )
+    (property "Datasheet" "https://nl.mouser.com/ProductDetail/Comchip-Technology/CPDT-12V?qs=tw%252BuQ%2FB6PO0KPAaKlo8Fww%3D%3D" (at 88.9 176.53 0)
+      (effects (font (size 1.27 1.27)) hide)
+    )
+    (pin "1")
+    (pin "2")
+    (instances
+      (project "Main board"
+        (path "/2f8cbac6-fd11-4240-8e40-3bb6952a0324/4e10d7ae-7c54-4ac5-ac67-e4842ffdf025"
+          (reference "D4") (unit 1)
+        )
+        (path "/2f8cbac6-fd11-4240-8e40-3bb6952a0324/b7530516-5ab1-4afa-9366-b30c4f029458"
+          (reference "D6") (unit 1)
+        )
+      )

Commit message: Main board, ordering of PCBs and LTspice simulations
Parts:
- added C1 (x4), C5, C9 (x3): 100n, Capacitor_SMD:C_0402_1005Metric, symbol Device:C
- added C13, C39: 22uF, Capacitor_THT:CP_Radial_D5.0mm_P2.00mm, symbol Device:C_Polarized
- added C27 (x2), C28 (x2): 1n, Capacitor_SMD:C_0805_2012Metric, symbol Device:C
- added C30 (x2): 2n7, Capacitor_SMD:C_0805_2012Metric, symbol Device:C
- added R1: 10R, Resistor_SMD:R_0805_2012Metric, symbol Device:R
- added R15 (x2), R16 (x2), R20 (x2): 1k, Resistor_SMD:R_0805_2012Metric, symbol Device:R
- added R19 (x2), R20 (x2): 270, Resistor_SMD:R_0805_2012Metric, symbol Device:R
- added R33 (x2), R34 (x2): 39, Resistor_SMD:R_0805_2012Metric, symbol Device:R
- added RN1: 22R, Resistor_SMD:R_Array_Convex_4x0402, symbol Device:R_Pack04
- added U24, U6: LM4562, Package_SO:SOIC-8_3.9x4.9mm_P1.27mm, symbol Audio-DSP:LM4562
- added unit 1 of U24
- added U4 (x2): OPA1632DR, Audio-DSP:VSSOP-8_3.0x3.0mm_P0.65_TP1.8x1.5, symbol Audio-DSP:OPA1632DR
- added U7: PCM1804, Package_SO:SSOP-28_5.3x10.2mm_P0.65mm, symbol Audio_DSP:PCM1804
Connections:
- net GND: now also C1.2, C1.2, C1.2, C1.2, C13.2, C39.2, C5.1, C9.1, C9.1, C9.1, U4.7 (ENABLE), U4.7 (ENABLE), U4.9 (GND), U4.9 (GND), U7.12 (BYPAS), U7.13 (DGND), U7.2 (AGNDL), U7.23 (AGND), U7.27 (AGNDR), U7.7 (FMT1), U7.8 (S/~{M})
- new net: C28.1, R16.2, R20.1, U4.1 (VIN-) (x2)
- new net: C28.2, R34.1, U4.4 (VOUT+) (x2)
- new net: C30.2, R20.2, R34.2, U7.24 (VINR-)
- new net: C27.1, R15.2, R19.1, U4.8 (VIN+) (x2)
- new net: C30.1, R19.2, R33.2, U7.4 (VINL+)
- new net: C1.1, R20.2, U7.3 (VCOML)
- new net: C27.2, R33.1, U4.5 (VOUT-) (x2)
- new net: C1.1, U7.1 (VREFL)
- new net: R15.1, U6.1, U6.2 (-)
- new net: U4.2 (VOCM), U6.6 (-), U6.7
- new net: C30.1, R19.2, R33.2, U7.25 (VINR+)
- new net: C13.1, C9.2, R1.2, U7.22 (VCC)
- new net: U24.6 (-), U24.7, U4.2 (VOCM)
- new net: RN1.4 (R4.1), U7.15 (DATA/DSDR)
- new net: RN1.3 (R3.1), U7.16 (BCK/DSDL)
- new net: RN1.2 (R2.1), U7.17 (LRCK/DSDBCK)
- new net: RN1.1 (R1.1), U7.18 (SCKI)
- new net: C1.1, R20.2, U7.26 (VCOMR)
- new net: C1.1, U7.28 (VREFR)
- new net: C30.2, R20.2, R34.2, U7.5 (VINL-)
- new net: C9.2, R20.1, U24.5 (+)
- new net: C9.2, R20.1, U6.5 (+)
- new net: R15.1, U24.1, U24.2 (-)
- new net +3V3D1: C39.1, C5.2, U7.10 (OSR1), U7.11 (OSR2), U7.14 (VDD), U7.19 (~{RST}), U7.6 (FMT0), U7.9 (OSR0)
- new net +5VA1: R1.1
- new net AGND_CH1: R16.1
- new net AGND_CH2: R16.1
- new net BCK_ADC_CH3_4: RN1.6 (R3.2)
- new net DATA_ADC_CH3_4: RN1.5 (R4.2)
- new net LRCK_ADC_CH3_4: RN1.7 (R2.2)
- new net SCKI_ADC_CH3_4: RN1.8 (R1.2)
- no-connect marks 0 -> 2
Other:
- note added: "Add 0R resistors to be able to change some settings? -Sample freq -bits"
- note added: "Check symbol and footprint with someone else"
- note added: "HPF active"
- note added: "I2S format"
- note added: "Master mode"
- note added: "QUAD mode"
- note added: "RST inactive"
- note added: "VCOMx is the common mode reference voltage of 2.5V. VREFx is the reference voltage of the internal BGR."
- moved on the sheet: C27, C28, C30, C9, D4, R1, R15, R16, R19, R20, R33, R34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
