File: KiCAD/Main board/DAC_CH3_4.kicad_sch (KiCad schematic)
At the start: 43 parts, among them U1 PCM1789, U3 OPA1632DR, U4 OPA1632DR

Commit message: Ad good as finilized the main board schematic
Other:
- note added: "Adress=1"
- note added: "Combine I2C busses of the DACs? Otherwise they can get the same adress."
- note removed: "-Use Panasonic 0805 ERA series for audio path resistors -Use C0G MLCC capacitors for audio path capacitors"
- title: (none) -> AUDIO-DSP_MAIN_BOARD
Changed lines of the file:
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@@
 (kicad_sch (version 20230121) (generator eeschema)
   (paper "A4")
+  (title_block
+    (title "AUDIO-DSP_MAIN_BOARD")
+    (rev "R01")
+  )
   (junction (at 173.99 115.57) (diameter 0) (color 0 0 0 0)
   )
@@
     (stroke (width 0) (type default))
   )
-  (text "-Use Panasonic 0805 ERA series for audio path resistors\n-Use C0G MLCC capacitors for audio path capacitors"
-    (at 181.61 17.78 0)
+  (text "Combine I2C busses of the DACs?\nOtherwise they can get the same adress."
+    (at 44.45 106.68 0)
     (effects (font (size 1.27 1.27) (color 200 0 200 1)) (justify left bottom))
   )
+  (text "Adress=1" (at 59.69 95.25 0)
+    (effects (font (size 1.27 1.27)) (justify left bottom))
+  )
   (hierarchical_label "VOUT_XLR_CH3(-)" (shape output) (at 175.26 29.21 0) (fields_autoplaced)
