File: KiCAD/Main board/DAC_CH5_6.kicad_sch (KiCad schematic)
At the start: 43 parts, among them U1 PCM1789, U3 OPA1632DR, U4 OPA1632DR

Commit message: Ad good as finilized the main board schematic
Other:
- note added: "Adress=2"
- note added: "Combine I2C busses of the DACs? Otherwise they can get the same adress."
- note removed: "-Use Panasonic 0805 ERA series for audio path resistors -Use C0G MLCC capacitors for audio path capacitors"
- title: (none) -> AUDIO-DSP_MAIN_BOARD
Changed lines of the file:
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@@
 (kicad_sch (version 20230121) (generator eeschema)
   (paper "A4")
+  (title_block
+    (title "AUDIO-DSP_MAIN_BOARD")
+    (rev "R01")
+  )
   (junction (at 99.06 34.29) (diameter 0) (color 0 0 0 0)
   )
@@
     (stroke (width 0) (type default))
   )
-  (text "-Use Panasonic 0805 ERA series for audio path resistors\n-Use C0G MLCC capacitors for audio path capacitors"
-    (at 176.53 17.78 0)
+  (text "Adress=2" (at 59.69 95.25 0)
+    (effects (font (size 1.27 1.27)) (justify left bottom))
+  )
+  (text "Combine I2C busses of the DACs?\nOtherwise they can get the same adress."
+    (at 44.45 107.95 0)
     (effects (font (size 1.27 1.27) (color 200 0 200 1)) (justify left bottom))
   )
