File: KiCAD/Main board/POWER_SUPPLIES.kicad_sch (KiCad schematic)
At the start: 43 parts, among them U18 12V, U19 5V, U20 8V, U21 15V, U23 LIN_REG_±5V, U24 LIN_REG_±12V, U28 12V, U29 AP2111H-3.3TRG1, U31 AP2111H-3.3TRG1, U9 SEPIC_-15V_LT3579

Commit message: PCB finished + gerber
Parts:
- added TP28, TP29: TestPoint, TestPoint:TestPoint_Pad_D2.0mm, symbol Connector:TestPoint
Connections:
- net GND: now also TP28.1, TP29.1
- net TP_U29: now reaches U29.4 (TP)
- net TP_U31: now reaches U31.4 (TP)
- no-connect marks 2 -> 0
Changed lines of the file:
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@@
   (junction (at 114.3 161.29) (diameter 0) (color 0 0 0 0)
   )
+  (junction (at 140.97 19.05) (diameter 0) (color 0 0 0 0)
+  )
   (junction (at 55.88 44.45) (diameter 0) (color 0 0 0 0)
   )
   (junction (at 129.54 19.05) (diameter 0) (color 0 0 0 0)
   )
+  (junction (at 140.97 29.21) (diameter 0) (color 0 0 0 0)
+  )
   (junction (at 100.33 97.79) (diameter 0) (color 0 0 0 0)
   )
@@
   (junction (at 30.48 124.46) (diameter 0) (color 0 0 0 0)
   )
-  (no_connect (at 125.73 176.53))
-  (no_connect (at 125.73 151.13))
   (wire (pts (xy 55.88 101.6) (xy 55.88 104.14))
     (stroke (width 0) (type default))
@@
     (stroke (width 0) (type default))
   )
+  (wire (pts (xy 140.97 29.21) (xy 152.4 29.21))
+    (stroke (width 0) (type default))
+  )
   (wire (pts (xy 115.57 85.09) (xy 116.84 85.09))
     (stroke (width 0) (type default))
@@
     (stroke (width 0) (type default))
   )
+  (wire (pts (xy 125.73 151.13) (xy 132.08 151.13))
+    (stroke (width 0) (type default))
+  )
   (wire (pts (xy 55.88 101.6) (xy 68.58 101.6))
     (stroke (width 0) (type default))
@@
     (stroke (width 0) (type default))
   )
+  (wire (pts (xy 125.73 176.53) (xy 132.08 176.53))
+    (stroke (width 0) (type default))
+  )
   (wire (pts (xy 30.48 62.23) (xy 30.48 101.6))
     (stroke (width 0) (type default))
@@
   )
   (wire (pts (xy 30.48 21.59) (xy 30.48 44.45))
+    (stroke (width 0) (type default))
+  )
+  (wire (pts (xy 140.97 19.05) (xy 152.4 19.05))
     (stroke (width 0) (type default))
   )
@@
   )
   (text "DAC" (at 140.97 175.26 0)
+    (effects (font (size 1.27 1.27)) (justify left bottom))
+  )
+  (label "TP_U29" (at 125.73 151.13 0) (fields_autoplaced)
+    (effects (font (size 1.27 1.27)) (justify left bottom))
+  )
+  (label "TP_U31" (at 125.73 176.53 0) (fields_autoplaced)
     (effects (font (size 1.27 1.27)) (justify left bottom))
   )
@@
     )
   )
+  (symbol (lib_id "Connector:TestPoint") (at 152.4 19.05 0) (unit 1)
+    (in_bom yes) (on_board yes) (dnp no)
+    (property "Reference" "TP28" (at 153.67 15.24 0)
+      (effects (font (size 1.27 1.27)) (justify left))
+    )
+    (property "Value" "TestPoint" (at 153.67 17.78 0)
+      (effects (font (size 1.27 1.27)) (justify left))
+    )
+    (property "Footprint" "TestPoint:TestPoint_Pad_D2.0mm" (at 157.48 19.05 0)
+      (effects (font (size 1.27 1.27)) hide)
+    )
+    (property "Datasheet" "~" (at 157.48 19.05 0)
+      (effects (font (size 1.27 1.27)) hide)
+    )
+    (pin "1")
+    (instances
+      (project "Main board"
+        (path "/2f8cbac6-fd11-4240-8e40-3bb6952a0324/fc272ee1-9060-465b-85c1-b8364d68deb3"
+          (reference "TP28") (unit 1)
+        )
+      )
+    )
+  )
   (symbol (lib_id "Audio-DSP:LIN_REG_±12V") (at 115.57 99.06 0) (unit 1)
     (in_bom yes) (on_board yes) (dnp no) (fields_autoplaced)
@@
         )
       )
+    )
+  )
+  (symbol (lib_id "Connector:TestPoint") (at 152.4 29.21 0) (unit 1)
+    (in_bom yes) (on_board yes) (dnp no)
+    (property "Reference" "TP29" (at 153.67 25.4 0)
+      (effects (font (size 1.27 1.27)) (justify left))
+    )
+    (property "Value" "TestPoint" (at 153.67 27.94 0)
+      (effects (font (size 1.27 1.27)) (justify left))
+    )
+    (property "Footprint" "TestPoint:TestPoint_Pad_D2.0mm" (at 157.48 29.21 0)
+      (effects (font (size 1.27 1.27)) hide)
+    )
+    (property "Datasheet" "~" (at 157.48 29.21 0)
+      (effects (font (size 1.27 1.27)) hide)
+    )
+    (pin "1")
+    (instances
+      (project "Main board"
+        (path "/2f8cbac6-fd11-4240-8e40-3bb6952a0324/fc272ee1-9060-465b-85c1-b8364d68deb3"
+          (reference "TP29") (unit 1)
+        )
+      )
