File: KiCAD/-15V SEPIC/_autosave--15V SEPIC.kicad_pcb (KiCad board)
At the start: 4 copper layers, 24 x 30 mm, 21 parts, among them J1 Conn_01x04_Pin, U1 LT3579

Commit message: GBR files sepic
Routing:
- net GND: vias 75 -> 57
Other:
- board text added: "AUDIO DSP"
- board text added: "JLCJLCJLCJLC"
- board text added: "SEPIC -15V"
