File: KiCAD/Generic_Buck_Converter/Generic_Buck_Converter.kicad_pcb (KiCad board)
At the start: 4 copper layers, 17.8 x 25 mm, 20 parts, among them IC1 MAX17634C, J1 Conn_01x03

Commit message: Worked on main board
Changed lines of the file:
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@@
     (connect_pads (clearance 0.5))
     (min_thickness 0.25) (filled_areas_thickness no)
-    (fill yes (thermal_gap 0.5) (thermal_bridge_width 0.5))
+    (fill (thermal_gap 0.5) (thermal_bridge_width 0.5))
     (polygon
       (pts
-        (xy 125 100)
-        (xy 125 125)
+        (xy 117.8 99.95)
+        (xy 117.8 124.95)
         (xy 100 125)
         (xy 100 100)

Commit message: Buck PCB
Parts:
- moved R4 0.50 mm to (102.5, 107.3)
- moved R6 0.50 mm to (102.5, 108.2)
- moved C2 0.25 mm to (105.8, 107.4)
- moved C6 0.14 mm to (101.8, 111.5)
Routing:
- net GND: track 0.79 -> 12.5 mm
- net Net-(IC1-EN/UVLO): track 0.00 -> 4.21 mm
- net Net-(IC1-RESET): track 0.00 -> 2.42 mm
- net Net-(IC1-INTVCC): track 0.00 -> 2.37 mm
- net Net-(IC1-RT): track 0.00 -> 2.22 mm
- net /Vin: track 0.00 -> 1.32 mm
- net Net-(IC1-SS): track 0.00 -> 1.22 mm
- net Net-(C5-Pad2): track 1.11 -> 0.01 mm
- added copper zone on F.Cu, net /Vin
- added copper zone on F.Cu, net /Vout
- added copper zone on F.Cu, net Net-(C5-Pad2)
Changed lines of the file:
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@@
   (net 13 "Net-(IC1-EN{slash}UVLO)")
   (footprint "Resistor_SMD:R_0402_1005Metric" (layer "F.Cu")
-    (at 102.45 106.8 180)
+    (at 102.49 107.3 180)
     (descr "Resistor SMD 0402 (1005 Metric), square (rectangular) end terminal, IPC_7351 nominal, (Body size source: IPC-SM-782 page 72, https://www.pcb-3d.com/wordpress/wp-content/uploads/ipc-sm-782a_amendment_1_and_2.pdf), generated with kicad-footprint-generator")
     (tags "resistor")
@@
   )
   (footprint "Resistor_SMD:R_0402_1005Metric" (layer "F.Cu")
-    (at 102.45 107.75 180)
+    (at 102.49 108.25 180)
     (descr "Resistor SMD 0402 (1005 Metric), square (rectangular) end terminal, IPC_7351 nominal, (Body size source: IPC-SM-782 page 72, https://www.pcb-3d.com/wordpress/wp-content/uploads/ipc-sm-782a_amendment_1_and_2.pdf), generated with kicad-footprint-generator")
     (tags "resistor")
@@
   )
   (footprint "Capacitor_SMD:C_1210_3225Metric" (layer "F.Cu")
-    (at 105.75 107.65)
+    (at 105.75 107.4)
     (descr "Capacitor SMD 1210 (3225 Metric), square (rectangular) end terminal, IPC_7351 nominal, (Body size source: IPC-SM-782 page 76, https://www.pcb-3d.com/wordpress/wp-content/uploads/ipc-sm-782a_amendment_1_and_2.pdf), generated with kicad-footprint-generator")
     (tags "capacitor")
@@
   )
   (footprint "Capacitor_SMD:C_0402_1005Metric" (layer "F.Cu")
-    (at 101.65 111.45 180)
+    (at 101.75 111.55 180)
     (descr "Capacitor SMD 0402 (1005 Metric), square (rectangular) end terminal, IPC_7351 nominal, (Body size source: IPC-SM-782 page 76, https://www.pcb-3d.com/wordpress/wp-content/uploads/ipc-sm-782a_amendment_1_and_2.pdf), generated with kicad-footprint-generator")
     (tags "capacitor")
@@
   (gr_rect (start 100 100) (end 117.8 125)
     (stroke (width 0.1) (type default)) (fill none) (layer "Edge.Cuts"))
+  (segment (start 103 107.3) (end 104.175 107.3) (width 0.25) (layer "F.Cu") (net 1))
+  (segment (start 104.175 107.3) (end 104.275 107.4) (width 0.25) (layer "F.Cu") (net 1))
+  (segment (start 104.325 112.875) (end 105.325 111.875) (width 0.25) (layer "F.Cu") (net 2))
   (segment (start 101.25 113.46) (end 101.25 114.25) (width 0.25) (layer "F.Cu") (net 2))
+  (segment (start 103.3125 111.375) (end 104.825 111.375) (width 0.25) (layer "F.Cu") (net 2))
+  (segment (start 104.825 113.8875) (end 104.825 112.375) (width 0.25) (layer "F.Cu") (net 2))
+  (segment (start 106.325 109.8625) (end 106.325 110.875) (width 0.25) (layer "F.Cu") (net 2))
+  (segment (start 104.825 111.375) (end 105.325 111.875) (width 0.25) (layer "F.Cu") (net 2))
+  (segment (start 106.325 110.875) (end 105.325 111.875) (width 0.25) (layer "F.Cu") (net 2))
+  (segment (start 104.825 112.375) (end 105.325 111.875) (width 0.25) (layer "F.Cu") (net 2))
+  (segment (start 106.325 112.875) (end 105.325 111.875) (width 0.25) (layer "F.Cu") (net 2))
+  (segment (start 104.325 113.8875) (end 104.325 112.875) (width 0.25) (layer "F.Cu") (net 2))
+  (segment (start 106.325 113.8875) (end 106.325 112.875) (width 0.25) (layer "F.Cu") (net 2))
   (via (at 101.25 114.25) (size 0.55) (drill 0.25) (layers "F.Cu" "B.Cu") (free) (net 2))
+  (segment (start 102.17 110.13) (end 102.2 110.16) (width 0.25) (layer "F.Cu") (net 3))
+  (segment (start 101.25 110.13) (end 102.17 110.13) (width 0.25) (layer "F.Cu") (net 3))
+  (segment (start 102.915 110.875) (end 102.2 110.16) (width 0.25) (layer "F.Cu") (net 3))
+  (segment (start 103.3125 110.875) (end 102.915 110.875) (width 0.25) (layer "F.Cu") (net 3))
   (segment (start 102.2 113.46) (end 102.2 114.25) (width 0.25) (layer "F.Cu") (net 4))
   (via (at 102.2 114.25) (size 0.55) (drill 0.25) (layers "F.Cu" "B.Cu") (free) (net 4))
@@
   (segment (start 108.405 110.875) (end 108.45 110.92) (width 0.25) (layer "F.Cu") (net 5))
   (segment (start 108.445 111.875) (end 108.45 111.88) (width 0.25) (layer "F.Cu") (net 6))
-  (segment (start 107.3375 111.875) (end 108.445 111.875) (width 0.25) (layer "F.Cu") (net 6))
+  (segment (start 102.555 111.875) (end 103.3125 111.875) (width 0.25) (layer "F.Cu") (net 7))
+  (segment (start 102.23 111.55) (end 102.555 111.875) (width 0.25) (layer "F.Cu") (net 7))
+  (segment (start 102.2 109.14) (end 102.9225 109.8625) (width 0.25) (layer "F.Cu") (net 8))
+  (segment (start 102.9225 109.8625) (end 104.325 109.8625) (width 0.25) (layer "F.Cu") (net 8))
   (segment (start 102.265 112.375) (end 103.3125 112.375) (width 0.25) (layer "F.Cu") (net 9))
   (segment (start 101.25 112.44) (end 102.2 112.44) (width 0.25) (layer "F.Cu") (net 9))
   (segment (start 102.2 112.44) (end 102.265 112.375) (width 0.25) (layer "F.Cu") (net 9))
-  (zone (net 2) (net_name "GND") (layer "F.Cu") (name "GND") (hatch edge 0.5)
-    (connect_pads (clearance 0.15))
-    (min_thickness 0.25) (filled_areas_thickness no)
+  (segment (start 102.95 113.2375) (end 103.3125 112.875) (width 0.25) (layer "F.Cu") (net 10))
+  (segment (start 102.95 114.94) (end 102.95 113.2375) (width 0.25) (layer "F.Cu") (net 10))
+  (segment (start 104.825 109.451992) (end 104.825 109.8625) (width 0.25) (layer "F.Cu") (net 13))
+  (segment (start 101.98 107.3) (end 102.000538 107.3) (width 0.25) (layer "F.Cu") (net 13))
+  (segment (start 103 108.25) (end 103 108.363173) (width 0.25) (layer "F.Cu") (net 13))
+  (segment (start 102.000538 107.3) (end 102.950538 108.25) (width 0.25) (layer "F.Cu") (net 13))
+  (segment (start 103.811827 109.175) (end 104.548008 109.175) (width 0.25) (layer "F.Cu") (net 13))
+  (segment (start 102.950538 108.25) (end 103 108.25) (width 0.25) (layer "F.Cu") (net 13))
+  (segment (start 103 108.363173) (end 103.811827 109.175) (width 0.25) (layer "F.Cu") (net 13))
+  (segment (start 104.548008 109.175) (end 104.825 109.451992) (width 0.25) (layer "F.Cu") (net 13))
+  (zone (net 1) (net_name "/Vin") (layer "F.Cu") (name "Vin") (hatch edge 0.5)
+    (priority 1)
+    (connect_pads yes (clearance 0.15))
+    (min_thickness 0.15) (filled_areas_thickness no)
     (fill yes (thermal_gap 0.5) (thermal_bridge_width 0.5))
     (polygon
       (pts
-        (xy 100 99.975)
-        (xy 117.8 99.975)
-        (xy 117.8 124.975)
-        (xy 100 124.975)
+        (xy 107.5 124.8)
+        (xy 103.45 124.8)
+        (xy 103.45 114.4)
+        (xy 105.5 114.4)
+        (xy 105.55 114.35)
+        (xy 105.55 113.35)
+        (xy 106.05 113.35)
+        (xy 106.1 113.4)
+        (xy 106.1 120.85)
+        (xy 107.5 122.25)
       )
     )
   )
-  (zone (net 2) (net_name "GND") (layers "In1.Cu" "In2.Cu") (hatch edge 0.5)
-    (connect_pads (clearance 0.5))
-    (min_thickness 0.25) (filled_areas_thickness no)
+  (zone (net 6) (net_name "Net-(C5-Pad2)") (layer "F.Cu") (name "lx") (hatch edge 0.5)
+    (priority 3)
+    (connect_pads yes (clearance 0.15))
+    (min_thickness 0.15) (filled_areas_thickness no)
+    (fill yes (thermal_gap 0.5) (thermal_bridge_width 0.5))
+    (polygon
+      (pts
+        (xy 106.9 113.4)
+        (xy 108 114.5)
+        (xy 111.9 114.5)
+        (xy 111.9 107.7)
+        (xy 111.9 107.7)
+        (xy 109.02742 107.7)
+        (xy 108.75 107.9)
+        (xy 108.75 110.3)
+        (xy 106.9 110.3)
+        (xy 106.9 113.4)
+      )
+    )
+  )
+  (zone (net 4) (net_name "/Vout") (layer "F.Cu") (name "Vout") (hatch edge 0.5)
+    (priority 1)
+    (connect_pads yes (clearance 0.15))
+    (min_thickness 0.15) (filled_areas_thickness no)
+    (fill yes (thermal_gap 0.5) (thermal_bridge_width 0.5))
+    (polygon
+      (pts
+        (xy 110.85 100.9)
+        (xy 110.85 107.553906)
+        (xy 110.85 107.553906)
+        (xy 112.920098 107.5)
+        (xy 112.25 107.5)
+        (xy 112.25 114.748684)
+        (xy 112.25 114.748684)
+        (xy 110.3 114.8)
+        (xy 110.3 115.5)
+        (xy 110.3 124.75)
+        (xy 114.6 124.75)
+        (xy 115.1 124.25)
+        (xy 115.1 114.75)
+        (xy 115.9 113.95)
+        (xy 115.95 113.95)
+        (xy 115.95 100.95)
+        (xy 115.9 100.9)
+      )
+    )
+  )
+  (zone (net 2) (net_name "GND") (layers "F.Cu" "In1.Cu" "In2.Cu" "B.Cu") (name "GND") (hatch edge 0.5)
+    (connect_pads yes (clearance 0.15))
+    (min_thickness 0.15) (filled_areas_thickness no)
     (fill yes (thermal_gap 0.5) (thermal_bridge_width 0.5))
     (polygon
       (pts
         (xy 100 100)
-        (xy 117.75 100)
-        (xy 117.75 125)
+        (xy 117.8 100)
+        (xy 117.8 125)
         (xy 100 125)
       )
     )
-  )
-  (zone (net 2) (net_name "GND") (layer "B.Cu") (hatch edge 0.5)
-    (connect_pads (clearance 0.5))
-    (min_thickness 0.25) (filled_areas_thickness no)
-    (fill (thermal_gap 0.5) (thermal_bridge_width 0.5))
-    (polygon
-      (pts
-        (xy 117.8 99.95)
-        (xy 117.8 124.95)
-        (xy 100 125)
-        (xy 100 100)
-      )
-    )

Commit message: PCB update
Parts:
- J1: value Conn_01x03 -> Conn_01x05; footprint Connector_PinHeader_2.54mm:PinHeader_1x03_P2.54mm_Horizontal -> Connector_PinHeader_2.54mm:PinHeader_1x05_P2.54mm_Horizontal
- moved J1 2.62 mm to (114.0, 123.0)
- moved C5 0.75 mm to (108.5, 110.7)
Connections:
- J1 pad 1: /Vout -> GND
- J1 pad 2: GND -> /Vout
- J1 pad 3: /Vin -> GND
Routing:
- net /Vout: track 0.79 -> 11.4 mm, vias 1 -> 2
- net GND: vias 1 -> 2
Other:
- board size 17.8 x 25 mm -> 17.8 x 27 mm

Commit message: PCB_update
Parts:
- moved C5 0.20 mm to (108.5, 110.5)
Connections:
- J1 pad 1: GND -> /Vout
Routing:
- net GND: vias 2 -> 14
- net /Vin: vias 0 -> 4
- added copper zone on In2.Cu, net /Vin
Other:
- board text added: "JLCJLCJLCJLC"
Changed lines of the file:
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@@
   )
   (footprint "Capacitor_SMD:C_0402_1005Metric" (layer "F.Cu")
-    (at 108.45 110.65 -90)
+    (at 108.45 110.45 -90)
     (descr "Capacitor SMD 0402 (1005 Metric), square (rectangular) end terminal, IPC_7351 nominal, (Body size source: IPC-SM-782 page 76, https://www.pcb-3d.com/wordpress/wp-content/uploads/ipc-sm-782a_amendment_1_and_2.pdf), generated with kicad-footprint-generator")
     (tags "capacitor")
@@
       (stroke (width 0.1) (type solid)) (layer "F.Fab"))
     (pad "1" thru_hole rect (at 0 0 270) (size 1.7 1.7) (drill 1) (layers "*.Cu" "*.Mask")
-      (net 2 "GND") (pinfunction "Pin_1") (pintype "passive"))
+      (net 4 "/Vout") (pinfunction "Pin_1") (pintype "passive"))
     (pad "2" thru_hole oval (at 0 2.54 270) (size 1.7 1.7) (drill 1) (layers "*.Cu" "*.Mask")
       (net 4 "/Vout") (pinfunction "Pin_2") (pintype "passive"))
@@
   (gr_rect (start 100 100) (end 117.8 127.05)
     (stroke (width 0.1) (type default)) (fill none) (layer "Edge.Cuts"))
+  (gr_text "JLCJLCJLCJLC" (at 108.55 101.35) (layer "B.SilkS")
+    (effects (font (size 0.8 0.8) (thickness 0.15) bold) (justify left bottom mirror))
+  )
   (segment (start 103 107.3) (end 104.175 107.3) (width 0.3) (layer "F.Cu") (net 1))
   (segment (start 104.175 107.3) (end 104.275 107.4) (width 0.3) (layer "F.Cu") (net 1))
+  (via (at 105.4 106.2) (size 0.55) (drill 0.25) (layers "F.Cu" "B.Cu") (free) (net 1))
+  (via (at 104.95 105.55) (size 0.55) (drill 0.25) (layers "F.Cu" "B.Cu") (free) (net 1))
+  (via (at 104.15 105.55) (size 0.55) (drill 0.25) (layers "F.Cu" "B.Cu") (free) (net 1))
+  (via (at 105 120) (size 0.55) (drill 0.25) (layers "F.Cu" "B.Cu") (free) (net 1))
   (segment (start 104.325 112.875) (end 105.325 111.875) (width 0.25) (layer "F.Cu") (net 2))
   (segment (start 101.25 113.46) (end 101.25 114.25) (width 0.25) (layer "F.Cu") (net 2))
@@
   (segment (start 104.325 113.8875) (end 104.325 112.875) (width 0.25) (layer "F.Cu") (net 2))
   (segment (start 106.325 113.8875) (end 106.325 112.875) (width 0.25) (layer "F.Cu") (net 2))
+  (via (at 107.55 120) (size 0.55) (drill 0.25) (layers "F.Cu" "B.Cu") (free) (net 2))
+  (via (at 117 102) (size 0.55) (drill 0.25) (layers "F.Cu" "B.Cu") (free) (net 2))
   (via (at 111.7 114.25) (size 0.55) (drill 0.25) (layers "F.Cu" "B.Cu") (free) (net 2))
+  (via (at 109 126) (size 0.55) (drill 0.25) (layers "F.Cu" "B.Cu") (free) (net 2))
+  (via (at 107.55 118.1) (size 0.55) (drill 0.25) (layers "F.Cu" "B.Cu") (free) (net 2))
+  (via (at 102 106) (size 0.55) (drill 0.25) (layers "F.Cu" "B.Cu") (free) (net 2))
+  (via (at 107 102) (size 0.55) (drill 0.25) (layers "F.Cu" "B.Cu") (free) (net 2))
   (via (at 101.25 114.25) (size 0.55) (drill 0.25) (layers "F.Cu" "B.Cu") (free) (net 2))
+  (via (at 106.95 109.35) (size 0.55) (drill 0.25) (layers "F.Cu" "B.Cu") (free) (net 2))
+  (via (at 102.35 116.6) (size 0.55) (drill 0.25) (layers "F.Cu" "B.Cu") (free) (net 2))
+  (via (at 104 126) (size 0.55) (drill 0.25) (layers "F.Cu" "B.Cu") (free) (net 2))
+  (via (at 115 126) (size 0.55) (drill 0.25) (layers "F.Cu" "B.Cu") (free) (net 2))
+  (via (at 102 102) (size 0.55) (drill 0.25) (layers "F.Cu" "B.Cu") (free) (net 2))
+  (via (at 117 106) (size 0.55) (drill 0.25) (layers "F.Cu" "B.Cu") (free) (net 2))
   (segment (start 102.17 110.13) (end 102.2 110.16) (width 0.25) (layer "F.Cu") (net 3))
   (segment (start 101.25 110.13) (end 102.17 110.13) (width 0.25) (layer "F.Cu") (net 3))
@@
   (segment (start 102.46 110.16) (end 102.2 110.16) (width 0.25) (layer "F.Cu") (net 3))
   (segment (start 102.2 113.46) (end 102.2 114.25) (width 0.25) (layer "F.Cu") (net 4))
-  (via (at 112.55 113.7) (size 0.55) (drill 0.25) (layers "F.Cu" "B.Cu") (free) (net 4))
+  (via (at 112.6 113.6) (size 0.55) (drill 0.25) (layers "F.Cu" "B.Cu") (free) (net 4))
   (via (at 102.2 114.25) (size 0.55) (drill 0.25) (layers "F.Cu" "B.Cu") (free) (net 4))
-  (segment (start 102.8 113.65) (end 112.5 113.65) (width 0.25) (layer "B.Cu") (net 4))
-  (segment (start 112.5 113.65) (end 112.55 113.7) (width 0.25) (layer "B.Cu") (net 4))
-  (segment (start 102.2 114.25) (end 102.8 113.65) (width 0.25) (layer "B.Cu") (net 4))
-  (segment (start 108.407035 110.17) (end 108.45 110.17) (width 0.3) (layer "F.Cu") (net 5))
-  (segment (start 107.3375 110.875) (end 107.702035 110.875) (width 0.3) (layer "F.Cu") (net 5))
-  (segment (start 107.702035 110.875) (end 108.407035 110.17) (width 0.3) (layer "F.Cu") (net 5))
+  (segment (start 112.6 113.6) (end 106.748529 113.6) (width 0.25) (layer "In2.Cu") (net 4))
+  (segment (start 106.748529 113.6) (end 106.098529 114.25) (width 0.25) (layer "In2.Cu") (net 4))
+  (segment (start 106.098529 114.25) (end 102.2 114.25) (width 0.25) (layer "In2.Cu") (net 4))
+  (segment (start 108.427035 109.95) (end 108.45 109.95) (width 0.3) (layer "F.Cu") (net 5))
+  (segment (start 107.3375 110.875) (end 107.502035 110.875) (width 0.3) (layer "F.Cu") (net 5))
+  (segment (start 107.502035 110.875) (end 108.427035 109.95) (width 0.3) (layer "F.Cu") (net 5))
   (segment (start 102.555 111.875) (end 103.3125 111.875) (width 0.25) (layer "F.Cu") (net 7))
   (segment (start 102.23 111.55) (end 102.555 111.875) (width 0.25) (layer "F.Cu") (net 7))
@@
     (polygon
       (pts
-        (xy 103.7 106.05)
-        (xy 103.7 108.75)
-        (xy 105.2 108.75)
+        (xy 105.6 105.1)
+        (xy 104.05 105.1)
+        (xy 103.7 105.45)
+        (xy 103.7 108.7)
+        (xy 103.75 108.75)
+        (xy 104.65 108.75)
+        (xy 105.2 109.3)
         (xy 105.2 110.15)
         (xy 105.2 110.2)
         (xy 105.95 110.2)
-        (xy 105.95 106.05)
+        (xy 105.95 108.125)
+        (xy 105.95 107.2)
+        (xy 105.95 105.45)
       )
     )
   )
   (zone (net 1) (net_name "/Vin") (layer "F.Cu") (name "Vin") (hatch edge 0.5)
-    (priority 1)
+    (priority 2)
     (connect_pads yes (clearance 0.15))
     (min_thickness 0.15) (filled_areas_thickness no)
@@
     (polygon
       (pts
-        (xy 104.7 123.9)
-        (xy 102.924054 123.9)
-        (xy 102.900706 117.548335)
-        (xy 103.7 116.683264)
-        (xy 103.7 115.95)
-        (xy 103.711767 114.4)
-        (xy 105.5 114.4)
-        (xy 105.55 114.35)
-        (xy 105.55 113.55)
-        (xy 106 113.55)
-        (xy 106.1 113.55)
-        (xy 106.1 120.873229)
-        (xy 104.7 122.323229)
+        (xy 105.95 114.05)
+        (xy 105.95 113.55)
+        (xy 105.7 113.55)
+        (xy 105.7 114.7)
+        (xy 105.65 114.75)
+        (xy 103.75 114.75)
+        (xy 103.7 114.8)
+        (xy 103.7 117.45)
+        (xy 102.75 118.526667)
+        (xy 102.75 123.85)
+        (xy 102.8 123.9)
+        (xy 104.85 123.9)
+        (xy 104.9 123.85)
+        (xy 104.9 122.345244)
+        (xy 105.95 121.245244)
+        (xy 105.95 113.55)
+        (xy 105.95 113.55)
+        (xy 105.7 113.55)
+        (xy 105.7 113.8)
       )
     )
@@
         (xy 107 112.5)
         (xy 107.7 112.5)
-        (xy 108.1 113.23098)
         (xy 108.95 113.95)
-        (xy 111.25 113.95)
-        (xy 111.25 108.35)
-        (xy 109.522596 108.35)
-        (xy 108.75 108.906986)
-        (xy 108.75 110.5)
-        (xy 108 110.610769)
-        (xy 107 111.3)
+        (xy 111.2 113.95)
+        (xy 111.25 113.9)
+        (xy 111.25 111.125)
+        (xy 111.25 108.4)
+        (xy 111.2 108.35)
+        (xy 109.7 108.35)
+        (xy 108.95 109.1)
+        (xy 108.95 110.320789)
+        (xy 108.553588 110.6621)
+        (xy 108.273535 110.662849)
+        (xy 107.690208 111.250687)
+        (xy 107 111.25)
       )
     )
@@
     (polygon
       (pts
-        (xy 110.85 100.9)
-        (xy 110.85 107.553906)
-        (xy 112.920098 107.5)
-        (xy 112.25 107.5)
-        (xy 112.25 114.748684)
-        (xy 110.3 114.8)
-        (xy 110.3 115.5)
+        (xy 110.9 100.95)
+        (xy 110.85 101)
+        (xy 110.85 107.549999)
+        (xy 110.9 107.603743)
+        (xy 112.2 107.6)
+        (xy 112.25 107.65)
+        (xy 112.25 114.75)
+        (xy 112.2 114.798715)
+        (xy 110.35 114.799764)
+        (xy 110.3 114.85)
         (xy 110.3 124.1)
-        (xy 115.25 124.1)
-        (xy 115.1 124.25)
-        (xy 115.1 114.75)
-        (xy 115.95 113.95)
-        (xy 115.95 113.95)
-        (xy 115.95 100.95)
-        (xy 115.9 100.9)
+        (xy 110.35 124.15)
+        (xy 115.05 124.15)
+        (xy 115.1 124.1)
+        (xy 115.1 114.8)
+        (xy 115.95 114)
+        (xy 115.95 101)
+        (xy 115.9 100.95)
       )
     )
@@
       )
     )
+  )
+  (zone (net 1) (net_name "/Vin") (layer "In2.Cu") (name "Vin") (hatch edge 0.5)
+    (priority 4)
+    (connect_pads yes (clearance 0.15))
+    (min_thickness 0.15) (filled_areas_thickness no)
+    (fill yes (thermal_gap 0.5) (thermal_bridge_width 0.5))
+    (polygon
+      (pts
+        (xy 103.5 105.5)
+        (xy 104 105)
+        (xy 111 105)
+        (xy 117 111.010563)
+        (xy 117 115.5)
+        (xy 113.4 119.2)
+        (xy 108.8 119.2)
+        (xy 104.995092 123.004908)
+        (xy 104.98869 124)
+        (xy 104.5 124.5)
+        (xy 103 124.475886)
+        (xy 102.45 124)
+        (xy 102.45 120.749183)
+        (xy 107.746227 115.499063)
+        (xy 112.05 115.499963)
+        (xy 113 114.45)
+        (xy 113 113)
+        (xy 110 110)
+        (xy 106 110)
+        (xy 103.5 107.5)
+      )
+    )
