File: KiCAD/Generic_Buck_Converter/Generic_Buck_Converter.kicad_sch (KiCad schematic)
At the start: 20 parts, among them IC1 MAX17634C, J1 Conn_01x03

Commit message: PCB update
Parts:
- J1: value Conn_01x03 -> Conn_01x05; footprint Connector_PinHeader_2.54mm:PinHeader_1x03_P2.54mm_Horizontal -> Connector_PinHeader_2.54mm:PinHeader_1x05_P2.54mm_Horizontal; symbol Connector_Generic:Conn_01x03 -> Connector_Generic:Conn_01x05
Connections:
- net GND: now also J1.1 (Pin_1), J1.3 (Pin_3), J1.4 (Pin_4); no longer J1.2 (Pin_2)
- net Vin: now also J1.5 (Pin_5); no longer J1.3 (Pin_3)
- net Vout: now also J1.2 (Pin_2); no longer J1.1 (Pin_1)
Changed lines of the file:
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@@
+    (stroke (width 0) (type default))
+  )
+  (wire (pts (xy 48.26 83.82) (xy 54.61 83.82))
     (stroke (width 0) (type default))
   )
@@
     (stroke (width 0) (type default))
   )
+  (wire (pts (xy 48.26 76.2) (xy 54.61 76.2))
+    (stroke (width 0) (type default))
+  )
   (wire (pts (xy 78.74 33.02) (xy 85.09 33.02))
     (stroke (width 0) (type default))
@@
     (stroke (width 0) (type default))
   )
-  (wire (pts (xy 54.61 76.2) (xy 48.26 76.2))
+  (wire (pts (xy 48.26 73.66) (xy 55.88 73.66))
     (stroke (width 0) (type default))
   )
@@
     (stroke (width 0) (type default))
   )
-  (label "Vin" (at 54.61 76.2 180) (fields_autoplaced)
+  (label "Vin" (at 55.88 73.66 180) (fields_autoplaced)
     (effects (font (size 1.27 1.27)) (justify right bottom))
   )
@@
     )
   )
-  (symbol (lib_id "Connector_Generic:Conn_01x03") (at 43.18 78.74 180) (unit 1)
+  (symbol (lib_id "Connector_Generic:Conn_01x05") (at 43.18 78.74 180) (unit 1)
     (in_bom yes) (on_board yes) (dnp no)
     (property "Reference" "J1" (at 40.64 79.375 0)
       (effects (font (size 1.27 1.27)) (justify left))
     )
-    (property "Value" "Conn_01x03" (at 40.64 76.835 0)
-      (effects (font (size 1.27 1.27)) (justify left))
-    )
-    (property "Footprint" "Connector_PinHeader_2.54mm:PinHeader_1x03_P2.54mm_Horizontal" (at 43.18 78.74 0)
+    (property "Value" "Conn_01x05" (at 40.64 76.835 0)
+      (effects (font (size 1.27 1.27)) (justify left))
+    )
+    (property "Footprint" "Connector_PinHeader_2.54mm:PinHeader_1x05_P2.54mm_Horizontal" (at 43.18 78.74 0)
       (effects (font (size 1.27 1.27)) hide)
     )
@@
     (pin "2")
     (pin "3")
+    (pin "4")
+    (pin "5")
     (instances
       (project "Generic_Buck_Converter"
@@
         (path "/ace91bca-b85b-47b2-a493-cf613897ba9e"
           (reference "R3") (unit 1)
+        )
+      )
+    )
+  )
+  (symbol (lib_id "power:GND") (at 54.61 83.82 90) (unit 1)
+    (in_bom yes) (on_board yes) (dnp no) (fields_autoplaced)
+    (property "Reference" "#PWR04" (at 60.96 83.82 0)
+      (effects (font (size 1.27 1.27)) hide)
+    )
+    (property "Value" "GND" (at 58.42 83.185 90)
+      (effects (font (size 1.27 1.27)) (justify right))
+    )
+    (property "Footprint" "" (at 54.61 83.82 0)
+      (effects (font (size 1.27 1.27)) hide)
+    )
+    (property "Datasheet" "" (at 54.61 83.82 0)
+      (effects (font (size 1.27 1.27)) hide)
+    )
+    (pin "1")
+    (instances
+      (project "Generic_Buck_Converter"
+        (path "/ace91bca-b85b-47b2-a493-cf613897ba9e"
+          (reference "#PWR04") (unit 1)
         )
       )
@@
         )
       )
+    )
+  )
+  (symbol (lib_id "power:GND") (at 54.61 76.2 90) (unit 1)
+    (in_bom yes) (on_board yes) (dnp no) (fields_autoplaced)
+    (property "Reference" "#PWR02" (at 60.96 76.2 0)
+      (effects (font (size 1.27 1.27)) hide)
+    )
+    (property "Value" "GND" (at 58.42 75.565 90)
+      (effects (font (size 1.27 1.27)) (justify right))
+    )
+    (property "Footprint" "" (at 54.61 76.2 0)
+      (effects (font (size 1.27 1.27)) hide)
+    )
+    (property "Datasheet" "" (at 54.61 76.2 0)
+      (effects (font (size 1.27 1.27)) hide)
+    )
+    (pin "1")
+    (instances
+      (project "Generic_Buck_Converter"
+        (path "/ace91bca-b85b-47b2-a493-cf613897ba9e"
+          (reference "#PWR02") (unit 1)
+        )
+      )

Commit message: PCB_update
Parts:
- C1, C2: value C -> 10u
- C10, C11, C4, C7, C8, C9: value C -> 50u
- C3: value C -> 2.2u
- C5: value C -> 0.1u
- C6: value C -> 33n
- L1: value L -> X
- R1, R2: value R -> X
- R3: value R -> 20k
- R4: value R -> 3M3
- R5: value R -> 10k
- R6: value R -> 220k
Connections:
- net GND: no longer J1.1 (Pin_1)
- net Vout: now also J1.1 (Pin_1)
Other:
- note added: "5V 8V 12V 15V L1: 4.7u 6.8u 10u 15u R1: 22k 15k 22k 30k R2: 100k 120k 270k 470k"
- moved on the sheet: C1, C2, L1, R1, R2, R4, R6

Commit message: Schematic orderlist update
Parts:
- L1: Datasheet2 (none) -> https://nl.mouser.com/c/passive-components/resistors/?case%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; Datasheet3 (none) -> https://nl.mouser.com/c/passive-components/resistors/?case%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; Datasheet4 (none) -> https://nl.mouser.com/c/passive-components/resistors/?case%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
Changed lines of the file:
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@@
       (effects (font (size 1.27 1.27)) hide)
     )
-    (property "Datasheet" "~" (at 87.63 92.71 0)
+    (property "Datasheet" "https://eu.mouser.com/ProductDetail/Murata-Electronics/GRM155Z71A225KE01D?qs=d0WKAl%252BL4Kaf7%252BbBwe1qxg%3D%3D" (at 87.63 92.71 0)
       (effects (font (size 1.27 1.27)) hide)
     )
@@
       (effects (font (size 1.27 1.27)) hide)
     )
-    (property "Datasheet" "~" (at 139.065 81.28 0)
-      (effects (font (size 1.27 1.27)) hide)
-    )
-    (property "Datasheet2" "" (at 139.065 81.28 90)
-      (effects (font (size 1.27 1.27)) hide)
-    )
-    (property "Datasheet3" "" (at 139.065 81.28 90)
-      (effects (font (size 1.27 1.27)) hide)
-    )
-    (property "Datasheet4" "" (at 139.065 81.28 90)
-      (effects (font (size 1.27 1.27)) hide)
-    )
+    (property "Datasheet" "https://nl.mouser.com/c/passive-components/resistors/?case%20code%20-%20in=0402&tolerance=0.01~~0.02%20%25%7C~0.05%20%25~~0.1%20%25&rp=passive-components%2Fresistors%7C~Tolerance" (at 139.065 81.28 0)
+      (effects (font (size 1.27 1.27)) hide)
+    )
+    (property "Datasheet2" "https://nl.mouser.com/c/passive-components/resistors/?case%20code%20-%20in=0402&tolerance=0.01~~0.02%20%25%7C~0.05%20%25~~0.1%20%25&rp=passive-components%2Fresistors%7C~Tolerance" (at 139.065 81.28 90)
+      (effects (font (size 1.27 1.27)) hide)
+    )
+    (property "Datasheet3" "https://nl.mouser.com/c/passive-components/resistors/?case%20code%20-%20in=0402&tolerance=0.01~~0.02%20%25%7C~0.05%20%25~~0.1%20%25&rp=passive-components%2Fresistors%7C~Tolerance" (at 139.065 81.28 90)
+      (effects (font (size 1.27 1.27)) hide)
+    )
+    (property "Datasheet4" "https://nl.mouser.com/c/passive-components/resistors/?case%20code%20-%20in=0402&tolerance=0.01~~0.02%20%25%7C~0.05%20%25~~0.1%20%25&rp=passive-components%2Fresistors%7C~Tolerance" (at 139.065 81.28 90)
+      (effects (font (size 1.27 1.27)) hide)
+    )
