File: KiCAD/Generic_Buck_Converter/Generic_Buck_Converter.kicad_sch (KiCad schematic)
At the start: 20 parts, among them IC1 MAX17634C, J1 Conn_01x05

Commit message: Added Gerber + Excel-sheet
Parts:
- C10, C11, C4, C7, C8, C9: value 50u -> 10u
- IC1: Order https://nl.farnell.com/analog-devices/max17634catp/dc-dc-co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 -> (none)
- L1: value X -> X L1; Datasheet2 (none) -> https://nl.farnell.com/coilcraft/xal6060-682mec/inductor-6-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; Datasheet3 (none) -> https://nl.farnell.com/coilcraft/xal6060-103mec/inductor-10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; Datasheet4 (none) -> https://nl.farnell.com/coilcraft/xal6060-153mec/inductor-15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
- R1: value X -> X R1; Datasheet2 (none) -> https://nl.mouser.com/ProductDetail/Vishay-Dale/CRCW040215K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; Datasheet3 (none) -> https://nl.mouser.com/ProductDetail/Vishay-Dale/CRCW040222K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; Datasheet4 (none) -> https://nl.mouser.com/ProductDetail/Vishay-Dale/CRCW040230K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
- R2: value X -> X R2; Datasheet2 (none) -> https://nl.mouser.com/ProductDetail/Vishay-Dale/CRCW0402120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; Datasheet3 (none) -> https://nl.mouser.com/ProductDetail/Vishay-Dale/CRCW0402270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; Datasheet4 (none) -> https://nl.mouser.com/ProductDetail/Vishay-Dale/CRCW0402470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
