File: KiCAD/Discrete_linear_regulator/Discrete_linear_regulator.kicad_pcb (KiCad board)
At the start: 4 copper layers, 50 x 36 mm, 40 parts, among them J1 Conn_01x06, Q1 PZT2222AT3G, Q10 BC857, Q11 BC857, Q2 BC857, Q3 BC857, Q4 PZT2222AT3G, Q5 PZT2907AT3G, Q8 PZT2907AT3G, U1 LM4562

Commit message: update linear pcb
Parts:
- R13, R6: value 8k2 -> 6K8
- R14, R7: value 2k4 -> 1K2
Other:
- board size 50 x 36 mm -> 40.1 x 36 mm
Changed lines of the file:
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@@
         (effects (font (size 1 1) (thickness 0.15)))
     )
-    (fp_text value "2k4" (at 0.02 1.17) (layer "F.Fab")
+    (fp_text value "1K2" (at 0.02 1.17) (layer "F.Fab")
         (effects (font (size 1 1) (thickness 0.15)))
     )
@@
     (model "${KICAD6_3DMODEL_DIR}/Capacitor_THT.3dshapes/CP_Radial_D8.0mm_P3.50mm.wrl"
       (offset (xyz 0 0 0))
-      (scale (xyz 1 1 1))
+      (scale (xyz 1 1 0.875))
       (rotate (xyz 0 0 0))
     )
@@
     (model "${KICAD6_3DMODEL_DIR}/Capacitor_THT.3dshapes/CP_Radial_D8.0mm_P3.50mm.wrl"
       (offset (xyz 0 0 0))
-      (scale (xyz 1 1 1))
+      (scale (xyz 1 1 0.875))
       (rotate (xyz 0 0 0))
     )
@@
     (model "${KICAD6_3DMODEL_DIR}/Capacitor_THT.3dshapes/CP_Radial_D8.0mm_P3.50mm.wrl"
       (offset (xyz 0 0 0))
-      (scale (xyz 1 1 1))
+      (scale (xyz 1 1 0.875))
       (rotate (xyz 0 0 0))
     )
@@
     (model "${KICAD6_3DMODEL_DIR}/Capacitor_THT.3dshapes/CP_Radial_D8.0mm_P3.50mm.wrl"
       (offset (xyz 0 0 0))
-      (scale (xyz 1 1 1))
+      (scale (xyz 1 1 0.875))
       (rotate (xyz 0 0 0))
     )
@@
         (effects (font (size 1 1) (thickness 0.15)))
     )
-    (fp_text value "8k2" (at -2.39 0.44) (layer "F.Fab")
+    (fp_text value "6K8" (at -2.39 0.44) (layer "F.Fab")
         (effects (font (size 1 1) (thickness 0.15)))
     )
@@
         (effects (font (size 1 1) (thickness 0.15)))
     )
-    (fp_text value "2k4" (at -4.15 3.84 180) (layer "F.Fab")
+    (fp_text value "1K2" (at -4.15 3.84 180) (layer "F.Fab")
         (effects (font (size 1 1) (thickness 0.15)))
     )
@@
     (model "${KICAD6_3DMODEL_DIR}/Capacitor_THT.3dshapes/CP_Radial_D8.0mm_P3.50mm.wrl"
       (offset (xyz 0 0 0))
-      (scale (xyz 1 1 1))
+      (scale (xyz 1 1 0.875))
       (rotate (xyz 0 0 0))
     )
@@
     (model "${KICAD6_3DMODEL_DIR}/Capacitor_THT.3dshapes/CP_Radial_D8.0mm_P3.50mm.wrl"
       (offset (xyz 0 0 0))
-      (scale (xyz 1 1 1))
+      (scale (xyz 1 1 0.875))
       (rotate (xyz 0 0 0))
     )
@@
         (effects (font (size 1 1) (thickness 0.15)))
     )
-    (fp_text value "8k2" (at 0 -1.2 90) (layer "F.Fab")
+    (fp_text value "6K8" (at 0 -1.2 90) (layer "F.Fab")
         (effects (font (size 1 1) (thickness 0.15)))
     )
@@
     )
   )
-  (gr_arc (start 129.05 116.497349) (mid 125.514466 115.032883) (end 124.05 111.497349)
+  (gr_arc (start 134.035534 116.499971) (mid 130.505121 115.034635) (end 129.050001 111.5)
     (stroke (width 0.1) (type default)) (layer "Edge.Cuts"))
-  (gr_arc (start 169.05 80.497349) (mid 172.585534 81.961815) (end 174.05 85.497349)
+  (gr_arc (start 163.95 80.500001) (mid 167.572468 81.921191) (end 169.101123 85.499636)
     (stroke (width 0.1) (type default)) (layer "Edge.Cuts"))
-  (gr_arc (start 124.05 85.497349) (mid 125.514466 81.961815) (end 129.05 80.497349)
+  (gr_arc (start 129.05 85.5) (mid 130.514466 81.964467) (end 134.05 80.500001)
     (stroke (width 0.1) (type default)) (layer "Edge.Cuts"))
-  (gr_line (start 174.05 85.497349) (end 174.05 111.497349)
+  (gr_line (start 169.101123 85.499636) (end 169.1 111.4)
     (stroke (width 0.1) (type default)) (layer "Edge.Cuts"))
-  (gr_line (start 124.05 111.497349) (end 124.05 85.497349)
+  (gr_line (start 129.05 111.5) (end 129.05 85.5)
     (stroke (width 0.1) (type default)) (layer "Edge.Cuts"))
-  (gr_arc (start 174.05 111.497349) (mid 172.585534 115.032883) (end 169.05 116.497349)
+  (gr_arc (start 169.1 111.4) (mid 167.680886 114.998332) (end 164.115734 116.498856)
     (stroke (width 0.1) (type default)) (layer "Edge.Cuts"))
-  (gr_line (start 169.05 116.497349) (end 129.05 116.497349)
+  (gr_line (start 164.115734 116.498856) (end 134.035534 116.499971)
     (stroke (width 0.1) (type default)) (layer "Edge.Cuts"))
-  (gr_line (start 129.05 80.497349) (end 169.05 80.497349)
+  (gr_line (start 134.05 80.500001) (end 163.95 80.5)
     (stroke (width 0.1) (type default)) (layer "Edge.Cuts"))
   (segment (start 146.545 92.932349) (end 146.886396 92.932349) (width 0.2) (layer "F.Cu") (net 2))
@@
       (pts
         (xy 154.3 110.247349)
-        (xy 172.25 110.247349)
-        (xy 172.35 82.747349)
-        (xy 170.75 81.097349)
+        (xy 168.85 110.197349)
+        (xy 168.95 82.697349)
+        (xy 168.95 81.15)
         (xy 162.55 81.097349)
         (xy 162.55 82.847349)
@@
         (xy 146.65 110.297349)
         (xy 146.65 107.897349)
-        (xy 138.1 107.897349)
-        (xy 135.45 104.497349)
-        (xy 135.45 81.097349)
+        (xy 139.45 107.9)
+        (xy 137.05 104.347349)
+        (xy 137.05 80.947349)
         (xy 142.6 81.097349)
         (xy 142.6 106.897349)
@@
       (pts
         (xy 143.75 110.247349)
-        (xy 125.8 110.247349)
-        (xy 125.7 82.747349)
-        (xy 127.25 81.097349)
+        (xy 130.15 110.047349)
+        (xy 130.05 82.547349)
+        (xy 130.05 81.1)
         (xy 135.4 81.097349)
-        (xy 135.4 82.847349)
-        (xy 135.4 104.547349)
-        (xy 138.5 108.047349)
+        (xy 136.95 82.747349)
+        (xy 136.95 104.447349)
+        (xy 139.3 108.05)
         (xy 143.75 108.047349)
       )
